File: MotherBoard/_saved_Motherboard.sch (KiCad schematic (older format))
At the start: 195 parts, among them P8 CONN_02X23, P8A CONN_01X23, P8A_A CONN_01X23, P8B CONN_01X23, P8B_B CONN_01X23, P9 CONN_02X23, P9A CONN_01X23, P9A_A CONN_01X23, U0 CD74HC4067, U1 CD74HC4067, U2 CD74HC4067, U3 CD74HC4067, U4 CD74HC4067, U6 CD74HC4067

Commit message: Switching computers. Mac cannot handle this
Connections:
- net Sheet5869F1F7/OUT is gone; now on net Sheet5869F1F7/OUT: U6.24 (Vcc)
- net Sheet5869F1F7/OUT: no longer U1.24 (Vcc)
- new net Sheet5869F1F7/OUT: U1.24 (Vcc)
Changed lines of the file:
@@
 Text Label 26450 7350 0    60   ~ 0
 DI
-$Comp
-L BARREL_JACK CON?
-U 1 1 5856F692
-P 4000 1000
-F 0 "CON?" H 4000 1250 50  0000 C CNN
-F 1 "BARREL_JACK" H 4000 800 50  0000 C CNN
-F 2 "" H 4000 1000 50  0000 C CNN
-F 3 "" H 4000 1000 50  0000 C CNN
-	1    4000 1000
-	1    0    0    -1
-$EndComp
-Wire Notes Line
-	3100 700  6300 700
-Wire Notes Line
-	6300 700  6300 1400
-Wire Notes Line
-	6300 1400 3100 1400
-Wire Notes Line
-	3100 1400 3100 700
-$Comp
-L CONN_01X02 P?
-U 1 1 58572B80
-P 5550 1000
-F 0 "P?" H 5550 1150 50  0000 C CNN
-F 1 "CONN_01X02" V 5650 1000 50  0001 C CNN
-F 2 "" H 5550 1000 50  0000 C CNN
-F 3 "" H 5550 1000 50  0000 C CNN
-	1    5550 1000
-	1    0    0    -1
-$EndComp
-Wire Wire Line
-	4300 900  5350 900
-Wire Wire Line
-	5350 900  5350 950
-Wire Wire Line
-	4300 1000 4300 1100
-Wire Wire Line
-	4300 1100 5350 1100
-Wire Wire Line
-	5350 1100 5350 1050
-Text Label 4800 900  0    60   ~ 0
-5V
-Text Label 4800 1100 0    60   ~ 0
-GND
-Text Notes 3900 1400 0    118  ~ 24
-POWER TO BBB
 Wire Wire Line
 	25900 8500 26850 8500
@@
 	1    0    0    -1
 $EndComp
+Text Notes 3900 1400 0    118  ~ 24
+POWER TO BBB
+Text Label 4800 1100 0    60   ~ 0
+GND
+Text Label 4800 900  0    60   ~ 0
+5V
+Wire Wire Line
+	5350 1100 5350 1050
+Wire Wire Line
+	4300 1100 5350 1100
+Wire Wire Line
+	4300 1000 4300 1100
+Wire Wire Line
+	5350 900  5350 950
+Wire Wire Line
+	4300 900  5350 900
+$Comp
+L CONN_01X02 P?
+U 1 1 58572B80
+P 5550 1000
+F 0 "P?" H 5550 1150 50  0000 C CNN
+F 1 "CONN_01X02" V 5650 1000 50  0001 C CNN
+F 2 "" H 5550 1000 50  0000 C CNN
+F 3 "" H 5550 1000 50  0000 C CNN
+	1    5550 1000
+	1    0    0    -1
+$EndComp
+Wire Notes Line
+	3100 1400 3100 700
+Wire Notes Line
+	6300 1400 3100 1400
+Wire Notes Line
+	6300 700  6300 1400
+Wire Notes Line
+	3100 700  6300 700
+$Comp
+L BARREL_JACK CON?
+U 1 1 5856F692
+P 4000 1000
+F 0 "CON?" H 4000 1250 50  0000 C CNN
+F 1 "BARREL_JACK" H 4000 800 50  0000 C CNN
+F 2 "" H 4000 1000 50  0000 C CNN
+F 3 "" H 4000 1000 50  0000 C CNN
+	1    4000 1000
+	1    0    0    -1
+$EndComp
