File: MotherBoard/MPYE_DAC.sch (KiCad schematic (older format))
At the start: 12 parts

Commit message: Switching computers. Mac cannot handle this
Parts:
- R?: value R -> 2.4k
- R? (x2): value R -> 30k
Connections:
- net labels removed: VDD
- wire segments 35 -> 43
Other:
- moved on the sheet: R?

Commit message: Committing changes from Luke on MotherBoard
Parts:
- C301, C302, C303, C304: renamed from C?; footprint (none) -> Capacitors_SMD:C_0603_HandSoldering
- R301, R302, R303, R304, R305, R306, R307: renamed from R?; footprint (none) -> Resistors_SMD:R_0603_HandSoldering
- U301: renamed from U?; footprint (none) -> Housings_DFN_QFN:QFN-16-1EP_3x3mm_Pitch0.5mm; Digikey P/N (none) -> MAX5550ETE+-ND
Connections:
- net ~CS~: now also R305.1
- net 5V renamed +5V
