File: MotherBoard/Motherboard.sch (KiCad schematic (older format))
At the start: 195 parts, among them P8 CONN_02X23, P8A CONN_01X23, P8A_A CONN_01X23, P8B CONN_01X23, P8B_B CONN_01X23, P9 CONN_02X23, P9A CONN_01X23, P9A_A CONN_01X23, U0 CD74HC4067, U1 CD74HC4067, U2 CD74HC4067, U3 CD74HC4067, U4 CD74HC4067, U6 CD74HC4067

Commit message: Committing changes from Luke on MotherBoard
Parts:
- removed CON?: BARREL_JACK, symbol BARREL_JACK
- removed JP? (x122): JUMPER, symbol JUMPER
- removed P8A, P8A_A, P8B, P8B_B, P9A, P9A_A, PB, PB_B: CONN_01X23, symbol CONN_01X23
- removed P?: CONN_01X02, symbol CONN_01X02
- removed P? (x2): CONN_01X32, symbol CONN_01X32
- removed R? (x16): 470, symbol R
- removed U? (x4): ACSL-6400, symbol ACSL-6400
- added C107, C108, C109, C110, C111, C113, C115, C119, C121: 1uF, Capacitors_SMD:C_0603_HandSoldering, symbol C
- added P103, P104, P111: CONN_02X08, moboFootprints:Molex_16pin_milliGrid, symbol CONN_02X08
- added P105, P118, P121, P122, P123: CONN_02X24, moboFootprints:02x48pin_2x2mm_Amphenol_header, symbol CONN_02X24
- added P119: CONN_01X02, moboFootprints:SolderWirePad_2x_1mmDrill, symbol CONN_01X02
- added P120: CONN_01X16, moboFootprints:16pin_screwTerminal, symbol CONN_01X16
- added P124: CONN_01X01, moboFootprints:1pin, symbol CONN_01X01
- added P125: CONN_01X06, moboFootprints:CONN_01x06_standard, symbol CONN_01X06
- added P126: CONN_01X12, moboFootprints:12pin_screwTerminal, symbol CONN_01X12
- added P8_A101, P8_B101, P9_A101, P9_B101: CONN_02X23, moboFootprints:header_2.54x2.54mm_spacing_pinName, symbol CONN_02X23
- added R101, R103, R117, R131, R133, R164, R165: R, Resistors_SMD:R_0603_HandSoldering, symbol R
- added R102, R105, R106, R110, R120, R129, R130, R135, R136, R137, R138, R140, R141: SAT, Resistors_SMD:R_0603_HandSoldering, symbol R
- added R107, R109, R111, R112, R113, R114, R115, R116, R118, R119, R121, R124, R125, R126, R127, R128, R134, R144, R145, R146, R147, R148, R149, R150, R151, R152, R153, R154, R155, R156, R157, R158, R159, R160, R161, R162, R163: 0, Resistors_SMD:R_0603_HandSoldering, symbol R
- added R122, R123, R132, R143: 700, Resistors_SMD:R_0603_HandSoldering, symbol R
- added U103, U104, U107: THS4211, Housings_SOIC:SOIC-8_3.9x4.9mm_Pitch1.27mm, symbol THS4211
- added U108, U110, U111, U112: mounting_hole_5.5mm, Mounting_Holes:MountingHole_5.5mm_Pad_Via, symbol mounting_hole_5.5mm
- added U6: CD74HC4067, Housings_SOIC:SOIC-24W_7.5x15.4mm_Pitch1.27mm, symbol CD74HC4067
- C101, C102, C103, C104, C105, C106, C112, C114, C116, C117, C118, C120: renamed from C?; footprint (none) -> Capacitors_SMD:C_0603_HandSoldering
- P101: renamed from P?; footprint (none) -> moboFootprints:TEconnectivity_2pin_screwTerminal; Digikey P/N (none) -> A98333-ND
- P102: renamed from P?; footprint (none) -> moboFootprints:pheonix_4pin_screwTerminal; Digikey P/N (none) -> 277-1275-ND
- P106, P108, P112, P114, P116: renamed from P?; footprint (none) -> moboFootprints:TEconnectivity_2pin_screwTerminal
- P107: renamed from P?; footprint (none) -> moboFootprints:pheonix_4pin_screwTerminal; Digikey P/N (none) -> 277-1275-Nd
- P109, P110, P113, P115, P117: renamed from P?; footprint (none) -> moboFootprints:pheonix_4pin_screwTerminal
- P8: footprint (none) -> moboFootprints:header_2.54x2.54mm_spacing_pinName
- P9: footprint (none) -> moboFootprints:header_2.54x2.54mm_spacing_pinName; Digikey P/N (none) -> S2011E-23-ND
- R104, R108, R139, R142: renamed from R?; footprint (none) -> Resistors_SMD:R_0603_HandSoldering
- U0: footprint (none) -> Housings_SOIC:SOIC-24W_7.5x15.4mm_Pitch1.27mm; Digikey P/N (none) -> CD74HCT4067MG4-ND
- U1, U2, U3, U4: footprint (none) -> Housings_SOIC:SOIC-24W_7.5x15.4mm_Pitch1.27mm
- U101, U102, U106: renamed from U?; footprint (none) -> Housings_SOIC:SOIC-8_3.9x4.9mm_Pitch1.27mm
- U105: renamed from U?; footprint (none) -> Housings_SOIC:SOIC-8_3.9x4.9mm_Pitch1.27mm; Digikey P/N (none) -> 296-13790-5-ND
- U5: renamed from U6; footprint (none) -> Housings_SOIC:SOIC-24W_7.5x15.4mm_Pitch1.27mm
Connections:
- net 5V_in is gone; now on net +5V: P110.3 (P3), P110.4 (P4)
- net Sheet5869F1F7/OUT is gone; now on net 4V: U1.24 (Vcc)
- net Sheet5869F1F7/OUT is gone; now on net 4V: U0.24 (Vcc)
- net Sheet5869F1F7/OUT is gone; now on net 4V: U2.24 (Vcc)
- net Sheet5869F1F7/OUT is gone; now on net 4V: U3.24 (Vcc)
- net Sheet5869F1F7/OUT is gone; now on net 4V: U5.24 (Vcc)
- net DAC0/OUTA: now also P109.3 (P3); no longer P102.3 (P3)
- net DAC0/OUTB: now also P113.3 (P3); no longer P107.3 (P3)
- net DAC1/OUTA: now also P102.3 (P3); no longer P109.3 (P3)
- net DAC1/OUTB: now also P107.3 (P3); no longer P113.3 (P3)
- net DI: now also P9_B101.30 (P30)
- net GND: now also P101.2 (P2), P102.2 (P2), P102.4 (P4), C107.1, C108.1, C109.1, C110.1, C111.1, C113.1, C115.1, C119.1, C121.1, P105.10 (P10), P105.15 (P15), P105.16 (P16), P105.21 (P21), P105.22 (P22), P105.27 (P27), P105.28 (P28), P105.3 (P3), P105.33 (P33), P105.34 (P34), P105.39 (P39), P105.4 (P4), P105.40 (P40), P105.45 (P45), P105.46 (P46), P105.9 (P9), P118.10 (P10), P118.15 (P15), P118.16 (P16), P118.21 (P21), P118.22 (P22), P118.27 (P27), P118.28 (P28), P118.3 (P3), P118.33 (P33), P118.34 (P34), P118.39 (P39), P118.4 (P4), P118.40 (P40), P118.45 (P45), P118.46 (P46), P118.9 (P9), P119.2 (P2), P121.10 (P10), P121.15 (P15), P121.16 (P16), P121.21 (P21), P121.22 (P22), P121.27 (P27), P121.28 (P28), P121.3 (P3), P121.33 (P33), P121.34 (P34), P121.39 (P39), P121.4 (P4), P121.40 (P40), P121.45 (P45), P121.46 (P46), P121.9 (P9), P122.10 (P10), P122.15 (P15), P122.16 (P16), P122.21 (P21), P122.22 (P22), P122.27 (P27), P122.28 (P28), P122.3 (P3), P122.33 (P33), P122.34 (P34), P122.39 (P39), P122.4 (P4), P122.40 (P40), P122.45 (P45), P122.46 (P46), P122.9 (P9), P123.10 (P10), P123.15 (P15), P123.16 (P16), P123.21 (P21), P123.22 (P22), P123.27 (P27), P123.28 (P28), P123.3 (P3), P123.33 (P33), P123.34 (P34), P123.39 (P39), P123.4 (P4), P123.40 (P40), P123.45 (P45), P123.46 (P46), P123.9 (P9), P9_A101.1 (P1), P9_A101.43 (P43), P9_A101.45 (P45), P9_B101.2 (P2), P9_B101.34 (P34), P9_B101.44 (P44), P9_B101.46 (P46), R102.2, R105.2, R106.1, R107.1, R110.1, R112.1, R118.1, R120.2, R123.1, R129.2, R130.1, R135.2, R136.2, R137.2, R138.1, R140.1, R141.1, R144.1, R145.1, R147.1, R148.1, R165.2, U103.4 (-Vs), U104.4 (-Vs), U107.4 (-Vs), U108.1, U110.1, U111.1, U112.1, U6.12 (GND)
- net S0: now also P8_A101.11 (P11), R109.1, R114.1, R124.1, R146.1, R150.1, R155.1, R156.1
- net S1: now also P8_B101.12 (P12), R111.1, R116.1, R125.1, R149.1, R152.1, R158.1, R159.1; no longer P8.16 (P16)
- net S2: now also P8_A101.25 (P25), R113.1, R119.1, R126.1, R151.1, R154.1, R160.1, R161.1
- net S3: now also P8_A101.27 (P27), R115.1, R121.1, R127.1, R153.1, R157.1, R162.1, R163.1; no longer P8.18 (P18)
- net SCLK: now also P9_A101.31 (P31)
- net at P9.1 (P1): now also P9_A101.2 (P2)
- net at P9.10 (P10): now also P9_B101.9 (P9)
- net at P9.11 (P11): now also P9_A101.12 (P12)
- net at P9.12 (P12): now also P9_B101.11 (P11)
- net at P9.13 (P13): now also P9_A101.14 (P14)
- net at P9.14 (P14): now also P9_B101.13 (P13)
- net at P9.15 (P15): now also P9_A101.16 (P16)
- net at P9.16 (P16): now also P9_B101.15 (P15)
- net at P9.17 (P17): now also P9_A101.18 (P18)
- net at P9.18 (P18): now also P9_B101.17 (P17)
- net at P9.19 (P19): now also P9_A101.20 (P20)
- net at P9.2 (P2): now also P9_B101.1 (P1)
- net at P9.20 (P20): now also P9_B101.19 (P19)
- net at P9.21 (P21): now also P9_A101.22 (P22)
- net at P9.22 (P22): now also P9_B101.21 (P21)
- net at P9.23 (P23): now also P9_A101.24 (P24)
- net at P9.24 (P24): now also P9_B101.23 (P23)
- net at P9.25 (P25): now also P9_A101.26 (P26)
- net at P9.26 (P26): now also P9_B101.25 (P25)
- net at P9.27 (P27): now also P9_A101.28 (P28)
- net at P9.28 (P28): now also P9_B101.27 (P27)
- net at P9.29 (P29): now also P9_A101.30 (P30)
- net at P9.3 (P3): now also P9_A101.4 (P4)
- net at P9.30 (P30): now also P9_B101.29 (P29)
- net at P9.31 (P31): now also P9_A101.32 (P32)
- net at P9.32 (P32): now also P9_B101.31 (P31)
- net at P9.33 (P33): now also P9_A101.34 (P34)
- net at P9.34 (P34): now also P9_B101.33 (P33)
- net at P9.35 (P35): now also P9_A101.36 (P36)
- net at P9.36 (P36): now also P9_B101.35 (P35)
- net at P9.37 (P37): now also P9_A101.38 (P38)
- net at P9.38 (P38): now also P9_B101.37 (P37)
- net at P9.39 (P39): now also P9_A101.40 (P40)
- net at P9.4 (P4): now also P9_B101.3 (P3)
- net at P9.40 (P40): now also P9_B101.39 (P39)
- net at P9.41 (P41): now also P9_A101.42 (P42)
- net at P9.42 (P42): now also P9_B101.41 (P41)
- net at P9.43 (P43): now also P9_A101.44 (P44)
- net at P9.44 (P44): now also P9_B101.43 (P43)
- net at P9.45 (P45): now also P9_A101.46 (P46)
- net at P9.46 (P46): now also P9_B101.45 (P45)
- net at P9.5 (P5): now also P9_A101.6 (P6)
- net at P9.6 (P6): now also P9_B101.5 (P5)
- net at P9.7 (P7): now also P9_A101.8 (P8)
- net at P9.8 (P8): now also P9_B101.7 (P7)
- net at P9.9 (P9): now also P9_A101.10 (P10)
- net at U4.10 (S0): now also R155.2
- net at U4.11 (S1): now also R158.2
- net at U4.13 (S3): now also R162.2
- net at U4.14 (S2): now also R160.2
- net at U4.15 (~E~): now also R147.2
- net at U4.16 (I15): now also P118.6 (P6)
- net at U4.17 (I14): now also P118.12 (P12)
- net at U4.18 (I13): now also P118.18 (P18)
- net at U4.19 (I12): now also P118.24 (P24)
- net at U4.2 (I7): now also P118.47 (P47)
- net at U4.20 (I11): now also P118.30 (P30)
- net at U4.21 (I10): now also P118.36 (P36)
- net at U4.22 (I9): now also P118.42 (P42)
- net at U4.23 (I8): now also P118.48 (P48)
- net 4V: now reaches U4.24 (Vcc)
- net 4V: now also U6.24 (Vcc)
- net at U4.3 (I6): now also P118.41 (P41)
- net at U4.4 (I5): now also P118.35 (P35)
- net at U4.5 (I4): now also P118.29 (P29)
- net at U4.6 (I3): now also P118.23 (P23)
- net at U4.7 (I2): now also P118.17 (P17)
- net at U4.8 (I1): now also P118.11 (P11)
- net at U4.9 (I0): now also P118.5 (P5)
- net at U1.1 (COM_I/O): now also R122.2
- net at U1.10 (S0): now also R124.2
- net at U1.11 (S1): now also R125.2
- net at U1.13 (S3): now also R127.2
- net at U1.14 (S2): now also R126.2
- net at U1.15 (~E~): now also R118.2
- net at U1.9 (I0): now also P103.16 (P16)
- net at U0.1 (COM_I/O): now also R132.2
- net at U0.10 (S0): now also R146.2
- net at U0.11 (S1): now also R149.2
- net at U0.13 (S3): now also R153.2
- net at U0.14 (S2): now also R151.2
- net at U0.15 (~E~): now also R145.2
- net at U2.10 (S0): now also R150.2
- net at U2.11 (S1): now also R152.2
- net at U2.13 (S3): now also R157.2
- net at U2.14 (S2): now also R154.2
- net at U2.15 (~E~): now also R144.2
- net at U2.16 (I15): now also P105.6 (P6)
- net at U2.17 (I14): now also P105.12 (P12)
- net at U2.18 (I13): now also P105.18 (P18)
- net at U2.19 (I12): now also P105.24 (P24)
- net at U2.2 (I7): now also P105.47 (P47)
- net at U2.20 (I11): now also P105.30 (P30)
- net at U2.21 (I10): now also P105.36 (P36)
- net at U2.22 (I9): now also P105.42 (P42)
- net at U2.23 (I8): now also P105.48 (P48)
- net at U2.3 (I6): now also P105.41 (P41)
- net at U2.4 (I5): now also P105.35 (P35)
- net at U2.5 (I4): now also P105.29 (P29)
- net at U2.6 (I3): now also P105.23 (P23)
- net at U2.7 (I2): now also P105.17 (P17)
- net at U2.8 (I1): now also P105.11 (P11)
- net at U2.9 (I0): now also P105.5 (P5)
- net at C118.2, U106.6 (Vout): now also P9_A101.37 (P37), R133.1; no longer U106.2 (-IN)
- net at C116.2, U105.6 (Vout): now also P9_A101.33 (P33), R131.1; no longer U105.2 (-IN)
- net at C103.2, U101.6 (Vout): now also P9_A101.39 (P39), R101.1; no longer U101.2 (-IN)
- net at C105.2, U102.6 (Vout): now also P9_A101.35 (P35), R103.1; no longer U102.2 (-IN)
- net at P8.1 (P1): now also P8_A101.2 (P2)
- net at P8.10 (P10): now also P8_B101.9 (P9)
- net at P8.11 (P11): now also P8_A101.12 (P12)
- net at P8.12 (P12): now also P8_B101.11 (P11)
- net at P8.13 (P13): now also P8_A101.14 (P14)
- net at P8.14 (P14): now also P8_B101.13 (P13)
- net at P8.15 (P15): now also P8_A101.16 (P16)
- net at P8.17 (P17): now also P8_A101.18 (P18)
- net at P8.19 (P19): now also P8_A101.20 (P20)
- net at P8.2 (P2): now also P8_B101.1 (P1)
- net at P8.20 (P20): now also P8_B101.19 (P19)
- net at P8.22 (P22): now also P8_B101.21 (P21)
- net at P8.24 (P24): now also P8_B101.23 (P23)
- net at P8.26 (P26): now also P8_B101.25 (P25)
- net at P8.27 (P27): now also P8_A101.28 (P28)
- net at P8.28 (P28): now also P8_B101.27 (P27)
- net at P8.29 (P29): now also P8_A101.30 (P30)
- net at P8.3 (P3): now also P8_A101.4 (P4)
- net at P8.30 (P30): now also P8_B101.29 (P29)
- net at P8.31 (P31): now also P8_A101.32 (P32)
- net at P8.32 (P32): now also P8_B101.31 (P31)
- net at P8.33 (P33): now also P8_A101.34 (P34)
- net at P8.34 (P34): now also P8_B101.33 (P33)
- net at P8.35 (P35): now also P8_A101.36 (P36)
- net at P8.36 (P36): now also P8_B101.35 (P35)
- net at P8.37 (P37): now also P8_A101.38 (P38)
- net at P8.38 (P38): now also P8_B101.37 (P37)
- net at P8.39 (P39): now also P8_A101.40 (P40)
- net at P8.4 (P4): now also P8_B101.3 (P3)
- net at P8.40 (P40): now also P8_B101.39 (P39)
- net at P8.41 (P41): now also P8_A101.42 (P42)
- net at P8.42 (P42): now also P8_B101.41 (P41)
- net at P8.43 (P43): now also P8_A101.44 (P44)
- net at P8.44 (P44): now also P8_B101.43 (P43)
- net at P8.45 (P45): now also P8_A101.46 (P46)
- net at P8.46 (P46): now also P8_B101.45 (P45)
- net at P8.5 (P5): now also P8_A101.6 (P6)
- net at P8.6 (P6): now also P8_B101.5 (P5)
- net at P8.7 (P7): now also P8_A101.8 (P8)
- net at P8.8 (P8): now also P8_B101.7 (P7)
- net at P8.9 (P9): now also P8_A101.10 (P10)
- net at R139.1, U105.3 (IN+): now also C117.2, R138.2
- net +24V: now reaches P101.1 (P1), P102.1 (P1)
- net +24V: now also P106.1 (P1), P107.1 (P1), P108.1 (P1), P109.1 (P1), P112.1 (P1), P113.1 (P1), P114.1 (P1), P115.1 (P1), P116.1 (P1), P117.1 (P1)
- net at R142.1, U106.3 (IN+): now also C120.2, R140.2
- net at U3.10 (S0): now also R114.2
- net at U3.11 (S1): now also R116.2
- net at U3.14 (S2): now also R119.2
- net at U3.13 (S3): now also R121.2
- net at U3.15 (~E~): now also R112.2
- net at C106.2, R108.1, U102.3 (IN+): now also R110.2
- net at U5.10 (S0): now also R109.2
- net at U5.11 (S1): now also R111.2
- net at U5.14 (S2): now also R113.2
- net at U5.13 (S3): now also R115.2
- net at U5.15 (~E~): now also R107.2
- net at C104.2, R104.1, U101.3 (IN+): now also R106.2
- net at U3.16 (I15): now also P121.6 (P6)
- net at U3.17 (I14): now also P121.12 (P12)
- net at U3.18 (I13): now also P121.18 (P18)
- net at U3.19 (I12): now also P121.24 (P24)
- net at U3.2 (I7): now also P121.47 (P47)
- net at U3.20 (I11): now also P121.30 (P30)
- net at U3.21 (I10): now also P121.36 (P36)
- net at U3.22 (I9): now also P121.42 (P42)
- net at U3.23 (I8): now also P121.48 (P48)
- net at U3.3 (I6): now also P121.41 (P41)
- net at U3.4 (I5): now also P121.35 (P35)
- net at U3.5 (I4): now also P121.29 (P29)
- net at U3.6 (I3): now also P121.23 (P23)
- net at U3.7 (I2): now also P121.17 (P17)
- net at U3.8 (I1): now also P121.11 (P11)
- net at U3.9 (I0): now also P121.5 (P5)
- net at U5.16 (I15): now also P122.6 (P6)
- net at U5.17 (I14): now also P122.12 (P12)
- net at U5.18 (I13): now also P122.18 (P18)
- net at U5.19 (I12): now also P122.24 (P24)
- net at U5.2 (I7): now also P122.47 (P47)
- net at U5.20 (I11): now also P122.30 (P30)
- net at U5.21 (I10): now also P122.36 (P36)
- net at U5.22 (I9): now also P122.42 (P42)
- net at U5.23 (I8): now also P122.48 (P48)
- net at U5.3 (I6): now also P122.41 (P41)
- net at U5.4 (I5): now also P122.35 (P35)
- net at U5.5 (I4): now also P122.29 (P29)
- net at U5.6 (I3): now also P122.23 (P23)
- net at U5.7 (I2): now also P122.17 (P17)
- net at U5.8 (I1): now also P122.11 (P11)
- net at U5.9 (I0): now also P122.5 (P5)
- net 5V renamed +5V
- net +5V: now also C107.2, C110.2, C115.2, P119.1 (P1), U103.7 (Vs+), U104.7 (Vs+), U107.7 (Vs+)
- net DAC0/~CS~: no longer names the net of P8.21 (P21)
- net DAC0/~CS~: now also P8_A101.22 (P22)
- net DAC1/~CS~: no longer names the net of P8.23 (P23)
- net DAC1/~CS~: now also P8_A101.24 (P24)
- net DAC2/~CS~: no longer names the net of P8.25 (P25)
- net DAC2/~CS~: now also P8_A101.26 (P26)
- net tempAmp0/OUT: no longer names the net of U0.9 (I0)
- net tempAmp0/OUT: now also P104.16 (P16)
- net tempAmp1/OUT: no longer names the net of U0.8 (I1)
- net tempAmp1/OUT: now also P104.14 (P14)
- net tempAmp10/OUT: no longer names the net of U0.21 (I10)
- net tempAmp10/OUT: now also P104.5 (P5)
- net tempAmp11/OUT: no longer names the net of U0.20 (I11)
- net tempAmp11/OUT: now also P104.7 (P7)
- net tempAmp12/OUT: no longer names the net of U0.19 (I12)
- net tempAmp12/OUT: now also P104.9 (P9)
- net tempAmp13/OUT: no longer names the net of U0.18 (I13)
- net tempAmp13/OUT: now also P104.11 (P11)
- net tempAmp14/OUT: no longer names the net of U0.17 (I14)
- net tempAmp14/OUT: now also P104.13 (P13)
- net tempAmp15/OUT: no longer names the net of U0.16 (I15)
- net tempAmp15/OUT: now also P104.15 (P15)
- net tempAmp17/OUT: no longer names the net of U1.8 (I1)
- net tempAmp17/OUT: now also P103.14 (P14)
- net tempAmp18/OUT: no longer names the net of U1.7 (I2)
- net tempAmp18/OUT: now also P103.12 (P12)
- net tempAmp19/OUT: no longer names the net of U1.6 (I3)
- net tempAmp19/OUT: now also P103.10 (P10)
- net tempAmp2/OUT: no longer names the net of U0.7 (I2)
- net tempAmp2/OUT: now also P104.12 (P12)
- net tempAmp20/OUT: no longer names the net of U1.5 (I4)
- net tempAmp20/OUT: now also P103.8 (P8)
- net tempAmp21/OUT: no longer names the net of U1.4 (I5)
- net tempAmp21/OUT: now also P103.6 (P6)
- net tempAmp22/OUT: no longer names the net of U1.3 (I6)
- net tempAmp22/OUT: now also P103.4 (P4)
- net tempAmp23/OUT: no longer names the net of U1.2 (I7)
- net tempAmp23/OUT: now also P103.2 (P2)
- net tempAmp24/OUT: no longer names the net of U1.23 (I8)
- net tempAmp24/OUT: now also P103.1 (P1)
- net tempAmp25/OUT: no longer names the net of U1.22 (I9)
- net tempAmp25/OUT: now also P103.3 (P3)
- net tempAmp26/OUT: no longer names the net of U1.21 (I10)
- net tempAmp26/OUT: now also P103.5 (P5)
- net tempAmp27/OUT: no longer names the net of U1.20 (I11)
- net tempAmp27/OUT: now also P103.7 (P7)
- net tempAmp28/OUT: no longer names the net of U1.19 (I12)
- net tempAmp28/OUT: now also P103.9 (P9)
- net tempAmp29/OUT: no longer names the net of U1.18 (I13)
- net tempAmp29/OUT: now also P103.11 (P11)
- net tempAmp3/OUT: no longer names the net of U0.6 (I3)
- net tempAmp3/OUT: now also P104.10 (P10)
- net tempAmp30/OUT: no longer names the net of U1.17 (I14)
- net tempAmp30/OUT: now also P103.13 (P13)
- net tempAmp31/OUT: no longer names the net of U1.16 (I15)
- net tempAmp31/OUT: now also P103.15 (P15)
- net tempAmp4/OUT: no longer names the net of U0.5 (I4)
- net tempAmp4/OUT: now also P104.8 (P8)
- net tempAmp5/OUT: no longer names the net of U0.4 (I5)
- net tempAmp5/OUT: now also P104.6 (P6)
- net tempAmp6/OUT: no longer names the net of U0.3 (I6)
- net tempAmp6/OUT: now also P104.4 (P4)
- net tempAmp7/OUT: no longer names the net of U0.2 (I7)
- net tempAmp7/OUT: now also P104.2 (P2)
- net tempAmp8/OUT: no longer names the net of U0.23 (I8)
- net tempAmp8/OUT: now also P104.1 (P1)
- net tempAmp9/OUT: no longer names the net of U0.22 (I9)
- net tempAmp9/OUT: now also P104.3 (P3)
- new net: P8.16 (P16), P8_B101.15 (P15)
- new net: P8.18 (P18), P8_B101.17 (P17)
- new net: R131.2, R135.1, U105.2 (-IN)
- new net: R133.2, R136.1, U106.2 (-IN)
- new net: P111.15 (P15), P9_A101.11 (P11)
- new net: P111.13 (P13), P9_A101.13 (P13)
- new net: P111.11 (P11), P9_A101.15 (P15)
- new net: P111.9 (P9), P9_A101.21 (P21)
- new net: P111.7 (P7), P9_A101.23 (P23)
- new net: P111.5 (P5), P9_A101.25 (P25)
- new net: P111.3 (P3), P9_A101.27 (P27)
- new net: P9_A101.9 (P9), R164.2, R165.1
- new net: P111.16 (P16), P9_B101.12 (P12)
- new net: P111.14 (P14), P9_B101.14 (P14)
- new net: P111.12 (P12), P9_B101.16 (P16)
- new net: P111.10 (P10), P9_B101.22 (P22)
- new net: P111.8 (P8), P9_B101.24 (P24)
- new net: P111.6 (P6), P9_B101.26 (P26)
- new net: P111.4 (P4), P9_B101.28 (P28)
- new net: C108.2, P9_B101.36 (P36), R117.1, U103.6 (Vout)
- new net: C111.2, P9_B101.38 (P38), R128.1, U104.6 (Vout)
- new net: C119.2, P9_B101.40 (P40), R134.1, U107.6 (Vout)
- new net: P125.1 (P1), P8_B101.20 (P20)
- new net: P125.2 (P2), P8_B101.22 (P22)
- new net: P125.3 (P3), P8_B101.24 (P24)
- new net: P125.4 (P4), P8_B101.26 (P26)
- new net: P125.5 (P5), P8_B101.28 (P28)
- new net: P125.6 (P6), P8_B101.30 (P30)
- new net: R103.2, R105.1, U102.2 (-IN)
- new net: R101.2, R102.1, U101.2 (-IN)
- new net: P105.1 (P1), P105.13 (P13), P105.19 (P19), P105.25 (P25), P105.31 (P31), P105.37 (P37), P105.43 (P43), P105.7 (P7)
- new net: P105.14 (P14), P105.2 (P2), P105.20 (P20), P105.26 (P26), P105.32 (P32), P105.38 (P38), P105.44 (P44), P105.8 (P8)
- new net: P121.1 (P1), P121.13 (P13), P121.19 (P19), P121.25 (P25), P121.31 (P31), P121.37 (P37), P121.43 (P43), P121.7 (P7)
- new net: P121.14 (P14), P121.2 (P2), P121.20 (P20), P121.26 (P26), P121.32 (P32), P121.38 (P38), P121.44 (P44), P121.8 (P8)
- new net: P124.1 (P1), R164.1
- new net: P118.1 (P1), P118.13 (P13), P118.19 (P19), P118.25 (P25), P118.31 (P31), P118.37 (P37), P118.43 (P43), P118.7 (P7)
- new net: P118.14 (P14), P118.2 (P2), P118.20 (P20), P118.26 (P26), P118.32 (P32), P118.38 (P38), P118.44 (P44), P118.8 (P8)
- new net: P122.1 (P1), P122.13 (P13), P122.19 (P19), P122.25 (P25), P122.31 (P31), P122.37 (P37), P122.43 (P43), P122.7 (P7)
- new net: P122.14 (P14), P122.2 (P2), P122.20 (P20), P122.26 (P26), P122.32 (P32), P122.38 (P38), P122.44 (P44), P122.8 (P8)
- new net: P123.1 (P1), P123.13 (P13), P123.19 (P19), P123.25 (P25), P123.31 (P31), P123.37 (P37), P123.43 (P43), P123.7 (P7)
- new net: P123.11 (P11), U6.8 (I1)
- new net: P123.12 (P12), U6.17 (I14)
- new net: P123.14 (P14), P123.2 (P2), P123.20 (P20), P123.26 (P26), P123.32 (P32), P123.38 (P38), P123.44 (P44), P123.8 (P8)
- new net: P123.17 (P17), U6.7 (I2)
- new net: P123.18 (P18), U6.18 (I13)
- new net: P123.23 (P23), U6.6 (I3)
- new net: P123.24 (P24), U6.19 (I12)
- new net: P123.29 (P29), U6.5 (I4)
- new net: P123.30 (P30), U6.20 (I11)
- new net: P123.35 (P35), U6.4 (I5)
- new net: P123.36 (P36), U6.21 (I10)
- new net: P123.41 (P41), U6.3 (I6)
- new net: P123.42 (P42), U6.22 (I9)
- new net: P123.47 (P47), U6.2 (I7)
- new net: P123.48 (P48), U6.23 (I8)
- new net: P123.5 (P5), U6.9 (I0)
- new net: P123.6 (P6), U6.16 (I15)
- new net: C113.2, R130.2, R132.1, U104.3 (IN+)
- new net: R128.2, R129.1, U104.2 (-IN)
- new net: C109.2, R122.1, R123.2, U103.3 (IN+)
- new net: R117.2, R120.1, U103.2 (-IN)
- new net: C121.2, R141.2, R143.1, U107.3 (IN+)
- new net: R143.2, U6.1 (COM_I/O)
- new net: R134.2, R137.1, U107.2 (-IN)
- new net: R156.2, U6.10 (S0)
- new net: R159.2, U6.11 (S1)
- new net: R161.2, U6.14 (S2)
- new net: R163.2, U6.13 (S3)
- new net: R148.2, U6.15 (~E~)
- new net 0-2: P126.2 (P2), P126.4 (P4), P126.6 (P6)
- new net 3-5: P126.10 (P10), P126.12 (P12), P126.8 (P8)
- new net 3.3V: P9_B101.4 (P4)
- new net CS_0: P8_B101.18 (P18)
- new net CS_1: P8_B101.16 (P16)
- new net CS_2: P8_B101.14 (P14)
- new net D0: P9_A101.29 (P29)
- new net GNDA: P8_A101.1 (P1), P8_B101.2 (P2)
- new net Opto_0/GPIO_0: P8_A101.31 (P31)
- new net Opto_0/GPIO_1: P8_A101.33 (P33)
- new net Opto_0/GPIO_2: P8_A101.35 (P35)
- new net Opto_0/GPIO_3: P8_A101.37 (P37)
- new net Opto_0/Vout_0: P120.13 (P13)
- new net Opto_0/Vout_1: P120.14 (P14)
- new net Opto_0/Vout_2: P120.15 (P15)
- new net Opto_0/Vout_3: P120.16 (P16)
- new net Opto_1/GPIO_0: P8_A101.39 (P39)
- new net Opto_1/GPIO_1: P8_A101.41 (P41)
- new net Opto_1/GPIO_2: P8_A101.43 (P43)
- new net Opto_1/GPIO_3: P8_A101.45 (P45)
- new net Opto_1/Vout_0: P120.9 (P9)
- new net Opto_1/Vout_1: P120.10 (P10)
- new net Opto_1/Vout_2: P120.11 (P11)
- new net Opto_1/Vout_3: P120.12 (P12)
- new net Opto_2/GPIO_0: P8_B101.32 (P32)
- new net Opto_2/GPIO_1: P8_B101.34 (P34)
- new net Opto_2/GPIO_2: P8_B101.36 (P36)
- new net Opto_2/GPIO_3: P8_B101.38 (P38)
- new net Opto_2/Vout_0: P120.1 (P1)
- new net Opto_2/Vout_1: P120.2 (P2)
- new net Opto_2/Vout_2: P120.3 (P3)
- new net Opto_2/Vout_3: P120.4 (P4)
- new net Opto_3/GPIO_0: P8_B101.40 (P40)
- new net Opto_3/GPIO_1: P8_B101.42 (P42)
- new net Opto_3/GPIO_2: P8_B101.44 (P44)
- new net Opto_3/GPIO_3: P8_B101.46 (P46)
- new net Opto_3/Vout_0: P120.5 (P5)
- new net Opto_3/Vout_1: P120.6 (P6)
- new net Opto_3/Vout_2: P120.7 (P7)
- new net Opto_3/Vout_3: P120.8 (P8)
- new net SHARP_0: P126.1 (P1), P8_A101.13 (P13)
- new net SHARP_1: P126.3 (P3), P8_A101.15 (P15)
- new net SHARP_2: P126.5 (P5), P8_A101.17 (P17)
- new net SHARP_3: P126.7 (P7), P8_A101.19 (P19)
- new net SHARP_4: P126.9 (P9), P8_A101.21 (P21)
- new net SHARP_5: P126.11 (P11), P8_A101.23 (P23)
- new net SYS_RESET: P9_B101.10 (P10)
Other:
- note added: "GPIO FOR SHARP SENSORS\n"
- note added: "GPIO supply for Sharp Sensors"
- note added: "LP_Transducers\n\n\n\n\n"
- note added: "Lateral_Distance\n\n\n\n"
- note added: "PWR_BUT\n"
- note added: "Photodiodes\n\n\n\n\n"
- note added: "SPARE\n"
- note added: "Sharp / photodiodes"
- note added: "To BBB"
- note added: "Use Thicker Traces for 24V & GND"
- note added: "Vertical_Distance\n\n\n\n\n"
- note removed: "24V\n"
- note removed: "4V\n"
- note removed: "EXTRA/\nSPARE\n\n"
- note removed: "LCD PINS"
- note removed: "POWER TO BBB"
- note removed: "Transducer0\n"
- moved on the sheet: C101, C103, C104, C112, C114, C116, C117, C118, C120, P101, P102, P106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
