File: MotherBoard/tempAmp.sch (KiCad schematic (older format))
At the start: 9 parts

Commit message: Switching computers. Mac cannot handle this
Connections:
- net GND: now also C?.2, U?.3 (-Vs)
Changed lines of the file:
@@
 $Descr A4 11693 8268
 encoding utf-8
-Sheet 8 41
+Sheet 26 41
 Title ""
 Date ""
@@
 Connection ~ 5400 2300
 Wire Wire Line
-	6350 2600 6350 2800
-Wire Wire Line
-	6350 2800 6100 2800
+	6350 2800 6350 2600
+Wire Wire Line
+	5850 2800 6350 2800
 Connection ~ 6350 2800
 $Comp
@@
 Wire Wire Line
 	5200 2650 4900 2650
+Wire Wire Line
+	5850 2500 5850 2800
+Connection ~ 6100 2800
+Connection ~ 5850 2500
 $EndSCHEMATC

Commit message: Committing changes from Luke on MotherBoard
Parts:
- removed C?: 0.1uF, symbol C
- C201, C204: renamed from C?; footprint (none) -> Capacitors_SMD:C_0603_HandSoldering
- C203, C205: renamed from 100nF; footprint (none) -> Capacitors_SMD:C_0603_HandSoldering
- R203: renamed from SAT; footprint (none) -> Resistors_SMD:R_0603_HandSoldering
- R204, R205: renamed from R?; footprint (none) -> Resistors_SMD:R_0603_HandSoldering
- U202: renamed from U?; footprint (none) -> Housings_SSOP:MSOP-8_3x3mm_Pitch0.65mm; Digikey P/N (none) -> AD8497ARMZ-ND; Mfr. P/N (none) -> AD8497ARMZ
Connections:
- net GND: no longer U202.2 (REF)
- net at C203.2, R204.1, U202.1 (-In): now also C204.1; no longer C204.2
- net at C205.1, R205.1, U202.8 (+IN): now also C204.2; no longer C204.1
- new net REF: U202.2 (REF)
Other:
- note added: "Debugging: If AD849X is not working, remove thermocouple and short V+ \nand V- to GND. Will output ambient temperature.\n"
