File: LEDBoard/LEDBoard.kicad_pcb (KiCad board)
At the start: 2 copper layers, 240 parts, among them U1 LEDboardcomparator, U10 LEDboardcomparator, U11 LEDboardcomparator, U12 LEDboardcomparator, U13 LEDboardcomparator, U14 LEDboardcomparator, U15 LEDboardcomparator, U16 LEDboardcomparator, U2 LEDboardcomparator, U3 LEDboardcomparator, U4 LEDboardcomparator, U5 LEDboardcomparator, U6 LEDboardcomparator, U7 LEDboardcomparator, U8 LEDboardcomparator, U9 LEDboardcomparator

Commit message: made major changed to the led board mostly dealing with schematic
Parts:
- added D201: LED, LEDs:LED_1206, F.Cu at (410.8, 91.3)
- added P101: CONN_01X02, hyperCustom:CONN_PHOENIX_1844210_2PIN, F.Cu at (338.7, 1.24)
- added P102: CONN_01X02, hyperCustom:CONN_PHOENIX_1844210_2PIN, F.Cu at (321.6, 18.0)
- added P103: CONN_01X02, hyperCustom:CONN_PHOENIX_1844210_2PIN, F.Cu at (307.9, 18.2)
- added P104: CONN_01X02, hyperCustom:CONN_PHOENIX_1844210_2PIN, F.Cu at (325.0, 1.24)
- added P105: CONN_01X02, hyperCustom:CONN_PHOENIX_1844210_2PIN, F.Cu at (311.4, 1.24)
- added P106: CONN_01X02, hyperCustom:CONN_PHOENIX_1844210_2PIN, F.Cu at (294.3, 18.2)
- added P107: connector to 18650 batteries, hyperCustom:CONN_PHOENIX_1844210_2PIN, F.Cu at (277.8, 16.3)
- added P108: CONN_01X04, hyperCustom:CONN_PHOENIX_1844236_4PIN_1, F.Cu at (290.6, 0.92)
- added P109: CONN_01X06, hyperCustom:CONN_PHOENIX_1844252_6PIN, F.Cu at (167.8, -81.4)
- added R1801: 600K, Resistors_SMD:R_1206_HandSoldering, F.Cu at (374.4, 83.3)
- added R1802: 100K, Resistors_SMD:R_1206_HandSoldering, F.Cu at (367.3, 76.7)
- added R1803: 100K, Resistors_SMD:R_1206_HandSoldering, F.Cu at (367.3, 83.3)
- added R1804: 400K, Resistors_SMD:R_1206_HandSoldering, F.Cu at (374.4, 76.7)
- added R201: R, Resistors_SMD:R_1206_HandSoldering, F.Cu at (441.2, 76.7)
- added R202: R, Resistors_SMD:R_1206_HandSoldering, F.Cu at (434.1, 76.7)
- added R204: R, Resistors_SMD:R_1206_HandSoldering, F.Cu at (418.3, 84.5)
- added R205: R, Resistors_SMD:R_1206_HandSoldering, F.Cu at (411.4, 84.8)
- added R206: R, Resistors_SMD:R_1206_HandSoldering, F.Cu at (427.2, 84.0)
- added R207: R, Resistors_SMD:R_1206_HandSoldering, F.Cu at (432.4, 90.8)
- added R208: R, Resistors_SMD:R_1206_HandSoldering, F.Cu at (427.2, 76.9)
- added R210: R, Resistors_SMD:R_1206_HandSoldering, F.Cu at (425.3, 90.8)
- added R211: R, Resistors_SMD:R_1206_HandSoldering, F.Cu at (433.9, 83.6)
- added R212: R, Resistors_SMD:R_1206_HandSoldering, F.Cu at (439.4, 90.6)
- added R213: R, Resistors_SMD:R_1206_HandSoldering, F.Cu at (440.5, 83.6)
- added R403: R, Resistors_SMD:R_1206_HandSoldering, F.Cu at (285.8, 48.3)
- added R409: R, Resistors_SMD:R_1206_HandSoldering, F.Cu at (277.0, 56.1)
- added U201: LEDboardcomparator, TO_SOT_Packages_SMD:SOT-23-5, F.Cu at (416.0, 77.3)
- moved R302 361.9 mm to (491.7, 20.9)
- moved D801 354.3 mm to (475.8, 6.04)
- moved R802 354.3 mm to (478.4, -0.31)
- moved R803 354.3 mm to (469.6, 6.34)
- moved R804 354.3 mm to (478.4, -6.96)
- moved R805 354.3 mm to (471.4, -0.31)
- moved R806 354.3 mm to (462.5, 6.34)
- moved R807 354.3 mm to (471.4, -6.96)
- moved R808 354.3 mm to (455.5, 7.54)
- moved R811 354.3 mm to (455.5, 0.89)
- moved R801 354.3 mm to (485.5, -6.96)
- moved R809 354.3 mm to (464.3, -0.31)
- moved R810 354.3 mm to (448.4, 7.54)
- moved R812 354.3 mm to (464.3, -6.96)
- moved R813 354.3 mm to (448.4, 0.89)
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- renumbered D9 to D1001, D10 to D1101, D11 to D1201, D12 to D1301, D13 to D1401, D14 to D1501, D15 to D1601, D16 to D1701, D1 to D201, D2 to D301, D3 to D401, D4 to D501, D5 to D601, D6 to D701, D7 to D801, D8 to D901, R105 to R1001, R106 to R1002, R107 to R1003, R108 to R1004, R109 to R1005, R110 to R1006, R111 to R1007, R112 to R1008, R113 to R1009, R114 to R1010, R115 to R1011, R116 to R1012, R117 to R1013, R118 to R1101, R119 to R1102, R120 to R1103, R121 to R1104, R122 to R1105, R123 to R1106, R124 to R1107, R125 to R1108, R126 to R1109, R127 to R1110, R128 to R1111, R129 to R1112, R130 to R1113, R131 to R1201, R132 to R1202, R133 to R1203, R134 to R1204, R135 to R1205, R136 to R1206, R137 to R1207, R138 to R1208, R139 to R1209, R140 to R1210, R141 to R1211, R142 to R1212, R143 to R1213, R144 to R1301, R145 to R1302, R146 to R1303, R147 to R1304, R148 to R1305, R149 to R1306, R150 to R1307, R151 to R1308, R152 to R1309, R153 to R1310, R154 to R1311, R155 to R1312, R156 to R1313, R157 to R1401, R158 to R1402, R159 to R1403, R160 to R1404, R161 to R1405, R162 to R1406, R163 to R1407, R164 to R1408, R165 to R1409, R166 to R1410, R167 to R1411, R168 to R1412, R169 to R1413, R170 to R1501, R171 to R1502, R172 to R1503, R173 to R1504, R174 to R1505, R175 to R1506, R176 to R1507, R177 to R1508, R178 to R1509, R179 to R1510, R180 to R1511, R181 to R1512, R182 to R1513, R183 to R1601, R184 to R1602, R185 to R1603, R186 to R1604, R187 to R1605, R188 to R1606, R189 to R1607, R190 to R1608, R191 to R1609, R192 to R1610, R193 to R1611, R194 to R1612, R195 to R1613, R196 to R1701, R197 to R1702, R198 to R1703, R199 to R1704, R200 to R1705, R201 to R1706, R202 to R1707, R203 to R1708, R204 to R1709, R205 to R1710, R206 to R1711, R207 to R1712, R208 to R1713, R1 to R201, R2 to R202, R3 to R203, R4 to R204, R5 to R205, R6 to R206, R7 to R207, R8 to R208, R9 to R209, R10 to R210, R11 to R211, R12 to R212, R13 to R213, R14 to R301, R15 to R302, R16 to R303, R17 to R304, R18 to R305, R19 to R306, R20 to R307, R21 to R308, R22 to R309, R23 to R310, R24 to R311, R25 to R312, R26 to R313, R27 to R401, R28 to R402, R29 to R403, R30 to R404, R31 to R405, R32 to R406, R33 to R407, R34 to R408, R35 to R409, R36 to R410, R37 to R411, R38 to R412, R39 to R413, R40 to R501, R41 to R502, R42 to R503, R43 to R504, R44 to R505, R45 to R506, R46 to R507, R47 to R508, R48 to R509, R49 to R510, R50 to R511, R51 to R512, R52 to R513, R53 to R601, R54 to R602, R55 to R603, R56 to R604, R57 to R605, R58 to R606, R59 to R607, R60 to R608, R61 to R609, R62 to R610, R63 to R611, R64 to R612, R65 to R613, R66 to R701, R67 to R702, R68 to R703, R69 to R704, R70 to R705, R71 to R706, R72 to R707, R73 to R708, R74 to R709, R75 to R710, R76 to R711, R77 to R712, R78 to R713, R79 to R801, R80 to R802, R81 to R803, R82 to R804, R83 to R805, R84 to R806, R85 to R807, R86 to R808, R87 to R809, R88 to R810, R89 to R811, R90 to R812, R91 to R813, R92 to R901, R93 to R902, R94 to R903, R95 to R904, R96 to R905, R97 to R906, R98 to R907, R99 to R908, R100 to R909, R101 to R910, R102 to R911, R103 to R912, R104 to R913, U9 to U1001, U10 to U1101, U11 to U1201, U12 to U1301, U13 to U1401, U14 to U1501, U15 to U1601, U16 to U1701, U1 to U201, U2 to U301, U3 to U401, U4 to U501, U5 to U601, U6 to U701, U7 to U801, U8 to U901
Connections:
- R1003 pad 1: / Indicator Circuit for <3>/Vin -> /State
- R1103 pad 1: / Indicator Circuit for <7>/Vin -> /MerklState
- R1203 pad 1: / Indicator Circuit for <11>/Vin -> /Ind1
- R1303 pad 1: / Indicator Circuit for <15>/Vin -> /Ind5
- R1403 pad 1: / Indicator Circuit for <4>/Vin -> /State
- R1503 pad 1: / Indicator Circuit for <8>/Vin -> /MerklState
- R1603 pad 1: / Indicator Circuit for <12>/Vin -> /Ind2
- R1703 pad 1: / Indicator Circuit for <16>/Vin -> /Ind6
- R203 pad 1: / Indicator Circuit for <battery charge on>/Vin -> /Vbat
- R303 pad 1: / Indicator Circuit for <5>/Vin -> /Vcc_Bat
- R503 pad 1: / Indicator Circuit for <13>/Vin -> /Ind3
- R603 pad 1: / Indicator Circuit for <battery status off>/Vin -> /Vbat
- R703 pad 1: / Indicator Circuit for <6>/Vin -> /Vcc_Bat
- R803 pad 1: / Indicator Circuit for <10>/Vin -> /Merkl2
- R903 pad 1: / Indicator Circuit for <14>/Vin -> /Ind4
Routing:
- net (no net): track 0.00 -> 101.9 mm
- net Net-(R1608-Pad1): track 0.00 -> 79.9 mm
- net / Indicator Circuit for <12>/Vin_div: track 0.00 -> 1.10 mm
Other:
- board outline added: 358.6 x 213 mm

Commit message: akdhf
Parts:
- removed D1001, D1101, D1201, D1301, D1401, D1501, D1601, D1701, D301, D401, D501, D601, D701, D801, D901: LED, LEDs:LED_1206
- removed the D201 at (410.8, 91.3)
- removed R1001, R1002, R1003, R1004, R1005, R1006, R1007, R1008, R1009, R1010, R1011, R1012, R1013, R1101, R1102, R1103, R1104, R1105, R1106, R1107, R1108, R1109, R1110, R1111, R1112, R1113, R1201, R1202, R1203, R1204, R1205, R1206, R1207, R1208, R1209, R1210, R1211, R1212, R1213, R1301, R1302, R1303, R1304, R1305, R1306, R1307, R1308, R1309, R1310, R1311, R1312, R1313, R1401, R1402, R1403, R1404, R1405, R1406, R1407, R1408, R1409, R1410, R1411, R1412, R1413, R1501, R1502, R1503, R1504, R1505, R1506, R1507, R1508, R1509, R1510, R1511, R1512, R1513, R1601, R1602, R1603, R1604, R1605, R1606, R1607, R1608, R1609, R1610, R1611, R1612, R1613, R1701, R1702, R1703, R1704, R1705, R1706, R1707, R1708, R1709, R1710, R1711, R1712, R1713, R301, R302, R303, R304, R305, R306, R307, R308, R309, R310, R311, R312, R313, R401, R402, R403 (x2), R404, R405, R406, R407, R408, R409 (x2), R410, R411, R412, R413, R501, R502, R503, R504, R505, R506, R507, R508, R509, R510, R511, R512, R513, R601, R602, R603, R604, R605, R606, R607, R608, R609, R610, R611, R612, R613, R701, R702, R703, R704, R705, R706, R707, R708, R709, R710, R711, R712, R713, R801, R802, R803, R804, R805, R806, R807, R808, R809, R810, R811, R812, R813, R901, R902, R903, R904, R905, R906, R907, R908, R909, R910, R911, R912, R913: R, Resistors_SMD:R_1206_HandSoldering
- removed R1801: 600K, Resistors_SMD:R_1206_HandSoldering
- removed R1802, R1803: 100K, Resistors_SMD:R_1206_HandSoldering
- removed R1804: 400K, Resistors_SMD:R_1206_HandSoldering
- removed the R201 at (441.2, 76.7)
- removed the R202 at (434.1, 76.7)
- removed the R204 at (418.3, 84.5)
- removed the R205 at (411.4, 84.8)
- removed the R206 at (427.2, 84.0)
- removed the R207 at (432.4, 90.8)
- removed the R208 at (427.2, 76.9)
- removed the R210 at (425.3, 90.8)
- removed the R211 at (433.9, 83.6)
- removed the R212 at (439.4, 90.6)
- removed the R213 at (440.5, 83.6)
- removed U1001, U1101, U1201, U1301, U1401, U1501, U1601, U1701, U301, U401, U501, U601, U701, U801, U901: LEDboardcomparator, TO_SOT_Packages_SMD:SOT-23-5
- removed the U201 at (416.0, 77.3)
- added D201: LED, LEDs:LED_1206, F.Cu at (53.3, 169.1)
- added D201: LED, LEDs:LED_1206, F.Cu at (48.7, 55.2)
- added D201: LED, LEDs:LED_1206, F.Cu at (76.7, 54.0)
- added D201: LED, LEDs:LED_1206, F.Cu at (160.2, 158.8)
- added D201: LED, LEDs:LED_1206, F.Cu at (100.8, 54.0)
- added D201: LED, LEDs:LED_1206, F.Cu at (52.7, 94.8)
- added D201: LED, LEDs:LED_1206, F.Cu at (51.4, 66.8)
- added D201: LED, LEDs:LED_1206, F.Cu at (52.7, 118.9)
- added D201: LED, LEDs:LED_1206, F.Cu at (135.4, 151.8)
- added D201: LED, LEDs:LED_1206, F.Cu at (107.5, 153.0)
- added D201: LED, LEDs:LED_1206, F.Cu at (55.4, 154.3)
- added D201: LED, LEDs:LED_1206, F.Cu at (83.3, 153.0)
- added D201: LED, LEDs:LED_1206, F.Cu at (144.1, 128.8)
- added D201: LED, LEDs:LED_1206, F.Cu at (145.4, 156.7)
- added D201: LED, LEDs:LED_1206, F.Cu at (144.1, 104.6)
- added D201: LED, LEDs:LED_1206, F.Cu at (142.9, 76.7)
- added P110: CONN_01X04, hyperCustom:CONN_PHOENIX_1844236_4PIN_1, F.Cu at (129.8, 193.9)
- added R201: R, Resistors_SMD:R_1206_HandSoldering, F.Cu at (137.1, 164.5)
- added R201: R, Resistors_SMD:R_1206_HandSoldering, F.Cu at (75.0, 41.3)
- added R201: R, Resistors_SMD:R_1206_HandSoldering, F.Cu at (127.1, 40.0)
- added R201: R, Resistors_SMD:R_1206_HandSoldering, F.Cu at (99.2, 41.3)
- added R201: R, Resistors_SMD:R_1206_HandSoldering, F.Cu at (40.0, 96.4)
- added R201: R, Resistors_SMD:R_1206_HandSoldering, F.Cu at (38.7, 68.5)
- added R201: R, Resistors_SMD:R_1206_HandSoldering, F.Cu at (40.0, 120.6)
- added R201: R, Resistors_SMD:R_1206_HandSoldering, F.Cu at (109.1, 165.7)
- added R201: R, Resistors_SMD:R_1206_HandSoldering, F.Cu at (57.1, 167.0)
- added R201: R, Resistors_SMD:R_1206_HandSoldering, F.Cu at (85.0, 165.7)
- added R201: R, Resistors_SMD:R_1206_HandSoldering, F.Cu at (156.8, 127.1)
- added R201: R, Resistors_SMD:R_1206_HandSoldering, F.Cu at (158.1, 155.0)
- added R201: R, Resistors_SMD:R_1206_HandSoldering, F.Cu at (156.8, 103.0)
- added R201: R, Resistors_SMD:R_1206_HandSoldering, F.Cu at (155.6, 75.0)
- added R201: R, Resistors_SMD:R_1206_HandSoldering, F.Cu at (47.1, 42.5)
- added R202: R, Resistors_SMD:R_1206_HandSoldering, F.Cu at (137.3, 177.2)
- added R202: R, Resistors_SMD:R_1206_HandSoldering, F.Cu at (74.8, 28.6)
- added R202: R, Resistors_SMD:R_1206_HandSoldering, F.Cu at (126.9, 27.3)
- added R202: R, Resistors_SMD:R_1206_HandSoldering, F.Cu at (99.0, 28.6)
- added R202: R, Resistors_SMD:R_1206_HandSoldering, F.Cu at (27.3, 96.6)
- added R202: R, Resistors_SMD:R_1206_HandSoldering, F.Cu at (26.0, 68.7)
- added R202: R, Resistors_SMD:R_1206_HandSoldering, F.Cu at (27.3, 120.7)
- added R202: R, Resistors_SMD:R_1206_HandSoldering, F.Cu at (109.3, 178.4)
- added R202: R, Resistors_SMD:R_1206_HandSoldering, F.Cu at (57.2, 179.7)
- added R202: R, Resistors_SMD:R_1206_HandSoldering, F.Cu at (85.2, 178.4)
- added R202: R, Resistors_SMD:R_1206_HandSoldering, F.Cu at (169.5, 126.9)
- added R202: R, Resistors_SMD:R_1206_HandSoldering, F.Cu at (170.8, 154.8)
- added R202: R, Resistors_SMD:R_1206_HandSoldering, F.Cu at (169.5, 102.8)
- added R202: R, Resistors_SMD:R_1206_HandSoldering, F.Cu at (168.3, 74.8)
- added R202: R, Resistors_SMD:R_1206_HandSoldering, F.Cu at (46.9, 29.8)
- added R203: R, Resistors_SMD:R_1206_HandSoldering, F.Cu at (127.1, 177.2)
- added R203: R, Resistors_SMD:R_1206_HandSoldering, F.Cu at (109.1, 28.6)
- added R203: R, Resistors_SMD:R_1206_HandSoldering, F.Cu at (82.5, 28.6)
- added R203: R, Resistors_SMD:R_1206_HandSoldering, F.Cu at (27.3, 113.1)
- added R203: R, Resistors_SMD:R_1206_HandSoldering, F.Cu at (27.3, 86.5)
- added R203: R, Resistors_SMD:R_1206_HandSoldering, F.Cu at (28.6, 138.5)
- added R203: R, Resistors_SMD:R_1206_HandSoldering, F.Cu at (75.0, 178.4)
- added R203: R, Resistors_SMD:R_1206_HandSoldering, F.Cu at (101.7, 178.4)
- added R203: R, Resistors_SMD:R_1206_HandSoldering, F.Cu at (169.5, 110.4)
- added R203: R, Resistors_SMD:R_1206_HandSoldering, F.Cu at (169.5, 137.1)
- added R203: R, Resistors_SMD:R_1206_HandSoldering, F.Cu at (168.3, 85.0)
- added R203: R, Resistors_SMD:R_1206_HandSoldering, F.Cu at (167.0, 57.1)
- added R203: R, Resistors_SMD:R_1206_HandSoldering, F.Cu at (29.1, 31.1)
- added R203: R, Resistors_SMD:R_1206_HandSoldering, F.Cu at (57.1, 29.8)
- added R204: R, Resistors_SMD:R_1206_HandSoldering, F.Cu at (144.9, 177.2)
- added R204: R, Resistors_SMD:R_1206_HandSoldering, F.Cu at (67.2, 28.6)
- added R204: R, Resistors_SMD:R_1206_HandSoldering, F.Cu at (119.3, 27.3)
- added R204: R, Resistors_SMD:R_1206_HandSoldering, F.Cu at (91.3, 28.6)
- added R204: R, Resistors_SMD:R_1206_HandSoldering, F.Cu at (27.3, 104.2)
- added R204: R, Resistors_SMD:R_1206_HandSoldering, F.Cu at (26.0, 76.3)
- added R204: R, Resistors_SMD:R_1206_HandSoldering, F.Cu at (27.3, 128.4)
- added R204: R, Resistors_SMD:R_1206_HandSoldering, F.Cu at (116.9, 178.4)
- added R204: R, Resistors_SMD:R_1206_HandSoldering, F.Cu at (64.9, 179.7)
- added R204: R, Resistors_SMD:R_1206_HandSoldering, F.Cu at (92.8, 178.4)
- added R204: R, Resistors_SMD:R_1206_HandSoldering, F.Cu at (169.5, 119.3)
- added R204: R, Resistors_SMD:R_1206_HandSoldering, F.Cu at (170.8, 147.2)
- added R204: R, Resistors_SMD:R_1206_HandSoldering, F.Cu at (169.5, 95.2)
- added R204: R, Resistors_SMD:R_1206_HandSoldering, F.Cu at (168.3, 67.2)
- added R204: R, Resistors_SMD:R_1206_HandSoldering, F.Cu at (39.3, 29.8)
- added R205: R, Resistors_SMD:R_1206_HandSoldering, F.Cu at (150.5, 173.4)
- added R205: R, Resistors_SMD:R_1206_HandSoldering, F.Cu at (61.6, 32.4)
- added R205: R, Resistors_SMD:R_1206_HandSoldering, F.Cu at (113.7, 31.1)
- added R205: R, Resistors_SMD:R_1206_HandSoldering, F.Cu at (85.7, 32.4)
- added R205: R, Resistors_SMD:R_1206_HandSoldering, F.Cu at (31.1, 109.9)
- added R205: R, Resistors_SMD:R_1206_HandSoldering, F.Cu at (29.8, 81.9)
- added R205: R, Resistors_SMD:R_1206_HandSoldering, F.Cu at (31.1, 134.0)
- added R205: R, Resistors_SMD:R_1206_HandSoldering, F.Cu at (122.6, 174.6)
- added R205: R, Resistors_SMD:R_1206_HandSoldering, F.Cu at (70.5, 175.9)
- added R205: R, Resistors_SMD:R_1206_HandSoldering, F.Cu at (98.4, 174.6)
- added R205: R, Resistors_SMD:R_1206_HandSoldering, F.Cu at (165.7, 113.7)
- added R205: R, Resistors_SMD:R_1206_HandSoldering, F.Cu at (167.0, 141.6)
- added R205: R, Resistors_SMD:R_1206_HandSoldering, F.Cu at (165.7, 89.5)
- added R205: R, Resistors_SMD:R_1206_HandSoldering, F.Cu at (164.5, 61.6)
- added R205: R, Resistors_SMD:R_1206_HandSoldering, F.Cu at (33.7, 33.7)
- added R206: R, Resistors_SMD:R_1206_HandSoldering, F.Cu at (136.5, 170.8)
- added R206: R, Resistors_SMD:R_1206_HandSoldering, F.Cu at (75.6, 34.9)
- added R206: R, Resistors_SMD:R_1206_HandSoldering, F.Cu at (127.6, 33.7)
- added R206: R, Resistors_SMD:R_1206_HandSoldering, F.Cu at (99.7, 34.9)
- added R206: R, Resistors_SMD:R_1206_HandSoldering, F.Cu at (33.7, 95.9)
- added R206: R, Resistors_SMD:R_1206_HandSoldering, F.Cu at (32.4, 67.9)
- added R206: R, Resistors_SMD:R_1206_HandSoldering, F.Cu at (33.7, 120.0)
- added R206: R, Resistors_SMD:R_1206_HandSoldering, F.Cu at (108.6, 172.1)
- added R206: R, Resistors_SMD:R_1206_HandSoldering, F.Cu at (56.5, 173.4)
- added R206: R, Resistors_SMD:R_1206_HandSoldering, F.Cu at (84.5, 172.1)
- added R206: R, Resistors_SMD:R_1206_HandSoldering, F.Cu at (163.2, 127.6)
- added R206: R, Resistors_SMD:R_1206_HandSoldering, F.Cu at (164.5, 155.6)
- added R206: R, Resistors_SMD:R_1206_HandSoldering, F.Cu at (163.2, 103.5)
- added R206: R, Resistors_SMD:R_1206_HandSoldering, F.Cu at (161.9, 75.6)
- added R206: R, Resistors_SMD:R_1206_HandSoldering, F.Cu at (47.6, 36.2)
- added R207: R, Resistors_SMD:R_1206_HandSoldering, F.Cu at (142.3, 173.4)
- added R207: R, Resistors_SMD:R_1206_HandSoldering, F.Cu at (69.8, 32.4)
- added R207: R, Resistors_SMD:R_1206_HandSoldering, F.Cu at (121.8, 31.1)
- added R207: R, Resistors_SMD:R_1206_HandSoldering, F.Cu at (93.9, 32.4)
- added R207: R, Resistors_SMD:R_1206_HandSoldering, F.Cu at (31.1, 101.7)
- added R207: R, Resistors_SMD:R_1206_HandSoldering, F.Cu at (29.8, 73.8)
- added R207: R, Resistors_SMD:R_1206_HandSoldering, F.Cu at (31.1, 125.8)
- added R207: R, Resistors_SMD:R_1206_HandSoldering, F.Cu at (114.4, 174.6)
- added R207: R, Resistors_SMD:R_1206_HandSoldering, F.Cu at (62.3, 175.9)
- added R207: R, Resistors_SMD:R_1206_HandSoldering, F.Cu at (90.3, 174.6)
- added R207: R, Resistors_SMD:R_1206_HandSoldering, F.Cu at (165.7, 121.8)
- added R207: R, Resistors_SMD:R_1206_HandSoldering, F.Cu at (167.0, 149.8)
- added R207: R, Resistors_SMD:R_1206_HandSoldering, F.Cu at (165.7, 97.7)
- added R207: R, Resistors_SMD:R_1206_HandSoldering, F.Cu at (164.5, 69.8)
- added R207: R, Resistors_SMD:R_1206_HandSoldering, F.Cu at (41.8, 33.7)
- added R208: R, Resistors_SMD:R_1206_HandSoldering, F.Cu at (150.5, 166.5)
- added R208: R, Resistors_SMD:R_1206_HandSoldering, F.Cu at (61.6, 39.3)
- added R208: R, Resistors_SMD:R_1206_HandSoldering, F.Cu at (113.7, 38.0)
- added R208: R, Resistors_SMD:R_1206_HandSoldering, F.Cu at (85.7, 39.3)
- added R208: R, Resistors_SMD:R_1206_HandSoldering, F.Cu at (38.0, 109.9)
- added R208: R, Resistors_SMD:R_1206_HandSoldering, F.Cu at (36.7, 81.9)
- added R208: R, Resistors_SMD:R_1206_HandSoldering, F.Cu at (38.0, 134.0)
- added R208: R, Resistors_SMD:R_1206_HandSoldering, F.Cu at (122.6, 167.7)
- added R208: R, Resistors_SMD:R_1206_HandSoldering, F.Cu at (70.5, 169.0)
- added R208: R, Resistors_SMD:R_1206_HandSoldering, F.Cu at (98.4, 167.7)
- added R208: R, Resistors_SMD:R_1206_HandSoldering, F.Cu at (158.8, 113.7)
- added R208: R, Resistors_SMD:R_1206_HandSoldering, F.Cu at (160.1, 141.6)
- added R208: R, Resistors_SMD:R_1206_HandSoldering, F.Cu at (158.8, 89.5)
- added R208: R, Resistors_SMD:R_1206_HandSoldering, F.Cu at (157.6, 61.6)
- added R208: R, Resistors_SMD:R_1206_HandSoldering, F.Cu at (33.7, 40.5)
- added R209: R, Resistors_SMD:R_1206_HandSoldering, F.Cu at (151.2, 178.4)
- added R209: R, Resistors_SMD:R_1206_HandSoldering, F.Cu at (60.9, 27.3)
- added R209: R, Resistors_SMD:R_1206_HandSoldering, F.Cu at (112.9, 26.0)
- added R209: R, Resistors_SMD:R_1206_HandSoldering, F.Cu at (85.0, 27.3)
- added R209: R, Resistors_SMD:R_1206_HandSoldering, F.Cu at (26.0, 110.6)
- added R209: R, Resistors_SMD:R_1206_HandSoldering, F.Cu at (24.8, 82.6)
- added R209: R, Resistors_SMD:R_1206_HandSoldering, F.Cu at (26.0, 134.7)
- added R209: R, Resistors_SMD:R_1206_HandSoldering, F.Cu at (123.3, 179.7)
- added R209: R, Resistors_SMD:R_1206_HandSoldering, F.Cu at (71.2, 181.0)
- added R209: R, Resistors_SMD:R_1206_HandSoldering, F.Cu at (99.2, 179.7)
- added R209: R, Resistors_SMD:R_1206_HandSoldering, F.Cu at (170.8, 112.9)
- added R209: R, Resistors_SMD:R_1206_HandSoldering, F.Cu at (172.1, 140.9)
- added R209: R, Resistors_SMD:R_1206_HandSoldering, F.Cu at (170.8, 88.8)
- added R209: R, Resistors_SMD:R_1206_HandSoldering, F.Cu at (169.5, 60.9)
- added R209: R, Resistors_SMD:R_1206_HandSoldering, F.Cu at (32.9, 28.6)
- added R210: R, Resistors_SMD:R_1206_HandSoldering, F.Cu at (142.9, 168.3)
- added R210: R, Resistors_SMD:R_1206_HandSoldering, F.Cu at (69.2, 37.5)
- added R210: R, Resistors_SMD:R_1206_HandSoldering, F.Cu at (121.3, 36.2)
- added R210: R, Resistors_SMD:R_1206_HandSoldering, F.Cu at (93.3, 37.5)
- added R210: R, Resistors_SMD:R_1206_HandSoldering, F.Cu at (36.2, 102.2)
- added R210: R, Resistors_SMD:R_1206_HandSoldering, F.Cu at (34.9, 74.3)
- added R210: R, Resistors_SMD:R_1206_HandSoldering, F.Cu at (36.2, 126.4)
- added R210: R, Resistors_SMD:R_1206_HandSoldering, F.Cu at (114.9, 169.5)
- added R210: R, Resistors_SMD:R_1206_HandSoldering, F.Cu at (62.9, 170.8)
- added R210: R, Resistors_SMD:R_1206_HandSoldering, F.Cu at (90.8, 169.5)
- added R210: R, Resistors_SMD:R_1206_HandSoldering, F.Cu at (160.7, 121.3)
- added R210: R, Resistors_SMD:R_1206_HandSoldering, F.Cu at (161.9, 149.2)
- added R210: R, Resistors_SMD:R_1206_HandSoldering, F.Cu at (160.7, 97.2)
- added R210: R, Resistors_SMD:R_1206_HandSoldering, F.Cu at (159.4, 69.2)
- added R210: R, Resistors_SMD:R_1206_HandSoldering, F.Cu at (41.3, 38.7)
- added R211: R, Resistors_SMD:R_1206_HandSoldering, F.Cu at (145.4, 163.7)
- added R211: R, Resistors_SMD:R_1206_HandSoldering, F.Cu at (66.7, 42.0)
- added R211: R, Resistors_SMD:R_1206_HandSoldering, F.Cu at (118.7, 40.7)
- added R211: R, Resistors_SMD:R_1206_HandSoldering, F.Cu at (90.8, 42.0)
- added R211: R, Resistors_SMD:R_1206_HandSoldering, F.Cu at (40.7, 104.8)
- added R211: R, Resistors_SMD:R_1206_HandSoldering, F.Cu at (39.5, 76.8)
- added R211: R, Resistors_SMD:R_1206_HandSoldering, F.Cu at (40.7, 128.9)
- added R211: R, Resistors_SMD:R_1206_HandSoldering, F.Cu at (117.5, 165.0)
- added R211: R, Resistors_SMD:R_1206_HandSoldering, F.Cu at (65.4, 166.3)
- added R211: R, Resistors_SMD:R_1206_HandSoldering, F.Cu at (93.3, 165.0)
- added R211: R, Resistors_SMD:R_1206_HandSoldering, F.Cu at (156.1, 118.7)
- added R211: R, Resistors_SMD:R_1206_HandSoldering, F.Cu at (157.4, 146.7)
- added R211: R, Resistors_SMD:R_1206_HandSoldering, F.Cu at (156.1, 94.6)
- added R211: R, Resistors_SMD:R_1206_HandSoldering, F.Cu at (154.8, 66.7)
- added R211: R, Resistors_SMD:R_1206_HandSoldering, F.Cu at (38.7, 43.3)
- added R212: R, Resistors_SMD:R_1206_HandSoldering, F.Cu at (148.0, 169.0)
- added R212: R, Resistors_SMD:R_1206_HandSoldering, F.Cu at (64.1, 36.7)
- added R212: R, Resistors_SMD:R_1206_HandSoldering, F.Cu at (116.2, 35.5)
- added R212: R, Resistors_SMD:R_1206_HandSoldering, F.Cu at (88.3, 36.7)
- added R212: R, Resistors_SMD:R_1206_HandSoldering, F.Cu at (35.5, 107.3)
- added R212: R, Resistors_SMD:R_1206_HandSoldering, F.Cu at (34.2, 79.4)
- added R212: R, Resistors_SMD:R_1206_HandSoldering, F.Cu at (35.5, 131.4)
- added R212: R, Resistors_SMD:R_1206_HandSoldering, F.Cu at (120.0, 170.3)
- added R212: R, Resistors_SMD:R_1206_HandSoldering, F.Cu at (67.9, 171.5)
- added R212: R, Resistors_SMD:R_1206_HandSoldering, F.Cu at (95.9, 170.3)
- added R212: R, Resistors_SMD:R_1206_HandSoldering, F.Cu at (161.4, 116.2)
- added R212: R, Resistors_SMD:R_1206_HandSoldering, F.Cu at (162.7, 144.1)
- added R212: R, Resistors_SMD:R_1206_HandSoldering, F.Cu at (161.4, 92.1)
- added R212: R, Resistors_SMD:R_1206_HandSoldering, F.Cu at (160.1, 64.1)
- added R212: R, Resistors_SMD:R_1206_HandSoldering, F.Cu at (36.2, 38.0)
- added R213: R, Resistors_SMD:R_1206_HandSoldering, F.Cu at (137.8, 159.9)
- added R213: R, Resistors_SMD:R_1206_HandSoldering, F.Cu at (74.3, 45.8)
- added R213: R, Resistors_SMD:R_1206_HandSoldering, F.Cu at (126.4, 44.5)
- added R213: R, Resistors_SMD:R_1206_HandSoldering, F.Cu at (98.4, 45.8)
- added R213: R, Resistors_SMD:R_1206_HandSoldering, F.Cu at (44.5, 97.2)
- added R213: R, Resistors_SMD:R_1206_HandSoldering, F.Cu at (43.3, 69.2)
- added R213: R, Resistors_SMD:R_1206_HandSoldering, F.Cu at (44.5, 121.3)
- added R213: R, Resistors_SMD:R_1206_HandSoldering, F.Cu at (109.9, 161.2)
- added R213: R, Resistors_SMD:R_1206_HandSoldering, F.Cu at (57.8, 162.5)
- added R213: R, Resistors_SMD:R_1206_HandSoldering, F.Cu at (85.7, 161.2)
- added R213: R, Resistors_SMD:R_1206_HandSoldering, F.Cu at (152.3, 126.4)
- added R213: R, Resistors_SMD:R_1206_HandSoldering, F.Cu at (153.6, 154.3)
- added R213: R, Resistors_SMD:R_1206_HandSoldering, F.Cu at (152.3, 102.2)
- added R213: R, Resistors_SMD:R_1206_HandSoldering, F.Cu at (151.0, 74.3)
- added R213: R, Resistors_SMD:R_1206_HandSoldering, F.Cu at (46.4, 47.1)
- added U201: LEDboardcomparator, TO_SOT_Packages_SMD:SOT-23-5, F.Cu at (141.3, 159.3)
- added U201: LEDboardcomparator, TO_SOT_Packages_SMD:SOT-23-5, F.Cu at (70.8, 46.4)
- added U201: LEDboardcomparator, TO_SOT_Packages_SMD:SOT-23-5, F.Cu at (122.9, 45.1)
- added U201: LEDboardcomparator, TO_SOT_Packages_SMD:SOT-23-5, F.Cu at (94.9, 46.4)
- added U201: LEDboardcomparator, TO_SOT_Packages_SMD:SOT-23-5, F.Cu at (45.1, 100.6)
- added U201: LEDboardcomparator, TO_SOT_Packages_SMD:SOT-23-5, F.Cu at (43.9, 72.7)
- added U201: LEDboardcomparator, TO_SOT_Packages_SMD:SOT-23-5, F.Cu at (45.1, 124.8)
- added U201: LEDboardcomparator, TO_SOT_Packages_SMD:SOT-23-5, F.Cu at (113.3, 160.6)
- added U201: LEDboardcomparator, TO_SOT_Packages_SMD:SOT-23-5, F.Cu at (61.3, 161.9)
- added U201: LEDboardcomparator, TO_SOT_Packages_SMD:SOT-23-5, F.Cu at (89.2, 160.6)
- added U201: LEDboardcomparator, TO_SOT_Packages_SMD:SOT-23-5, F.Cu at (151.7, 122.9)
- added U201: LEDboardcomparator, TO_SOT_Packages_SMD:SOT-23-5, F.Cu at (153.0, 150.8)
- added U201: LEDboardcomparator, TO_SOT_Packages_SMD:SOT-23-5, F.Cu at (151.7, 98.7)
- added U201: LEDboardcomparator, TO_SOT_Packages_SMD:SOT-23-5, F.Cu at (150.4, 70.8)
- added U201: LEDboardcomparator, TO_SOT_Packages_SMD:SOT-23-5, F.Cu at (42.9, 47.7)
- moved P102 279.9 mm to (104.4, 194.5)
- moved P106 279.9 mm to (77.1, 194.7)
- moved P107 279.9 mm to (60.7, 192.8)
- moved P103 279.9 mm to (90.8, 194.7)
- moved P109 261.9 mm to (17.7, 133.2), turned to 90 degrees
- moved P101 155.4 mm to (184.1, 16.9), turned to 90 degrees
- moved P104 143.9 mm to (184.1, 30.6), turned to 90 degrees
- moved P105 134.3 mm to (184.1, 44.2), turned to 90 degrees
- moved R203 131.0 mm to (29.8, 166.5), turned to 90 degrees
- moved R209 130.0 mm to (27.3, 162.7), turned to 90 degrees
- moved P108 124.5 mm to (183.8, 65.0), turned to 90 degrees
- moved R205 124.0 mm to (32.4, 161.9), turned to 180 degrees
- moved R204 123.0 mm to (28.6, 156.3), turned to 90 degrees
- moved R212 117.0 mm to (36.7, 159.4), turned to 180 degrees
- moved R208 116.9 mm to (39.3, 161.9), turned to 180 degrees
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Connections:
- P109 pad 3: /Vcc_Bat -> /PowerBoard
Routing:
- net Net-(R205-Pad1): track 49.6 -> 794.2 mm
- net Net-(R208-Pad1): track 40.8 -> 653.2 mm
- net / Indicator Circuit for <battery charge on>/Vref: track 29.4 -> 469.7 mm
- net GND: track 24.6 -> 393.9 mm
- net / Indicator Circuit for <battery charge on>/Vout: track 16.4 -> 261.8 mm
- net / Indicator Circuit for <battery charge on>/Vin_div: track 15.6 -> 250.3 mm
- net (no net): track 101.9 -> 0.00 mm
- net VCC: track 6.52 -> 104.3 mm
- net Net-(R1608-Pad1): track 79.9 -> 0.00 mm
- net / Indicator Circuit for <12>/Vin_div: track 1.10 -> 0.00 mm
Other:
- board size 358.6 x 213 mm -> 196 x 196.5 mm
