File: LEDBoard/powerswitch.sch (KiCad schematic (older format))
At the start: 9 parts

Commit message: made major changed to the led board mostly dealing with schematic
Parts:
- gave numbers to parts that had none: 9
Connections:
- net 5VIn is gone; now on net VCC: R1803.1
Changed lines of the file:
@@
 EESchema Schematic File Version 2
+LIBS:LEDBoard-rescue
 LIBS:power
 LIBS:device
@@
 $EndDescr
 $Comp
-L LMx93 U?
+L LMx93 U1801
 U 1 1 584C918B
 P 5550 3450
-F 0 "U?" H 5550 3150 60  0000 C CNN
+F 0 "U1801" H 5550 3150 60  0000 C CNN
 F 1 "LMx93" H 5550 3700 60  0000 C CNN
 F 2 "" H 5450 3700 60  0001 C CNN
@@
 $EndComp
 $Comp
-L GND #PWR?
+L GND #PWR1804
 U 1 1 584C920E
 P 4750 3800
-F 0 "#PWR?" H 4750 3550 50  0001 C CNN
+F 0 "#PWR1804" H 4750 3550 50  0001 C CNN
 F 1 "GND" H 4750 3650 50  0000 C CNN
 F 2 "" H 4750 3800 50  0000 C CNN
@@
 $EndComp
 $Comp
-L R R?
+L R R1804
 U 1 1 584C92F0
 P 1850 5650
-F 0 "R?" V 1930 5650 50  0000 C CNN
+F 0 "R1804" V 1930 5650 50  0000 C CNN
 F 1 "400K" V 1850 5650 50  0000 C CNN
 F 2 "Resistors_SMD:R_1206_HandSoldering" V 1780 5650 50  0001 C CNN
@@
 $EndComp
 $Comp
-L 5VoltRegulator U?
+L 5VoltRegulator U1803
 U 1 1 584C9549
 P 8500 5000
-F 0 "U?" V 8800 5000 60  0000 C CNN
+F 0 "U1803" V 8800 5000 60  0000 C CNN
 F 1 "5VoltRegulator" V 8200 5000 60  0000 C CNN
 F 2 "" H 8450 5350 60  0001 C CNN
@@
 $EndComp
 $Comp
-L GND #PWR?
+L GND #PWR1811
 U 1 1 584C960B
 P 9450 5000
-F 0 "#PWR?" H 9450 4750 50  0001 C CNN
+F 0 "#PWR1811" H 9450 4750 50  0001 C CNN
 F 1 "GND" H 9450 4850 50  0000 C CNN
 F 2 "" H 9450 5000 50  0000 C CNN
@@
 $EndComp
 $Comp
-L GND #PWR?
+L GND #PWR1801
 U 1 1 584C976B
 P 1750 3300
-F 0 "#PWR?" H 1750 3050 50  0001 C CNN
+F 0 "#PWR1801" H 1750 3050 50  0001 C CNN
 F 1 "GND" H 1750 3150 50  0000 C CNN
 F 2 "" H 1750 3300 50  0000 C CNN
@@
 $EndComp
 $Comp
-L GND #PWR?
+L GND #PWR1803
 U 1 1 584C979B
 P 1850 6100
-F 0 "#PWR?" H 1850 5850 50  0001 C CNN
+F 0 "#PWR1803" H 1850 5850 50  0001 C CNN
 F 1 "GND" H 1850 5950 50  0000 C CNN
 F 2 "" H 1850 6100 50  0000 C CNN
@@
 	1    0    0    -1
 $EndComp
-Text HLabel 1850 4350 1    60   Output ~ 0
-5VIn
 Wire Wire Line
 	1850 4950 1850 5500
@@
 	8150 5150 7700 5150
 $Comp
-L R R?
+L R R1803
 U 1 1 584C9AFD
 P 1850 4800
-F 0 "R?" V 1930 4800 50  0000 C CNN
+F 0 "R1803" V 1930 4800 50  0000 C CNN
 F 1 "100K" V 1850 4800 50  0000 C CNN
 F 2 "Resistors_SMD:R_1206_HandSoldering" V 1780 4800 50  0001 C CNN
@@
 $EndComp
 $Comp
-L R R?
+L R R1802
 U 1 1 584C9BB1
 P 1750 2950
-F 0 "R?" V 1830 2950 50  0000 C CNN
+F 0 "R1802" V 1830 2950 50  0000 C CNN
 F 1 "100K" V 1750 2950 50  0000 C CNN
 F 2 "Resistors_SMD:R_1206_HandSoldering" V 1680 2950 50  0001 C CNN
@@
 $EndComp
 $Comp
-L R R?
+L R R1801
 U 1 1 584C9C00
 P 1750 2000
-F 0 "R?" V 1830 2000 50  0000 C CNN
+F 0 "R1801" V 1830 2000 50  0000 C CNN
 F 1 "600K" V 1750 2000 50  0000 C CNN
 F 2 "Resistors_SMD:R_1206_HandSoldering" V 1680 2000 50  0001 C CNN
@@
 $EndComp
 $Comp
-L 5VoltRegulator U?
+L 5VoltRegulator U1802
 U 1 1 584C9EE8
 P 8500 4050
-F 0 "U?" V 8800 4050 60  0000 C CNN
+F 0 "U1802" V 8800 4050 60  0000 C CNN
 F 1 "5VoltRegulator" V 8200 4050 60  0000 C CNN
 F 2 "" H 8450 4400 60  0001 C CNN
@@
 $EndComp
 $Comp
-L GND #PWR?
+L GND #PWR1810
 U 1 1 584C9EEE
 P 9450 4050
-F 0 "#PWR?" H 9450 3800 50  0001 C CNN
+F 0 "#PWR1810" H 9450 3800 50  0001 C CNN
 F 1 "GND" H 9450 3900 50  0000 C CNN
 F 2 "" H 9450 4050 50  0000 C CNN
@@
 Vref
 $Comp
-L VCC #PWR?
+L VCC #PWR1808
 U 1 1 584CA19A
 P 7700 4200
-F 0 "#PWR?" H 7700 4050 50  0001 C CNN
+F 0 "#PWR1808" H 7700 4050 50  0001 C CNN
 F 1 "VCC" H 7700 4350 50  0000 C CNN
 F 2 "" H 7700 4200 50  0000 C CNN
@@
 $EndComp
 $Comp
-L VCC #PWR?
+L VCC #PWR1809
 U 1 1 584CA9A7
 P 7700 5150
-F 0 "#PWR?" H 7700 5000 50  0001 C CNN
+F 0 "#PWR1809" H 7700 5000 50  0001 C CNN
 F 1 "VCC" H 7700 5300 50  0000 C CNN
 F 2 "" H 7700 5150 50  0000 C CNN
@@
 $EndComp
 $Comp
-L VCC #PWR?
+L VCC #PWR1805
 U 1 1 584CA9C9
 P 6000 3300
-F 0 "#PWR?" H 6000 3150 50  0001 C CNN
+F 0 "#PWR1805" H 6000 3150 50  0001 C CNN
 F 1 "VCC" H 6000 3450 50  0000 C CNN
 F 2 "" H 6000 3300 50  0000 C CNN
@@
 	7650 4900 7650 4850
 $Comp
-L C C?
+L C C1801
 U 1 1 584CAAA2
 P 7500 4850
-F 0 "C?" H 7525 4950 50  0000 L CNN
+F 0 "C1801" H 7525 4950 50  0000 L CNN
 F 1 "C" H 7525 4750 50  0000 L CNN
 F 2 "" H 7538 4700 50  0000 C CNN
@@
 $EndComp
 $Comp
-L C C?
+L C C1802
 U 1 1 584CAAF6
 P 8000 3950
-F 0 "C?" H 8025 4050 50  0000 L CNN
+F 0 "C1802" H 8025 4050 50  0000 L CNN
 F 1 "C" H 8025 3850 50  0000 L CNN
 F 2 "" H 8038 3800 50  0000 C CNN
@@
 	7200 3950 7850 3950
 $Comp
-L GND #PWR?
+L GND #PWR1807
 U 1 1 584CADC7
 P 7200 3950
-F 0 "#PWR?" H 7200 3700 50  0001 C CNN
+F 0 "#PWR1807" H 7200 3700 50  0001 C CNN
 F 1 "GND" H 7200 3800 50  0000 C CNN
 F 2 "" H 7200 3950 50  0000 C CNN
@@
 $EndComp
 $Comp
-L GND #PWR?
+L GND #PWR1806
 U 1 1 584CADF6
 P 7150 4850
-F 0 "#PWR?" H 7150 4600 50  0001 C CNN
+F 0 "#PWR1806" H 7150 4600 50  0001 C CNN
 F 1 "GND" H 7150 4700 50  0000 C CNN
 F 2 "" H 7150 4850 50  0000 C CNN
@@
 Wire Wire Line
 	7350 4850 7150 4850
+$Comp
+L VCC #PWR1802
+U 1 1 5851796A
+P 1850 4350
+F 0 "#PWR1802" H 1850 4200 50  0001 C CNN
+F 1 "VCC" H 1850 4500 50  0000 C CNN
+F 2 "" H 1850 4350 50  0000 C CNN
+F 3 "" H 1850 4350 50  0000 C CNN
+	1    1850 4350
+	1    0    0    -1
+$EndComp
 $EndSCHEMATC
