File: PusherProtectionBoard/PusherProtectionBoard.sch (KiCad schematic (older format))
At the start: 22 parts, among them J101 CONN_01X02, J102 CONN_01X04, J103 CONN_01X02, J104 CONN_01X02, J105 CONN_01X02, J106 CONN_01X02, J107 CONN_01X02, J108 CONN_01X02, J109 CONN_01X02, J110 CONN_01X02, J111 CONN_01X02, J112 CONN_01X02, J113 CONN_01X02, J114 MOUNTING_HOLE, J115 MOUNTING_HOLE, J116 MOUNTING_HOLE, J117 MOUNTING_HOLE, U101 LM2936HV

Commit message: Finalized silkscreen for Pusher Protection Board and compiled final Gerbers, pending results of DFM check.
Parts:
- C101: DigiKey PN (none) -> 311-2007-1-ND; Mfg. (none) -> Yageo; Mfg. PN (none) -> CC1206ZRY5V6BB106
- J102: DigiKey PN (none) -> 277-2419-ND; Mfg. (none) -> Phoenix; Mfg. PN (none) -> 1844236
- R102: DigiKey PN (none) -> 311-10KERCT-ND; Mfg. (none) -> Yageo; Mfg. PN (none) -> RC1206JR-0710KL
- U101: DigiKey PN (none) -> LM2936HVMAX-5.0/NOPBCT-ND; Mfg. (none) -> Texas Instruments; Mfg. PN (none) -> LM2936HVMAX-5.0/NOPB
Changed lines of the file:
@@
 F 2 "Resistors_SMD:R_1206_HandSoldering" V 2280 3650 30  0001 C CNN
 F 3 "" H 2350 3650 30  0000 C CNN
+F 4 "Yageo" V 2350 3650 60  0001 C CNN "Mfg."
+F 5 "RC1206JR-0710KL" V 2350 3650 60  0001 C CNN "Mfg. PN"
+F 6 "311-10KERCT-ND" V 2350 3650 60  0001 C CNN "DigiKey PN"
 	1    2350 3650
 	-1   0    0    1
@@
 F 2 "hyperCustom:LM2936HV_SOIC8" H 3100 1000 60  0001 C CNN
 F 3 "" H 3100 1000 60  0000 C CNN
+F 4 "Texas Instruments" H 3100 1000 60  0001 C CNN "Mfg."
+F 5 "LM2936HVMAX-5.0/NOPB" H 3100 1000 60  0001 C CNN "Mfg. PN"
+F 6 "LM2936HVMAX-5.0/NOPBCT-ND" H 3100 1000 60  0001 C CNN "DigiKey PN"
 	1    3100 1000
 	1    0    0    -1
@@
 F 2 "hyperCustom:CONN_PHOENIX_1844236_4PIN_1" H 900 5200 60  0001 C CNN
 F 3 "" H 900 5200 60  0000 C CNN
+F 4 "Phoenix" H 900 5200 60  0001 C CNN "Mfg."
+F 5 "1844236" H 900 5200 60  0001 C CNN "Mfg. PN"
+F 6 "277-2419-ND" H 900 5200 60  0001 C CNN "DigiKey PN"
 	1    900  5200
 	-1   0    0    -1
@@
 F 2 "Capacitors_SMD:C_1206_HandSoldering" H 3988 1100 30  0001 C CNN
 F 3 "" H 3950 1250 60  0000 C CNN
+F 4 "Yageo" H 3950 1250 60  0001 C CNN "Mfg."
+F 5 "CC1206ZRY5V6BB106" H 3950 1250 60  0001 C CNN "Mfg. PN"
+F 6 "311-2007-1-ND" H 3950 1250 60  0001 C CNN "DigiKey PN"
 	1    3950 1250
 	1    0    0    -1

Commit message: Corrected problem with Pusher Protection Board. Updated both schematic and layout and regenerated and zipped Gerbers. Ready for fab.
Parts:
- R102: DigiKey PN 311-10KERCT-ND -> 311-10.0KFRCT-ND; Mfg. PN RC1206JR-0710KL -> RC1206FR-0710KL
Changed lines of the file:
@@
 F 3 "" H 2350 3650 30  0000 C CNN
 F 4 "Yageo" V 2350 3650 60  0001 C CNN "Mfg."
-F 5 "RC1206JR-0710KL" V 2350 3650 60  0001 C CNN "Mfg. PN"
-F 6 "311-10KERCT-ND" V 2350 3650 60  0001 C CNN "DigiKey PN"
+F 5 "RC1206FR-0710KL" V 2350 3650 60  0001 C CNN "Mfg. PN"
+F 6 "311-10.0KFRCT-ND" V 2350 3650 60  0001 C CNN "DigiKey PN"
 	1    2350 3650
 	-1   0    0    1
