File: Motherboard/optocouplesL.sch (KiCad schematic (older format))
At the start: 9 parts, among them U4201 MC74HC1G14, U4203 NC7WZ07, U4204 ACSL-6400, U4205 NC7WZ07, U4207 MC74HC1G14

Commit message: Full Motherboard Rev1 -- sent for fab
Parts:
- U4205: Digikey P/N (none) -> NC7WZ16P6XCT-ND
Connections:
- net +5V: no longer U4203.5 (VCC), U4205.5 (VCC)
- net 3.3V: now also U4203.5 (VCC), U4205.5 (VCC)
Changed lines of the file:
@@
 $Descr A4 11693 8268
 encoding utf-8
-Sheet 6 12
+Sheet 5 12
 Title ""
 Date ""
@@
 $EndDescr
 $Comp
-L GND #PWR504
+L GND #PWR066
 U 1 1 5867C4A6
 P 6400 4800
-AR Path="/5867159E/5867C4A6" Ref="#PWR504"  Part="1"
-AR Path="/586B16FC/5867C4A6" Ref="#PWR604"  Part="1"
+AR Path="/5867159E/5867C4A6" Ref="#PWR066"  Part="1"
+AR Path="/586B16FC/5867C4A6" Ref="#PWR071"  Part="1"
 AR Path="/586E13E6/5867C4A6" Ref="#PWR0192"  Part="1"
 AR Path="/586E13F1/5867C4A6" Ref="#PWR0197"  Part="1"
-F 0 "#PWR604" H 6400 4550 50  0001 C CNN
+F 0 "#PWR071" H 6400 4550 50  0001 C CNN
 F 1 "GND" H 6400 4650 50  0000 C CNN
 F 2 "" H 6400 4800 50  0000 C CNN
@@
 	1    0    0    -1
 $EndComp
-Text GLabel 2350 2450 1    60   Input ~ 0
-+5V
-$Comp
-L GND #PWR502
+$Comp
+L GND #PWR067
 U 1 1 585E2A2C
 P 2350 3400
-AR Path="/5867159E/585E2A2C" Ref="#PWR502"  Part="1"
-AR Path="/586B16FC/585E2A2C" Ref="#PWR602"  Part="1"
+AR Path="/5867159E/585E2A2C" Ref="#PWR067"  Part="1"
+AR Path="/586B16FC/585E2A2C" Ref="#PWR072"  Part="1"
 AR Path="/586E13E6/585E2A2C" Ref="#PWR0193"  Part="1"
 AR Path="/586E13F1/585E2A2C" Ref="#PWR0198"  Part="1"
-F 0 "#PWR602" H 2350 3150 50  0001 C CNN
+F 0 "#PWR072" H 2350 3150 50  0001 C CNN
 F 1 "GND" H 2350 3250 50  0000 C CNN
 F 2 "" H 2350 3400 50  0000 C CNN
@@
 F 2 "TO_SOT_Packages_SMD:SC-70-6_Handsoldering" H 3250 3300 60  0001 C CNN
 F 3 "" H 3250 3300 60  0001 C CNN
+F 4 "NC7WZ16P6XCT-ND" H 2150 2900 60  0001 C CNN "Digikey P/N"
 	1    2150 2900
 	1    0    0    -1
@@
 	0    -1   -1   0
 $EndComp
-Text GLabel 2350 3800 1    60   Input ~ 0
-+5V
-$Comp
-L GND #PWR503
+$Comp
+L GND #PWR068
 U 1 1 5867D2DA
 P 2350 4750
-AR Path="/5867159E/5867D2DA" Ref="#PWR503"  Part="1"
-AR Path="/586B16FC/5867D2DA" Ref="#PWR603"  Part="1"
+AR Path="/5867159E/5867D2DA" Ref="#PWR068"  Part="1"
+AR Path="/586B16FC/5867D2DA" Ref="#PWR073"  Part="1"
 AR Path="/586E13E6/5867D2DA" Ref="#PWR0194"  Part="1"
 AR Path="/586E13F1/5867D2DA" Ref="#PWR0199"  Part="1"
-F 0 "#PWR603" H 2350 4500 50  0001 C CNN
+F 0 "#PWR073" H 2350 4500 50  0001 C CNN
 F 1 "GND" H 2350 4600 50  0000 C CNN
 F 2 "" H 2350 4750 50  0000 C CNN
@@
 $EndComp
 $Comp
-L GND #PWR505
+L GND #PWR069
 U 1 1 585E2A32
 P 3400 7600
-AR Path="/5867159E/585E2A32" Ref="#PWR505"  Part="1"
-AR Path="/586B16FC/585E2A32" Ref="#PWR605"  Part="1"
+AR Path="/5867159E/585E2A32" Ref="#PWR069"  Part="1"
+AR Path="/586B16FC/585E2A32" Ref="#PWR074"  Part="1"
 AR Path="/586E13E6/585E2A32" Ref="#PWR0195"  Part="1"
 AR Path="/586E13F1/585E2A32" Ref="#PWR0200"  Part="1"
-F 0 "#PWR605" H 3400 7350 50  0001 C CNN
+F 0 "#PWR074" H 3400 7350 50  0001 C CNN
 F 1 "GND" H 3400 7450 50  0000 C CNN
 F 2 "" H 3400 7600 50  0000 C CNN
@@
 $EndComp
 $Comp
-L GND #PWR501
+L GND #PWR070
 U 1 1 585E2A34
 P 4500 1600
-AR Path="/5867159E/585E2A34" Ref="#PWR501"  Part="1"
-AR Path="/586B16FC/585E2A34" Ref="#PWR601"  Part="1"
+AR Path="/5867159E/585E2A34" Ref="#PWR070"  Part="1"
+AR Path="/586B16FC/585E2A34" Ref="#PWR075"  Part="1"
 AR Path="/586E13E6/585E2A34" Ref="#PWR0196"  Part="1"
 AR Path="/586E13F1/585E2A34" Ref="#PWR0201"  Part="1"
-F 0 "#PWR601" H 4500 1350 50  0001 C CNN
+F 0 "#PWR075" H 4500 1350 50  0001 C CNN
 F 1 "GND" H 4500 1450 50  0000 C CNN
 F 2 "" H 4500 1600 50  0000 C CNN
@@
 	1    0    0    -1
 $EndComp
-Text GLabel 4500 800  1    60   Input ~ 0
-3.3V
 Text HLabel 3950 1200 0    60   Input ~ 0
 SYS_RESET
@@
 Text HLabel 7000 4150 2    60   Input ~ 0
 Vout_3
-Text GLabel 3400 6800 1    60   Input ~ 0
-3.3V
 Wire Wire Line
 	6400 4600 6400 4800
@@
 Wire Wire Line
 	3600 3700 6000 3700
+Wire Wire Line
+	4500 800  4650 800
+Wire Wire Line
+	3400 6800 3400 6700
+Text GLabel 4650 800  2    60   Input ~ 0
+3.3V
+Text GLabel 3400 6700 2    60   Input ~ 0
+3.3V
+Text GLabel 2500 2450 2    60   Input ~ 0
+3.3V
+Wire Wire Line
+	2350 2450 2500 2450
+Text GLabel 2500 3800 2    60   Input ~ 0
+3.3V
+Wire Wire Line
+	2350 3800 2500 3800
 $EndSCHEMATC
