File: Motherboard/file5919FB3B.sch (KiCad schematic (older format))
At the start: 19 parts

Commit message: Moving along
Parts:
- removed R?: 22, symbol R
- added R302: 22, Resistors_SMD:R_0805_HandSoldering, symbol R
- P301: renamed from P?; footprint (none) -> Connect:USB_Mini-B; Digikey P/N (none) -> 609-4700-1-ND; MFR P/N (none) -> 10033526-N3212LF
- R301: renamed from R?; footprint (none) -> Resistors_SMD:R_0805_HandSoldering; Digikey P/N (none) -> 311-22ARCT-ND; MFR P/N (none) -> RC0805JR-0722RL
- U301: renamed from U?; footprint SSOP-28 -> Housings_SSOP:SSOP-28_5.3x10.2mm_Pitch0.65mm
- gave numbers to parts that had none: 15
Connections:
- net +5V is gone; now on net USB_VCC: R304.1, R305.1
- net at U301.16 (USBD-): now also R302.1
- net at P301.2 (D-), VR302.1: now also R302.2
Other:
- note added: "FT232 should only be active when USB is inserted. Sole purpose is plan B programming of the ATMEGA.\nCurrent from BBB should be more than sufficient if BBB RX/TX to the ATMEGA fails.\nMay need to increase varistor and fuse values if BBB-> USB is necessary."
- note added: "YELLOW\n"
- note removed: "FT232 should only be active when USB is inserted. Sole purpose is plan B programming of the ATMEGA.\nCurrent from BBB should be more than sufficient if BBB RX/TX to the ATMEGA fails.\nMay need to increase varistor and fuse values if on-Pod USB is necessary."
Changed lines of the file:
@@
 $Descr A4 11693 8268
 encoding utf-8
-Sheet 3 15
+Sheet 3 16
 Title "Motherboard"
 Date ""
@@
 $EndDescr
 $Comp
-L FT232RL U?
+L FT232RL U301
 U 1 1 591946CE
 P 5700 2900
-F 0 "U?" H 5050 3800 50  0000 L CNN
+F 0 "U301" H 5050 3800 50  0000 L CNN
 F 1 "FT232RL" H 6100 3800 50  0000 L CNN
-F 2 "SSOP-28" H 5700 2900 50  0000 C CNN
+F 2 "Housings_SSOP:SSOP-28_5.3x10.2mm_Pitch0.65mm" H 5700 2900 50  0001 C CNN
 F 3 "" H 5700 2900 50  0000 C CNN
 F 4 "768-1007-1-ND" H 5700 2900 60  0001 C CNN "Digikey P/N"
@@
 USB MICRO\n
 $Comp
-L USB_OTG P?
+L USB_OTG P301
 U 1 1 591A98C8
 P 800 2750
-F 0 "P?" H 1125 2625 50  0000 C CNN
+F 0 "P301" H 1125 2625 50  0000 C CNN
 F 1 "USB_OTG" H 800 2950 50  0000 C CNN
-F 2 "" V 750 2650 50  0000 C CNN
+F 2 "Connect:USB_Mini-B" V 750 2650 50  0001 C CNN
 F 3 "" V 750 2650 50  0000 C CNN
+F 4 "609-4700-1-ND" H 800 2750 60  0001 C CNN "Digikey P/N"
+F 5 "10033526-N3212LF" H 800 2750 60  0001 C CNN "MFR P/N"
 	1    800  2750
 	0    -1   -1   0
@@
 RX_UART
 $Comp
-L LED D?
+L LED D301
 U 1 1 591EF1B4
 P 7950 3200
-F 0 "D?" H 7950 3300 50  0000 C CNN
+F 0 "D301" H 7950 3300 50  0000 C CNN
 F 1 "TX_LED" H 7950 3100 50  0000 C CNN
 F 2 "" H 7950 3200 50  0000 C CNN
@@
 $EndComp
 $Comp
-L LED D?
+L LED D302
 U 1 1 591EF725
 P 7950 3500
-F 0 "D?" H 7950 3600 50  0000 C CNN
+F 0 "D302" H 7950 3600 50  0000 C CNN
 F 1 "RX_LED" H 7950 3400 50  0000 C CNN
 F 2 "" H 7950 3500 50  0000 C CNN
@@
 $EndComp
 $Comp
-L R R?
+L R R304
 U 1 1 591EF7A4
 P 8550 3200
-F 0 "R?" V 8630 3200 50  0000 C CNN
+F 0 "R304" V 8630 3200 50  0000 C CNN
 F 1 "270" V 8550 3200 50  0000 C CNN
 F 2 "" V 8480 3200 50  0000 C CNN
@@
 $EndComp
 $Comp
-L R R?
+L R R305
 U 1 1 591EF7D4
 P 8550 3500
-F 0 "R?" V 8630 3500 50  0000 C CNN
+F 0 "R305" V 8630 3500 50  0000 C CNN
 F 1 "270" V 8550 3500 50  0000 C CNN
 F 2 "" V 8480 3500 50  0000 C CNN
@@
 	0    1    1    0
 $EndComp
-$Comp
-L +5V #PWR?
-U 1 1 591EF856
-P 8900 3150
-F 0 "#PWR?" H 8900 3000 50  0001 C CNN
-F 1 "+5V" H 8900 3290 50  0000 C CNN
-F 2 "" H 8900 3150 50  0000 C CNN
-F 3 "" H 8900 3150 50  0000 C CNN
-	1    8900 3150
-	1    0    0    -1
-$EndComp
 Text HLabel 7450 2400 2    60   Input ~ 0
 RTS_OUT
@@
 CTS_OUT
 $Comp
-L GND #PWR?
+L GND #PWR306
 U 1 1 591EFDC3
 P 5700 4050
-F 0 "#PWR?" H 5700 3800 50  0001 C CNN
+F 0 "#PWR306" H 5700 3800 50  0001 C CNN
 F 1 "GND" H 5700 3900 50  0000 C CNN
 F 2 "" H 5700 4050 50  0000 C CNN
@@
 $EndComp
 $Comp
-L C C?
+L C C301
 U 1 1 591F012F
 P 3750 1750
-F 0 "C?" H 3775 1850 50  0000 L CNN
+F 0 "C301" H 3775 1850 50  0000 L CNN
 F 1 "100nF" H 3775 1650 50  0000 L CNN
 F 2 "" H 3788 1600 50  0000 C CNN
@@
 $EndComp
 $Comp
-L GND #PWR?
+L GND #PWR301
 U 1 1 591F018C
 P 3750 1900
-F 0 "#PWR?" H 3750 1650 50  0001 C CNN
+F 0 "#PWR301" H 3750 1650 50  0001 C CNN
 F 1 "GND" H 3750 1750 50  0000 C CNN
 F 2 "" H 3750 1900 50  0000 C CNN
@@
 USB_VCC
 $Comp
-L R R?
-U 1 1 591F0F44
-P 2200 2700
-F 0 "R?" V 2280 2700 50  0000 C CNN
-F 1 "22" V 2200 2700 50  0000 C CNN
-F 2 "" V 2130 2700 50  0000 C CNN
-F 3 "" H 2200 2700 50  0000 C CNN
-	1    2200 2700
-	0    1    1    0
-$EndComp
-$Comp
-L R R?
+L R R301
 U 1 1 591F0FCF
 P 2200 2500
-F 0 "R?" V 2280 2500 50  0000 C CNN
+F 0 "R301" V 2280 2500 50  0000 C CNN
 F 1 "22" V 2200 2500 50  0000 C CNN
-F 2 "" V 2130 2500 50  0000 C CNN
+F 2 "Resistors_SMD:R_0805_HandSoldering" V 2130 2500 50  0001 C CNN
 F 3 "" H 2200 2500 50  0000 C CNN
+F 4 "311-22ARCT-ND" V 2200 2500 60  0001 C CNN "Digikey P/N"
+F 5 "RC0805JR-0722RL" V 2200 2500 60  0001 C CNN "MFR P/N"
 	1    2200 2500
 	0    1    1    0
 $EndComp
 $Comp
-L GND #PWR?
+L GND #PWR305
 U 1 1 591F12E5
 P 1800 3750
-F 0 "#PWR?" H 1800 3500 50  0001 C CNN
+F 0 "#PWR305" H 1800 3500 50  0001 C CNN
 F 1 "GND" H 1800 3600 50  0000 C CNN
 F 2 "" H 1800 3750 50  0000 C CNN
@@
 PWR_EN
 $Comp
-L R R?
+L R R303
 U 1 1 59225868
 P 4450 2900
-F 0 "R?" V 4530 2900 50  0000 C CNN
+F 0 "R303" V 4530 2900 50  0000 C CNN
 F 1 "R" V 4450 2900 50  0000 C CNN
 F 2 "" V 4380 2900 50  0000 C CNN
@@
 $EndComp
 $Comp
-L SW_PUSH SW?
+L SW_PUSH SW301
 U 1 1 59225B77
 P 4350 3150
-F 0 "SW?" H 4500 3260 50  0000 C CNN
+F 0 "SW301" H 4500 3260 50  0000 C CNN
 F 1 "SW_PUSH" H 4350 3070 50  0000 C CNN
 F 2 "" H 4350 3150 50  0000 C CNN
@@
 	8400 3500 8150 3500
 Wire Wire Line
-	8700 3200 8700 3350
-Wire Wire Line
-	8700 3350 8700 3500
+	8700 3200 8700 3500
 Wire Wire Line
 	8900 3150 8900 3350
@@
 	6500 2500 7450 2500
 Wire Wire Line
-	4750 3900 5500 3900
-Wire Wire Line
-	5500 3900 5700 3900
-Wire Wire Line
-	5700 3900 5800 3900
-Wire Wire Line
-	5800 3900 5900 3900
+	4750 3900 5900 3900
 Connection ~ 5700 3900
 Connection ~ 5800 3900
@@
 	1500 2850 1500 2700
 Wire Wire Line
-	1500 2700 1950 2700
-Wire Wire Line
-	1950 2700 2050 2700
+	1500 2700 2050 2700
 Wire Wire Line
 	1100 2750 1450 2750
@@
 	1450 2750 1450 2500
 Wire Wire Line
-	1450 2500 1650 2500
-Wire Wire Line
-	1650 2500 2050 2500
+	1450 2500 2050 2500
 Wire Wire Line
 	1650 2900 1650 2500
@@
 	2600 2700 2350 2700
 Wire Wire Line
-	5800 1900 5800 1600
-Wire Wire Line
-	5800 1600 5800 1350
+	5800 1350 5800 1900
 Wire Wire Line
 	5600 1600 5600 1900
 Wire Wire Line
-	4600 2900 4650 2900
-Wire Wire Line
-	4650 2900 4900 2900
+	4600 2900 4900 2900
 Wire Wire Line
 	3850 2800 3850 2900
@@
 	4050 3150 4050 3350
 $Comp
-L GND #PWR?
+L GND #PWR304
 U 1 1 59225F84
 P 4050 3350
-F 0 "#PWR?" H 4050 3100 50  0001 C CNN
+F 0 "#PWR304" H 4050 3100 50  0001 C CNN
 F 1 "GND" H 4050 3200 50  0000 C CNN
 F 2 "" H 4050 3350 50  0000 C CNN
@@
 $EndComp
 $Comp
-L R R?
+L R R306
 U 1 1 59226C41
 P 7050 3700
-F 0 "R?" V 7130 3700 50  0000 C CNN
+F 0 "R306" V 7130 3700 50  0000 C CNN
 F 1 "10k" V 7050 3700 50  0000 C CNN
 F 2 "" V 6980 3700 50  0000 C CNN
@@
 	6800 3500 6800 3850
 Wire Wire Line
-	6800 3850 7050 3850
-Wire Wire Line
-	7050 3850 7300 3850
+	6800 3850 7300 3850
 Connection ~ 7050 3850
 Wire Wire Line
@@
 USB_VCC
 Text Notes 600  850  0    60   ~ 0
-FT232 should only be active when USB is inserted. Sole purpose is plan B programming of the ATMEGA.\nCurrent from BBB should be more than sufficient if BBB RX/TX to the ATMEGA fails.\nMay need to increase varistor and fuse values if on-Pod USB is necessary.
+FT232 should only be active when USB is inserted. Sole purpose is plan B programming of the ATMEGA.\nCurrent from BBB should be more than sufficient if BBB RX/TX to the ATMEGA fails.\nMay need to increase varistor and fuse values if BBB-> USB is necessary.
 NoConn ~ 1100 2650
 Wire Wire Line
@@
 	4900 1600 3750 1600
 Wire Wire Line
-	5600 1600 5800 1600
-Wire Wire Line
-	5800 1600 6500 1600
-Wire Wire Line
-	6500 1600 6900 1600
+	5600 1600 6900 1600
 Connection ~ 5800 1600
 $Comp
-L VR VR?
+L VR VR301
 U 1 1 59229228
 P 1650 3150
-F 0 "VR?" V 1710 3104 50  0000 C TNN
+F 0 "VR301" V 1710 3104 50  0000 C TNN
 F 1 "5V" V 1650 3150 50  0000 C CNN
 F 2 "" H 1650 3150 50  0000 C CNN
@@
 $EndComp
 $Comp
-L VR VR?
+L VR VR302
 U 1 1 5922935A
 P 1950 3150
-F 0 "VR?" V 2010 3104 50  0000 C TNN
+F 0 "VR302" V 2010 3104 50  0000 C TNN
 F 1 "5V" V 1950 3150 50  0000 C CNN
 F 2 "" H 1950 3150 50  0000 C CNN
@@
 $EndComp
 $Comp
-L Ferrite__BLM21_Murata B?
+L Ferrite__BLM21_Murata B301
 U 1 1 5922978C
 P 1800 3550
-F 0 "B?" V 1880 3550 50  0000 C CNN
+F 0 "B301" V 1880 3550 50  0000 C CNN
 F 1 "Ferrite__BLM21_Murata" V 1800 3550 50  0001 C CNN
 F 2 "" V 1730 3550 50  0000 C CNN
@@
 	1800 3700 1800 3750
 $Comp
-L FUSE F?
+L FUSE F301
 U 1 1 5922A236
 P 1100 4150
-F 0 "F?" H 1200 4200 50  0000 C CNN
+F 0 "F301" H 1200 4200 50  0000 C CNN
 F 1 "FUSE" H 1000 4100 50  0000 C CNN
 F 2 "" H 1100 4150 50  0000 C CNN
@@
 $EndComp
 $Comp
-L R R?
+L R R307
 U 1 1 5922A072
 P 4750 3750
-F 0 "R?" V 4830 3750 50  0000 C CNN
+F 0 "R307" V 4830 3750 50  0000 C CNN
 F 1 "0" V 4750 3750 50  0000 C CNN
 F 2 "" V 4680 3750 50  0000 C CNN
@@
 	4750 3600 4900 3600
 $Comp
-L GND #PWR?
+L GND #PWR303
 U 1 1 5922A650
 P 1350 2550
-F 0 "#PWR?" H 1350 2300 50  0001 C CNN
+F 0 "#PWR303" H 1350 2300 50  0001 C CNN
 F 1 "GND" H 1350 2400 50  0000 C CNN
 F 2 "" H 1350 2550 50  0000 C CNN
@@
 SHIELD
 Wire Wire Line
-	1600 3400 1650 3400
-Wire Wire Line
-	1650 3400 1800 3400
-Wire Wire Line
-	1800 3400 1950 3400
+	1600 3400 1950 3400
 Connection ~ 1650 3400
 Connection ~ 1800 3400
@@
 NoConn ~ 6500 2900
 $Comp
-L C C?
+L C C302
 U 1 1 5922B59E
 P 6500 1750
-F 0 "C?" H 6525 1850 50  0000 L CNN
+F 0 "C302" H 6525 1850 50  0000 L CNN
 F 1 "100nF" H 6525 1650 50  0000 L CNN
 F 2 "" H 6538 1600 50  0000 C CNN
@@
 $EndComp
 $Comp
-L C C?
+L C C303
 U 1 1 5922B61D
 P 6900 1750
-F 0 "C?" H 6925 1850 50  0000 L CNN
+F 0 "C303" H 6925 1850 50  0000 L CNN
 F 1 "4.7uF" H 6925 1650 50  0000 L CNN
 F 2 "" H 6938 1600 50  0000 C CNN
@@
 Connection ~ 6500 1600
 Wire Wire Line
-	6500 1900 6650 1900
-Wire Wire Line
-	6650 1900 6900 1900
-$Comp
-L GND #PWR?
+	6500 1900 6900 1900
+$Comp
+L GND #PWR302
 U 1 1 5922B762
 P 6650 1900
-F 0 "#PWR?" H 6650 1650 50  0001 C CNN
+F 0 "#PWR302" H 6650 1650 50  0001 C CNN
 F 1 "GND" H 6650 1750 50  0000 C CNN
 F 2 "" H 6650 1900 50  0000 C CNN
@@
 $EndComp
 Connection ~ 6650 1900
+Text Notes 7800 3000 0    60   ~ 0
+YELLOW\n
+Wire Notes Line
+	7700 2900 7700 3700
+Wire Notes Line
+	7700 3700 8200 3700
+Wire Notes Line
+	8200 3700 8200 2900
+Wire Notes Line
+	8200 2900 7700 2900
+$Comp
+L R R302
+U 1 1 59383E0B
+P 2200 2700
+F 0 "R302" V 2280 2700 50  0000 C CNN
+F 1 "22" V 2200 2700 50  0000 C CNN
+F 2 "Resistors_SMD:R_0805_HandSoldering" V 2130 2700 50  0001 C CNN
+F 3 "" H 2200 2700 50  0000 C CNN
+F 4 "311-22ARCT-ND" V 2200 2700 60  0001 C CNN "Digikey P/N"
+F 5 "RC0805JR-0722RL" V 2200 2700 60  0001 C CNN "MFR P/N"
+	1    2200 2700
+	0    1    1    0
+$EndComp
+Text Label 8900 3150 0    60   ~ 0
+USB_VCC
 $EndSCHEMATC

Commit message: Final edits -- awaiting review before sending out
Parts:
- B301, R303, R304, R305, R306, R307: footprint (none) -> Resistors_SMD:R_0805_HandSoldering
- C301, C302, C303: footprint (none) -> Capacitors_SMD:C_0805_HandSoldering
- D301: footprint (none) -> Diodes_SMD:D_0805; Digikey P/N (none) -> L62507CT-ND; Mfr. P/N (none) -> CMD17-21VYD/TR8
- D302: value RX_LED -> TX_LED; footprint (none) -> Diodes_SMD:D_0805; Digikey P/N (none) -> L62507CT-ND; Mfr. P/N (none) -> CMD17-21VYD/TR8
- F301: footprint (none) -> Resistors_SMD:R_1812_HandSoldering
- SW301: footprint (none) -> Buttons_Switches_SMD:SW_SPST_B3S-1000; Digikey P/N (none) -> SW836CT-ND; Mfr. P/N (none) -> B3S-1000P
- VR301, VR302: footprint (none) -> Resistors_SMD:R_0603_HandSoldering
Changed lines of the file:
@@
 $Descr A4 11693 8268
 encoding utf-8
-Sheet 3 16
+Sheet 3 15
 Title "Motherboard"
 Date ""
@@
 	0    -1   -1   0
 $EndComp
-Text HLabel 7450 2200 2    60   Input ~ 0
+Text HLabel 6500 2200 2    60   Input ~ 0
 TX_UART
-Text HLabel 7450 2300 2    60   Input ~ 0
+Text HLabel 6500 2300 2    60   Input ~ 0
 RX_UART
 $Comp
@@
 F 0 "D301" H 7950 3300 50  0000 C CNN
 F 1 "TX_LED" H 7950 3100 50  0000 C CNN
-F 2 "" H 7950 3200 50  0000 C CNN
+F 2 "Diodes_SMD:D_0805" H 7950 3200 50  0001 C CNN
 F 3 "" H 7950 3200 50  0000 C CNN
+F 4 "L62507CT-ND" H 7950 3200 60  0001 C CNN "Digikey P/N"
+F 5 "CMD17-21VYD/TR8" H 7950 3200 60  0001 C CNN "Mfr. P/N"
 	1    7950 3200
-	1    0    0    -1
-$EndComp
-$Comp
-L LED D302
-U 1 1 591EF725
-P 7950 3500
-F 0 "D302" H 7950 3600 50  0000 C CNN
-F 1 "RX_LED" H 7950 3400 50  0000 C CNN
-F 2 "" H 7950 3500 50  0000 C CNN
-F 3 "" H 7950 3500 50  0000 C CNN
-	1    7950 3500
 	1    0    0    -1
 $EndComp
@@
 F 0 "R304" V 8630 3200 50  0000 C CNN
 F 1 "270" V 8550 3200 50  0000 C CNN
-F 2 "" V 8480 3200 50  0000 C CNN
+F 2 "Resistors_SMD:R_0805_HandSoldering" V 8480 3200 50  0001 C CNN
 F 3 "" H 8550 3200 50  0000 C CNN
 	1    8550 3200
@@
 F 0 "R305" V 8630 3500 50  0000 C CNN
 F 1 "270" V 8550 3500 50  0000 C CNN
-F 2 "" V 8480 3500 50  0000 C CNN
+F 2 "Resistors_SMD:R_0805_HandSoldering" V 8480 3500 50  0001 C CNN
 F 3 "" H 8550 3500 50  0000 C CNN
 	1    8550 3500
 	0    1    1    0
 $EndComp
-Text HLabel 7450 2400 2    60   Input ~ 0
+Text HLabel 6500 2400 2    60   Input ~ 0
 RTS_OUT
-Text HLabel 7450 2500 2    60   Input ~ 0
+Text HLabel 6500 2500 2    60   Input ~ 0
 CTS_OUT
 $Comp
@@
 F 0 "C301" H 3775 1850 50  0000 L CNN
 F 1 "100nF" H 3775 1650 50  0000 L CNN
-F 2 "" H 3788 1600 50  0000 C CNN
+F 2 "Capacitors_SMD:C_0805_HandSoldering" H 3788 1600 50  0001 C CNN
 F 3 "" H 3750 1750 50  0000 C CNN
 	1    3750 1750
@@
 F 0 "R303" V 4530 2900 50  0000 C CNN
 F 1 "R" V 4450 2900 50  0000 C CNN
-F 2 "" V 4380 2900 50  0000 C CNN
+F 2 "Resistors_SMD:R_0805_HandSoldering" V 4380 2900 50  0001 C CNN
 F 3 "" H 4450 2900 50  0000 C CNN
 	1    4450 2900
@@
 F 0 "SW301" H 4500 3260 50  0000 C CNN
 F 1 "SW_PUSH" H 4350 3070 50  0000 C CNN
-F 2 "" H 4350 3150 50  0000 C CNN
+F 2 "Buttons_Switches_SMD:SW_SPST_B3S-1000" H 4350 3150 50  0001 C CNN
 F 3 "" H 4350 3150 50  0000 C CNN
+F 4 "SW836CT-ND" H 4350 3150 60  0001 C CNN "Digikey P/N"
+F 5 "B3S-1000P" H 4350 3150 60  0001 C CNN "Mfr. P/N"
 	1    4350 3150
 	1    0    0    -1
@@
 USB_VCC
 Wire Wire Line
-	6500 2200 7450 2200
-Wire Wire Line
-	6500 2300 7450 2300
-Wire Wire Line
 	6500 3200 7750 3200
 Wire Wire Line
@@
 	8900 3350 8700 3350
 Connection ~ 8700 3350
-Wire Wire Line
-	6500 2400 7450 2400
-Wire Wire Line
-	6500 2500 7450 2500
 Wire Wire Line
 	4750 3900 5900 3900
@@
 F 0 "R306" V 7130 3700 50  0000 C CNN
 F 1 "10k" V 7050 3700 50  0000 C CNN
-F 2 "" V 6980 3700 50  0000 C CNN
+F 2 "Resistors_SMD:R_0805_HandSoldering" V 6980 3700 50  0001 C CNN
 F 3 "" H 7050 3700 50  0000 C CNN
 	1    7050 3700
@@
 F 0 "VR301" V 1710 3104 50  0000 C TNN
 F 1 "5V" V 1650 3150 50  0000 C CNN
-F 2 "" H 1650 3150 50  0000 C CNN
+F 2 "Resistors_SMD:R_0603_HandSoldering" H 1650 3150 50  0001 C CNN
 F 3 "" H 1650 3150 50  0000 C CNN
 F 4 "CG0603MLC-05LECT-ND" V 1650 3150 60  0001 C CNN "Digikey P/N"
@@
 F 0 "VR302" V 2010 3104 50  0000 C TNN
 F 1 "5V" V 1950 3150 50  0000 C CNN
-F 2 "" H 1950 3150 50  0000 C CNN
+F 2 "Resistors_SMD:R_0603_HandSoldering" H 1950 3150 50  0001 C CNN
 F 3 "" H 1950 3150 50  0000 C CNN
 F 4 "CG0603MLC-05LECT-ND" V 1950 3150 60  0001 C CNN "Digikey P/N"
@@
 F 0 "B301" V 1880 3550 50  0000 C CNN
 F 1 "Ferrite__BLM21_Murata" V 1800 3550 50  0001 C CNN
-F 2 "" V 1730 3550 50  0000 C CNN
+F 2 "Resistors_SMD:R_0805_HandSoldering" V 1730 3550 50  0001 C CNN
 F 3 "" H 1800 3550 50  0000 C CNN
 F 4 "490-1040-1-ND" V 1800 3550 60  0001 C CNN "Digikey P/N"
@@
 F 0 "F301" H 1200 4200 50  0000 C CNN
 F 1 "FUSE" H 1000 4100 50  0000 C CNN
-F 2 "" H 1100 4150 50  0000 C CNN
+F 2 "Resistors_SMD:R_1812_HandSoldering" H 1100 4150 50  0001 C CNN
 F 3 "" H 1100 4150 50  0000 C CNN
 F 4 "MS-MSMF050-2CT-ND" H 1100 4150 60  0001 C CNN "Digikey P/N"
@@
 F 0 "R307" V 4830 3750 50  0000 C CNN
 F 1 "0" V 4750 3750 50  0000 C CNN
-F 2 "" V 4680 3750 50  0000 C CNN
+F 2 "Resistors_SMD:R_0805_HandSoldering" V 4680 3750 50  0001 C CNN
 F 3 "" H 4750 3750 50  0000 C CNN
 	1    4750 3750
@@
 F 0 "C302" H 6525 1850 50  0000 L CNN
 F 1 "100nF" H 6525 1650 50  0000 L CNN
-F 2 "" H 6538 1600 50  0000 C CNN
+F 2 "Capacitors_SMD:C_0805_HandSoldering" H 6538 1600 50  0001 C CNN
 F 3 "" H 6500 1750 50  0000 C CNN
 	1    6500 1750
@@
 F 0 "C303" H 6925 1850 50  0000 L CNN
 F 1 "4.7uF" H 6925 1650 50  0000 L CNN
-F 2 "" H 6938 1600 50  0000 C CNN
+F 2 "Capacitors_SMD:C_0805_HandSoldering" H 6938 1600 50  0001 C CNN
 F 3 "" H 6900 1750 50  0000 C CNN
 	1    6900 1750
@@
 Text Label 8900 3150 0    60   ~ 0
 USB_VCC
+$Comp
+L LED D302
+U 1 1 59643610
+P 7950 3500
+F 0 "D302" H 7950 3600 50  0000 C CNN
+F 1 "TX_LED" H 7950 3400 50  0000 C CNN
+F 2 "Diodes_SMD:D_0805" H 7950 3500 50  0001 C CNN
+F 3 "" H 7950 3500 50  0000 C CNN
+F 4 "L62507CT-ND" H 7950 3500 60  0001 C CNN "Digikey P/N"
+F 5 "CMD17-21VYD/TR8" H 7950 3500 60  0001 C CNN "Mfr. P/N"
+	1    7950 3500
+	1    0    0    -1
+$EndComp
 $EndSCHEMATC

Commit message: computer is dying
Parts:
- D302: value TX_LED -> RX_LED
Changed lines of the file:
@@
 CTS_OUT
 $Comp
-L GND #PWR08
+L GND #PWR306
 U 1 1 591EFDC3
 P 5700 4050
-F 0 "#PWR08" H 5700 3800 50  0001 C CNN
+F 0 "#PWR306" H 5700 3800 50  0001 C CNN
 F 1 "GND" H 5700 3900 50  0000 C CNN
 F 2 "" H 5700 4050 50  0000 C CNN
@@
 $EndComp
 $Comp
-L GND #PWR09
+L GND #PWR301
 U 1 1 591F018C
 P 3750 1900
-F 0 "#PWR09" H 3750 1650 50  0001 C CNN
+F 0 "#PWR301" H 3750 1650 50  0001 C CNN
 F 1 "GND" H 3750 1750 50  0000 C CNN
 F 2 "" H 3750 1900 50  0000 C CNN
@@
 $EndComp
 $Comp
-L GND #PWR010
+L GND #PWR305
 U 1 1 591F12E5
 P 1800 3750
-F 0 "#PWR010" H 1800 3500 50  0001 C CNN
+F 0 "#PWR305" H 1800 3500 50  0001 C CNN
 F 1 "GND" H 1800 3600 50  0000 C CNN
 F 2 "" H 1800 3750 50  0000 C CNN
@@
 	4050 3150 4050 3350
 $Comp
-L GND #PWR011
+L GND #PWR304
 U 1 1 59225F84
 P 4050 3350
-F 0 "#PWR011" H 4050 3100 50  0001 C CNN
+F 0 "#PWR304" H 4050 3100 50  0001 C CNN
 F 1 "GND" H 4050 3200 50  0000 C CNN
 F 2 "" H 4050 3350 50  0000 C CNN
@@
 	4750 3600 4900 3600
 $Comp
-L GND #PWR012
+L GND #PWR303
 U 1 1 5922A650
 P 1350 2550
-F 0 "#PWR012" H 1350 2300 50  0001 C CNN
+F 0 "#PWR303" H 1350 2300 50  0001 C CNN
 F 1 "GND" H 1350 2400 50  0000 C CNN
 F 2 "" H 1350 2550 50  0000 C CNN
@@
 	6500 1900 6900 1900
 $Comp
-L GND #PWR013
+L GND #PWR302
 U 1 1 5922B762
 P 6650 1900
-F 0 "#PWR013" H 6650 1650 50  0001 C CNN
+F 0 "#PWR302" H 6650 1650 50  0001 C CNN
 F 1 "GND" H 6650 1750 50  0000 C CNN
 F 2 "" H 6650 1900 50  0000 C CNN
@@
 P 7950 3500
 F 0 "D302" H 7950 3600 50  0000 C CNN
-F 1 "TX_LED" H 7950 3400 50  0000 C CNN
+F 1 "RX_LED" H 7950 3400 50  0000 C CNN
 F 2 "Diodes_SMD:D_0805" H 7950 3500 50  0001 C CNN
 F 3 "" H 7950 3500 50  0000 C CNN
