File: SolidStateRelayBoard/SSRBlock.sch (KiCad schematic (older format))
At the start: 6 parts, among them Q201 NPN, U201 SSR

Commit message: Completed most of layout for SSR board.
Parts:
- added D202: LED, hyperCustom:SOD-123, symbol LED
- added R204: 910, Resistors_SMD:R_1206_HandSoldering, symbol R
- D201: value 3.5V -> 5.6V; footprint (none) -> hyperCustom:SOD-123; DigiKey PN (none) -> MMSZ5232B-FDICT-ND; Mfg. (none) -> Diodes; Mfg. PN (none) -> MMSZ5232B-7-F
- Q201: value NPN -> MMBT2222ALT1G; footprint (none) -> TO_SOT_Packages_SMD:SOT-23_Handsoldering; symbol NPN -> MMBT2222ALT1G; DigiKey PN (none) -> MMBT2222ALT1GOSCT-ND; Mfg. (none) -> ON Semi; Mfg. PN (none) -> MMBT2222ALT1G
- R201: value 50k -> 100k; DigiKey PN 311-49.9KFRCT-ND -> 311-100KFRCT-ND; Mfg. PN RC1206FR-0749K9L -> RC1206FR-07100KL
- U201: footprint (none) -> hyperCustom:VISHAY_6SMD_OPTOCOUPLER
Connections:
- wire segments 17 -> 20

Commit message: Finished layout of SSR Board. Ready for fab.
Parts:
- R201: value 100k -> 10k; DigiKey PN 311-100KFRCT-ND -> 311-10.0KFRCT-ND; Mfg. PN RC1206FR-07100KL -> RC1206FR-0710KL
Changed lines of the file:
@@
 $Descr A4 11693 8268
 encoding utf-8
-Sheet 17 17
+Sheet 2 17
 Title ""
 Date ""
@@
 AR Path="/586B7988/586B33BB" Ref="Q1601"  Part="1"
 AR Path="/586B7996/586B33BB" Ref="Q1701"  Part="1"
-F 0 "Q1701" H 5100 3400 50  0000 R CNN
+F 0 "Q201" H 5100 3400 50  0000 R CNN
 F 1 "MMBT2222ALT1G" H 5100 3400 50  0001 R CNN
 F 2 "TO_SOT_Packages_SMD:SOT-23_Handsoldering" H 5100 3250 60  0001 C CNN
@@
 AR Path="/586B7988/586B33E9" Ref="R1603"  Part="1"
 AR Path="/586B7996/586B33E9" Ref="R1703"  Part="1"
-F 0 "R1703" H 5000 2450 50  0000 C CNN
+F 0 "R203" H 5000 2450 50  0000 C CNN
 F 1 "910" H 5050 2150 50  0000 C CNN
 F 2 "Resistors_SMD:R_1206_HandSoldering" V 5130 2300 30  0001 C CNN
@@
 AR Path="/586B7988/586B3431" Ref="R1601"  Part="1"
 AR Path="/586B7996/586B3431" Ref="R1701"  Part="1"
-F 0 "R1701" V 4300 3050 50  0000 C CNN
-F 1 "100k" V 4300 3400 50  0000 C CNN
+F 0 "R201" V 4300 3050 50  0000 C CNN
+F 1 "10k" V 4300 3400 50  0000 C CNN
 F 2 "Resistors_SMD:R_1206_HandSoldering" V 4330 3250 30  0001 C CNN
 F 3 "" H 4400 3250 30  0000 C CNN
 F 4 "Yageo" V 4400 3250 60  0001 C CNN "Mfg."
-F 5 "RC1206FR-07100KL" V 4400 3250 60  0001 C CNN "Mfg. PN"
-F 6 "311-100KFRCT-ND" V 4400 3250 60  0001 C CNN "DigiKey PN"
+F 5 "RC1206FR-0710KL" V 4400 3250 60  0001 C CNN "Mfg. PN"
+F 6 "311-10.0KFRCT-ND" V 4400 3250 60  0001 C CNN "DigiKey PN"
 	1    4400 3250
 	0    1    1    0
@@
 AR Path="/586B7988/586B354B" Ref="#PWR1604"  Part="1"
 AR Path="/586B7996/586B354B" Ref="#PWR1704"  Part="1"
-F 0 "#PWR1704" H 5200 3350 60  0001 C CNN
+F 0 "#PWR204" H 5200 3350 60  0001 C CNN
 F 1 "GND" H 5200 3450 60  0000 C CNN
 F 2 "" H 5200 3600 60  0000 C CNN
@@
 AR Path="/586B7988/586B3681" Ref="D1601"  Part="1"
 AR Path="/586B7996/586B3681" Ref="D1701"  Part="1"
-F 0 "D1701" V 3450 3700 50  0000 C CNN
+F 0 "D201" V 3450 3700 50  0000 C CNN
 F 1 "5.6V" V 3250 3700 50  0000 C CNN
 F 2 "hyperCustom:SOD-123" H 3350 3500 60  0001 C CNN
@@
 AR Path="/586B7988/586B36D9" Ref="#PWR1601"  Part="1"
 AR Path="/586B7996/586B36D9" Ref="#PWR1701"  Part="1"
-F 0 "#PWR1701" H 3350 3500 60  0001 C CNN
+F 0 "#PWR201" H 3350 3500 60  0001 C CNN
 F 1 "GND" H 3350 3600 60  0000 C CNN
 F 2 "" H 3350 3750 60  0000 C CNN
@@
 AR Path="/586B7988/586B39A4" Ref="R1602"  Part="1"
 AR Path="/586B7996/586B39A4" Ref="R1702"  Part="1"
-F 0 "R1702" H 4650 3750 50  0000 C CNN
+F 0 "R202" H 4650 3750 50  0000 C CNN
 F 1 "1M" H 4650 3450 50  0000 C CNN
 F 2 "Resistors_SMD:R_1206_HandSoldering" V 4730 3600 30  0001 C CNN
@@
 AR Path="/586B7988/586B3A19" Ref="#PWR1603"  Part="1"
 AR Path="/586B7996/586B3A19" Ref="#PWR1703"  Part="1"
-F 0 "#PWR1703" H 4800 3700 60  0001 C CNN
+F 0 "#PWR203" H 4800 3700 60  0001 C CNN
 F 1 "GND" H 4800 3800 60  0000 C CNN
 F 2 "" H 4800 3950 60  0000 C CNN
@@
 AR Path="/586B7988/586D88E1" Ref="U1601"  Part="1"
 AR Path="/586B7996/586D88E1" Ref="U1701"  Part="1"
-F 0 "U1701" H 5750 3150 60  0000 C CNN
+F 0 "U201" H 5750 3150 60  0000 C CNN
 F 1 "SSR" H 6200 2550 60  0000 C CNN
 F 2 "hyperCustom:VISHAY_6SMD_OPTOCOUPLER" H 6000 2850 60  0001 C CNN
@@
 AR Path="/586B7988/586E6B18" Ref="D1602"  Part="1"
 AR Path="/586B7996/586E6B18" Ref="D1702"  Part="1"
-F 0 "D1702" H 3850 3650 50  0000 C CNN
+F 0 "D202" H 3850 3650 50  0000 C CNN
 F 1 "LED" H 3850 3450 50  0000 C CNN
 F 2 "hyperCustom:SOD-123" H 3850 3550 60  0001 C CNN
@@
 AR Path="/586B7988/586E6B5D" Ref="R1604"  Part="1"
 AR Path="/586B7996/586E6B5D" Ref="R1704"  Part="1"
-F 0 "R1704" H 3650 4250 50  0000 C CNN
+F 0 "R204" H 3650 4250 50  0000 C CNN
 F 1 "910" H 3700 3950 50  0000 C CNN
 F 2 "Resistors_SMD:R_1206_HandSoldering" V 3780 4100 30  0001 C CNN
@@
 AR Path="/586B7988/586E6C2B" Ref="#PWR1602"  Part="1"
 AR Path="/586B7996/586E6C2B" Ref="#PWR1702"  Part="1"
-F 0 "#PWR1702" H 3850 4200 60  0001 C CNN
+F 0 "#PWR202" H 3850 4200 60  0001 C CNN
 F 1 "GND" H 3850 4300 60  0000 C CNN
 F 2 "" H 3850 4450 60  0000 C CNN

Commit message: Updated battery board and SSR Board. Completed schematic and layout for Pusher Protection Board (and also renamed it from Emergency Board).
Parts:
- D202: DigiKey PN (none) -> 754-1939-1-ND; Mfg. (none) -> Kingbright; Mfg. PN (none) -> APT2012LZGCK
Changed lines of the file:
@@
 	5200 3450 5200 3600
 $Comp
-L GND #PWR204
+L GND #PWR035
 U 1 1 586B354B
 P 5200 3600
-AR Path="/586B2B8E/586B354B" Ref="#PWR204"  Part="1"
-AR Path="/586B3F68/586B354B" Ref="#PWR304"  Part="1"
-AR Path="/586B4A2A/586B354B" Ref="#PWR404"  Part="1"
-AR Path="/586B4A38/586B354B" Ref="#PWR504"  Part="1"
-AR Path="/586B65A6/586B354B" Ref="#PWR604"  Part="1"
-AR Path="/586B65B4/586B354B" Ref="#PWR704"  Part="1"
-AR Path="/586B65C2/586B354B" Ref="#PWR804"  Part="1"
-AR Path="/586B65D0/586B354B" Ref="#PWR904"  Part="1"
-AR Path="/586B7934/586B354B" Ref="#PWR1004"  Part="1"
-AR Path="/586B7942/586B354B" Ref="#PWR1104"  Part="1"
-AR Path="/586B7950/586B354B" Ref="#PWR1204"  Part="1"
-AR Path="/586B795E/586B354B" Ref="#PWR1304"  Part="1"
-AR Path="/586B796C/586B354B" Ref="#PWR1404"  Part="1"
-AR Path="/586B797A/586B354B" Ref="#PWR1504"  Part="1"
-AR Path="/586B7988/586B354B" Ref="#PWR1604"  Part="1"
-AR Path="/586B7996/586B354B" Ref="#PWR1704"  Part="1"
-F 0 "#PWR204" H 5200 3350 60  0001 C CNN
+AR Path="/586B2B8E/586B354B" Ref="#PWR035"  Part="1"
+AR Path="/586B3F68/586B354B" Ref="#PWR039"  Part="1"
+AR Path="/586B4A2A/586B354B" Ref="#PWR043"  Part="1"
+AR Path="/586B4A38/586B354B" Ref="#PWR047"  Part="1"
+AR Path="/586B65A6/586B354B" Ref="#PWR051"  Part="1"
+AR Path="/586B65B4/586B354B" Ref="#PWR055"  Part="1"
+AR Path="/586B65C2/586B354B" Ref="#PWR059"  Part="1"
+AR Path="/586B65D0/586B354B" Ref="#PWR063"  Part="1"
+AR Path="/586B7934/586B354B" Ref="#PWR067"  Part="1"
+AR Path="/586B7942/586B354B" Ref="#PWR071"  Part="1"
+AR Path="/586B7950/586B354B" Ref="#PWR075"  Part="1"
+AR Path="/586B795E/586B354B" Ref="#PWR079"  Part="1"
+AR Path="/586B796C/586B354B" Ref="#PWR083"  Part="1"
+AR Path="/586B797A/586B354B" Ref="#PWR087"  Part="1"
+AR Path="/586B7988/586B354B" Ref="#PWR091"  Part="1"
+AR Path="/586B7996/586B354B" Ref="#PWR095"  Part="1"
+F 0 "#PWR035" H 5200 3350 60  0001 C CNN
 F 1 "GND" H 5200 3450 60  0000 C CNN
 F 2 "" H 5200 3600 60  0000 C CNN
@@
 	3350 3700 3350 3750
 $Comp
-L GND #PWR201
+L GND #PWR036
 U 1 1 586B36D9
 P 3350 3750
-AR Path="/586B2B8E/586B36D9" Ref="#PWR201"  Part="1"
-AR Path="/586B3F68/586B36D9" Ref="#PWR301"  Part="1"
-AR Path="/586B4A2A/586B36D9" Ref="#PWR401"  Part="1"
-AR Path="/586B4A38/586B36D9" Ref="#PWR501"  Part="1"
-AR Path="/586B65A6/586B36D9" Ref="#PWR601"  Part="1"
-AR Path="/586B65B4/586B36D9" Ref="#PWR701"  Part="1"
-AR Path="/586B65C2/586B36D9" Ref="#PWR801"  Part="1"
-AR Path="/586B65D0/586B36D9" Ref="#PWR901"  Part="1"
-AR Path="/586B7934/586B36D9" Ref="#PWR1001"  Part="1"
-AR Path="/586B7942/586B36D9" Ref="#PWR1101"  Part="1"
-AR Path="/586B7950/586B36D9" Ref="#PWR1201"  Part="1"
-AR Path="/586B795E/586B36D9" Ref="#PWR1301"  Part="1"
-AR Path="/586B796C/586B36D9" Ref="#PWR1401"  Part="1"
-AR Path="/586B797A/586B36D9" Ref="#PWR1501"  Part="1"
-AR Path="/586B7988/586B36D9" Ref="#PWR1601"  Part="1"
-AR Path="/586B7996/586B36D9" Ref="#PWR1701"  Part="1"
-F 0 "#PWR201" H 3350 3500 60  0001 C CNN
+AR Path="/586B2B8E/586B36D9" Ref="#PWR036"  Part="1"
+AR Path="/586B3F68/586B36D9" Ref="#PWR040"  Part="1"
+AR Path="/586B4A2A/586B36D9" Ref="#PWR044"  Part="1"
+AR Path="/586B4A38/586B36D9" Ref="#PWR048"  Part="1"
+AR Path="/586B65A6/586B36D9" Ref="#PWR052"  Part="1"
+AR Path="/586B65B4/586B36D9" Ref="#PWR056"  Part="1"
+AR Path="/586B65C2/586B36D9" Ref="#PWR060"  Part="1"
+AR Path="/586B65D0/586B36D9" Ref="#PWR064"  Part="1"
+AR Path="/586B7934/586B36D9" Ref="#PWR068"  Part="1"
+AR Path="/586B7942/586B36D9" Ref="#PWR072"  Part="1"
+AR Path="/586B7950/586B36D9" Ref="#PWR076"  Part="1"
+AR Path="/586B795E/586B36D9" Ref="#PWR080"  Part="1"
+AR Path="/586B796C/586B36D9" Ref="#PWR084"  Part="1"
+AR Path="/586B797A/586B36D9" Ref="#PWR088"  Part="1"
+AR Path="/586B7988/586B36D9" Ref="#PWR092"  Part="1"
+AR Path="/586B7996/586B36D9" Ref="#PWR096"  Part="1"
+F 0 "#PWR036" H 3350 3500 60  0001 C CNN
 F 1 "GND" H 3350 3600 60  0000 C CNN
 F 2 "" H 3350 3750 60  0000 C CNN
@@
 	4800 3850 4800 3950
 $Comp
-L GND #PWR203
+L GND #PWR037
 U 1 1 586B3A19
 P 4800 3950
-AR Path="/586B2B8E/586B3A19" Ref="#PWR203"  Part="1"
-AR Path="/586B3F68/586B3A19" Ref="#PWR303"  Part="1"
-AR Path="/586B4A2A/586B3A19" Ref="#PWR403"  Part="1"
-AR Path="/586B4A38/586B3A19" Ref="#PWR503"  Part="1"
-AR Path="/586B65A6/586B3A19" Ref="#PWR603"  Part="1"
-AR Path="/586B65B4/586B3A19" Ref="#PWR703"  Part="1"
-AR Path="/586B65C2/586B3A19" Ref="#PWR803"  Part="1"
-AR Path="/586B65D0/586B3A19" Ref="#PWR903"  Part="1"
-AR Path="/586B7934/586B3A19" Ref="#PWR1003"  Part="1"
-AR Path="/586B7942/586B3A19" Ref="#PWR1103"  Part="1"
-AR Path="/586B7950/586B3A19" Ref="#PWR1203"  Part="1"
-AR Path="/586B795E/586B3A19" Ref="#PWR1303"  Part="1"
-AR Path="/586B796C/586B3A19" Ref="#PWR1403"  Part="1"
-AR Path="/586B797A/586B3A19" Ref="#PWR1503"  Part="1"
-AR Path="/586B7988/586B3A19" Ref="#PWR1603"  Part="1"
-AR Path="/586B7996/586B3A19" Ref="#PWR1703"  Part="1"
-F 0 "#PWR203" H 4800 3700 60  0001 C CNN
+AR Path="/586B2B8E/586B3A19" Ref="#PWR037"  Part="1"
+AR Path="/586B3F68/586B3A19" Ref="#PWR041"  Part="1"
+AR Path="/586B4A2A/586B3A19" Ref="#PWR045"  Part="1"
+AR Path="/586B4A38/586B3A19" Ref="#PWR049"  Part="1"
+AR Path="/586B65A6/586B3A19" Ref="#PWR053"  Part="1"
+AR Path="/586B65B4/586B3A19" Ref="#PWR057"  Part="1"
+AR Path="/586B65C2/586B3A19" Ref="#PWR061"  Part="1"
+AR Path="/586B65D0/586B3A19" Ref="#PWR065"  Part="1"
+AR Path="/586B7934/586B3A19" Ref="#PWR069"  Part="1"
+AR Path="/586B7942/586B3A19" Ref="#PWR073"  Part="1"
+AR Path="/586B7950/586B3A19" Ref="#PWR077"  Part="1"
+AR Path="/586B795E/586B3A19" Ref="#PWR081"  Part="1"
+AR Path="/586B796C/586B3A19" Ref="#PWR085"  Part="1"
+AR Path="/586B797A/586B3A19" Ref="#PWR089"  Part="1"
+AR Path="/586B7988/586B3A19" Ref="#PWR093"  Part="1"
+AR Path="/586B7996/586B3A19" Ref="#PWR097"  Part="1"
+F 0 "#PWR037" H 4800 3700 60  0001 C CNN
 F 1 "GND" H 4800 3800 60  0000 C CNN
 F 2 "" H 4800 3950 60  0000 C CNN
@@
 F 2 "hyperCustom:SOD-123" H 3850 3550 60  0001 C CNN
 F 3 "" H 3850 3550 60  0000 C CNN
+F 4 "Kingbright" H 3850 3550 60  0001 C CNN "Mfg."
+F 5 "APT2012LZGCK" H 3850 3550 60  0001 C CNN "Mfg. PN"
+F 6 "754-1939-1-ND" H 3850 3550 60  0001 C CNN "DigiKey PN"
 	1    3850 3550
 	0    1    1    0
@@
 	3850 4350 3850 4450
 $Comp
-L GND #PWR202
+L GND #PWR038
 U 1 1 586E6C2B
 P 3850 4450
-AR Path="/586B2B8E/586E6C2B" Ref="#PWR202"  Part="1"
-AR Path="/586B3F68/586E6C2B" Ref="#PWR302"  Part="1"
-AR Path="/586B4A2A/586E6C2B" Ref="#PWR402"  Part="1"
-AR Path="/586B4A38/586E6C2B" Ref="#PWR502"  Part="1"
-AR Path="/586B65A6/586E6C2B" Ref="#PWR602"  Part="1"
-AR Path="/586B65B4/586E6C2B" Ref="#PWR702"  Part="1"
-AR Path="/586B65C2/586E6C2B" Ref="#PWR802"  Part="1"
-AR Path="/586B65D0/586E6C2B" Ref="#PWR902"  Part="1"
-AR Path="/586B7934/586E6C2B" Ref="#PWR1002"  Part="1"
-AR Path="/586B7942/586E6C2B" Ref="#PWR1102"  Part="1"
-AR Path="/586B7950/586E6C2B" Ref="#PWR1202"  Part="1"
-AR Path="/586B795E/586E6C2B" Ref="#PWR1302"  Part="1"
-AR Path="/586B796C/586E6C2B" Ref="#PWR1402"  Part="1"
-AR Path="/586B797A/586E6C2B" Ref="#PWR1502"  Part="1"
-AR Path="/586B7988/586E6C2B" Ref="#PWR1602"  Part="1"
-AR Path="/586B7996/586E6C2B" Ref="#PWR1702"  Part="1"
-F 0 "#PWR202" H 3850 4200 60  0001 C CNN
+AR Path="/586B2B8E/586E6C2B" Ref="#PWR038"  Part="1"
+AR Path="/586B3F68/586E6C2B" Ref="#PWR042"  Part="1"
+AR Path="/586B4A2A/586E6C2B" Ref="#PWR046"  Part="1"
+AR Path="/586B4A38/586E6C2B" Ref="#PWR050"  Part="1"
+AR Path="/586B65A6/586E6C2B" Ref="#PWR054"  Part="1"
+AR Path="/586B65B4/586E6C2B" Ref="#PWR058"  Part="1"
+AR Path="/586B65C2/586E6C2B" Ref="#PWR062"  Part="1"
+AR Path="/586B65D0/586E6C2B" Ref="#PWR066"  Part="1"
+AR Path="/586B7934/586E6C2B" Ref="#PWR070"  Part="1"
+AR Path="/586B7942/586E6C2B" Ref="#PWR074"  Part="1"
+AR Path="/586B7950/586E6C2B" Ref="#PWR078"  Part="1"
+AR Path="/586B795E/586E6C2B" Ref="#PWR082"  Part="1"
+AR Path="/586B796C/586E6C2B" Ref="#PWR086"  Part="1"
+AR Path="/586B797A/586E6C2B" Ref="#PWR090"  Part="1"
+AR Path="/586B7988/586E6C2B" Ref="#PWR094"  Part="1"
+AR Path="/586B7996/586E6C2B" Ref="#PWR098"  Part="1"
+F 0 "#PWR038" H 3850 4200 60  0001 C CNN
 F 1 "GND" H 3850 4300 60  0000 C CNN
 F 2 "" H 3850 4450 60  0000 C CNN

Commit message: Deleted some of the unnecessary circuits for the relays that won’t be used anymore since we will have two boards now.
Parts:
- D201: symbol ZENER -> ZENER-RESCUE-SSRBoard
- D202: symbol LED -> LED-RESCUE-SSRBoard
- R201, R202, R203, R204: symbol R -> R-RESCUE-SSRBoard
Changed lines of the file:
@@
 EESchema Schematic File Version 2
+LIBS:SSRBoard-rescue
 LIBS:transistors
 LIBS:device
@@
 LIBS:silabs
 LIBS:siliconi
-LIBS:special
 LIBS:stm8
 LIBS:stm32
@@
 $EndComp
 $Comp
-L R R203
+L R-RESCUE-SSRBoard R203
 U 1 1 586B33E9
 P 5200 2300
@@
 $EndComp
 $Comp
-L R R201
+L R-RESCUE-SSRBoard R201
 U 1 1 586B3431
 P 4400 3250
@@
 	3150 3250 4150 3250
 $Comp
-L ZENER D201
+L ZENER-RESCUE-SSRBoard D201
 U 1 1 586B3681
 P 3350 3500
@@
 $EndComp
 $Comp
-L R R202
+L R-RESCUE-SSRBoard R202
 U 1 1 586B39A4
 P 4800 3600
@@
 $EndComp
 $Comp
-L LED D202
+L LED-RESCUE-SSRBoard D202
 U 1 1 586E6B18
 P 3850 3550
@@
 AR Path="/586B7988/586E6B18" Ref="D1602"  Part="1"
 AR Path="/586B7996/586E6B18" Ref="D1702"  Part="1"
+AR Path="/586E6B18" Ref="D202"  Part="1"
 F 0 "D202" H 3850 3650 50  0000 C CNN
 F 1 "LED" H 3850 3450 50  0000 C CNN
@@
 $EndComp
 $Comp
-L R R204
+L R-RESCUE-SSRBoard R204
 U 1 1 586E6B5D
 P 3850 4100

Commit message: SSR Board
Misc small changes
Changed lines of the file:
@@
 $Descr A4 11693 8268
 encoding utf-8
-Sheet 2 14
+Sheet 7 14
 Title ""
 Date ""
@@
 AR Path="/586B7988/586B33BB" Ref="Q1601"  Part="1"
 AR Path="/586B7996/586B33BB" Ref="Q1701"  Part="1"
-F 0 "Q201" H 5100 3400 50  0000 R CNN
+F 0 "Q701" H 5100 3400 50  0000 R CNN
 F 1 "MMBT2222ALT1G" H 5100 3400 50  0001 R CNN
 F 2 "TO_SOT_Packages_SMD:SOT-23_Handsoldering" H 5100 3250 60  0001 C CNN
@@
 AR Path="/586B7988/586B33E9" Ref="R1603"  Part="1"
 AR Path="/586B7996/586B33E9" Ref="R1703"  Part="1"
-F 0 "R203" H 5000 2450 50  0000 C CNN
+F 0 "R703" H 5000 2450 50  0000 C CNN
 F 1 "910" H 5050 2150 50  0000 C CNN
 F 2 "Resistors_SMD:R_1206_HandSoldering" V 5130 2300 30  0001 C CNN
@@
 AR Path="/586B7988/586B3431" Ref="R1601"  Part="1"
 AR Path="/586B7996/586B3431" Ref="R1701"  Part="1"
-F 0 "R201" V 4300 3050 50  0000 C CNN
+F 0 "R701" V 4300 3050 50  0000 C CNN
 F 1 "10k" V 4300 3400 50  0000 C CNN
 F 2 "Resistors_SMD:R_1206_HandSoldering" V 4330 3250 30  0001 C CNN
@@
 AR Path="/586B7988/586B354B" Ref="#PWR091"  Part="1"
 AR Path="/586B7996/586B354B" Ref="#PWR095"  Part="1"
-F 0 "#PWR084" H 5200 3350 60  0001 C CNN
+F 0 "#PWR056" H 5200 3350 60  0001 C CNN
 F 1 "GND" H 5200 3450 60  0000 C CNN
 F 2 "" H 5200 3600 60  0000 C CNN
@@
 AR Path="/586B7988/586B3681" Ref="D1601"  Part="1"
 AR Path="/586B7996/586B3681" Ref="D1701"  Part="1"
-F 0 "D201" V 3450 3700 50  0000 C CNN
+F 0 "D701" V 3450 3700 50  0000 C CNN
 F 1 "5.6V" V 3250 3700 50  0000 C CNN
 F 2 "hyperCustom:SOD-123" H 3350 3500 60  0001 C CNN
@@
 AR Path="/586B7988/586B36D9" Ref="#PWR092"  Part="1"
 AR Path="/586B7996/586B36D9" Ref="#PWR096"  Part="1"
-F 0 "#PWR085" H 3350 3500 60  0001 C CNN
+F 0 "#PWR057" H 3350 3500 60  0001 C CNN
 F 1 "GND" H 3350 3600 60  0000 C CNN
 F 2 "" H 3350 3750 60  0000 C CNN
@@
 AR Path="/586B7988/586B39A4" Ref="R1602"  Part="1"
 AR Path="/586B7996/586B39A4" Ref="R1702"  Part="1"
-F 0 "R202" H 4650 3750 50  0000 C CNN
+F 0 "R702" H 4650 3750 50  0000 C CNN
 F 1 "1M" H 4650 3450 50  0000 C CNN
 F 2 "Resistors_SMD:R_1206_HandSoldering" V 4730 3600 30  0001 C CNN
@@
 AR Path="/586B7988/586B3A19" Ref="#PWR093"  Part="1"
 AR Path="/586B7996/586B3A19" Ref="#PWR097"  Part="1"
-F 0 "#PWR086" H 4800 3700 60  0001 C CNN
+F 0 "#PWR058" H 4800 3700 60  0001 C CNN
 F 1 "GND" H 4800 3800 60  0000 C CNN
 F 2 "" H 4800 3950 60  0000 C CNN
@@
 AR Path="/586B7988/586D88E1" Ref="U1601"  Part="1"
 AR Path="/586B7996/586D88E1" Ref="U1701"  Part="1"
-F 0 "U201" H 5750 3150 60  0000 C CNN
+F 0 "U701" H 5750 3150 60  0000 C CNN
 F 1 "SSR" H 6200 2550 60  0000 C CNN
 F 2 "hyperCustom:VISHAY_6SMD_OPTOCOUPLER" H 6000 2850 60  0001 C CNN
@@
 AR Path="/586B7996/586E6B18" Ref="D1702"  Part="1"
 AR Path="/586E6B18" Ref="D202"  Part="1"
-F 0 "D202" H 3850 3650 50  0000 C CNN
+F 0 "D702" H 3850 3650 50  0000 C CNN
 F 1 "LED" H 3850 3450 50  0000 C CNN
 F 2 "hyperCustom:SOD-123" H 3850 3550 60  0001 C CNN
@@
 AR Path="/586B7988/586E6B5D" Ref="R1604"  Part="1"
 AR Path="/586B7996/586E6B5D" Ref="R1704"  Part="1"
-F 0 "R204" H 3650 4250 50  0000 C CNN
+F 0 "R704" H 3650 4250 50  0000 C CNN
 F 1 "910" H 3700 3950 50  0000 C CNN
 F 2 "Resistors_SMD:R_1206_HandSoldering" V 3780 4100 30  0001 C CNN
@@
 AR Path="/586B7988/586E6C2B" Ref="#PWR094"  Part="1"
 AR Path="/586B7996/586E6C2B" Ref="#PWR098"  Part="1"
-F 0 "#PWR087" H 3850 4200 60  0001 C CNN
+F 0 "#PWR059" H 3850 4200 60  0001 C CNN
 F 1 "GND" H 3850 4300 60  0000 C CNN
 F 2 "" H 3850 4450 60  0000 C CNN
