File: BBB-Cape/KiCAD/BBB-Cape.kicad_pcb (KiCad board)
At the start: 2 copper layers, 75.3 x 54.6 mm, 70 parts, among them J1 01x06_Stackable Header, J2 RJ45-TRANSFO, P8 02x23_Stackable Header, P9 02x23_Stackable Header, SW1 W5500_RST, SW2 SYS_RST, SW3 Power, U1 WIZnet W5500, Y1 25MHz

Commit message: Rev1 Board Post for Checkup
Parts:
- removed I2C1_1, I2C1_2, I2C1_3, I2C2_1, I2C2_2, I2C2_3: Conn_01x02, Pin_Headers:Pin_Header_Straight_1x02_Pitch2.54mm
- removed REF** (x4): 1pin, Connectors:1pin
- removed SPI0_2: Conn_01x04, Pin_Headers:Pin_Header_Straight_1x04_Pitch2.54mm
- removed SPI1_2: Conn_01x05, Pin_Headers:Pin_Header_Straight_1x05_Pitch2.54mm
- added I2C1_0: Conn_01x02, Pin_Headers:Pin_Header_Straight_1x02_Pitch2.54mm_SMD_Pin1Left, F.Cu at (166.6, 113.5)
- added I2C2_0: Conn_01x02, Pin_Headers:Pin_Header_Straight_1x02_Pitch2.54mm_SMD_Pin1Left, F.Cu at (130.2, 113.4)
- AIN(1.8V)1: footprint Pin_Headers:Pin_Header_Straight_2x05_Pitch2.54mm -> Pin_Headers:Pin_Header_Straight_2x05_Pitch2.54mm_SMD
- GPIO1: footprint Pin_Headers:Pin_Header_Straight_2x11_Pitch2.54mm -> Pin_Headers:Pin_Header_Straight_2x11_Pitch2.54mm_SMD
- PRUs1: footprint Pin_Headers:Pin_Header_Straight_2x07_Pitch2.54mm -> Pin_Headers:Pin_Header_Straight_2x07_Pitch2.54mm_SMD
- PWR1: footprint Pin_Headers:Pin_Header_Straight_2x08_Pitch2.54mm -> Pin_Headers:Pin_Header_Straight_2x08_Pitch2.54mm_SMD
- SPI0_1, UART4, UART5: footprint Pin_Headers:Pin_Header_Straight_1x04_Pitch2.54mm -> Pin_Headers:Pin_Header_Straight_1x04_Pitch2.54mm_SMD_Pin1Left
- SPI1_1: footprint Pin_Headers:Pin_Header_Straight_1x05_Pitch2.54mm -> Pin_Headers:Pin_Header_Straight_1x05_Pitch2.54mm_SMD_Pin1Left
- TIMER/PWM1: footprint Pin_Headers:Pin_Header_Straight_2x04_Pitch2.54mm -> Pin_Headers:Pin_Header_Straight_2x04_Pitch2.54mm_SMD
- UART3: footprint Pin_Headers:Pin_Header_Straight_1x03_Pitch2.54mm -> Pin_Headers:Pin_Header_Straight_1x03_Pitch2.54mm_SMD_Pin1Left
- moved U1 66.5 mm to (128.9, 98.9)
- moved UART3 16.6 mm to (137.3, 83.7), turned to 180 degrees
- moved GPIO1 11.0 mm to (129.2, 94.0)
- moved R21 10.8 mm to (109.9, 118.2), turned to 90 degrees
- moved UART5 10.8 mm to (157.7, 83.7), turned to 0 degrees
- moved D1 9.16 mm to (105.2, 118.5), turned to 90 degrees
- moved UART4 9.08 mm to (148.3, 84.1), turned to 180 degrees
- moved PWR1 7.37 mm to (125.3, 104.3)
- moved SPI0_1 7.04 mm to (119.0, 113.7)
- moved PRUs1 7.00 mm to (121.0, 83.2)
- moved TIMER/PWM1 3.66 mm to (103.8, 83.9)
- moved SPI1_1 2.62 mm to (142.2, 108.6), turned to 0 degrees
- moved AIN(1.8V)1 1.74 mm to (154.5, 114.7)
- moved J1 0.38 mm to (126.9, 119.8)
Connections:
- GPIO1 pad 21: Net-(GPIO1-Pad21) -> DGND
