File: BatteryShield/Isolation.sch (KiCad schematic (older format))
At the start: 0 parts

Commit message: Added some ideas for isolation and an alternate temp sensor
Parts:
- added D?: LED, symbol LED
- added D?: D, symbol D
- added Q?: BSC030N08NS5ATMA1, TO_SOT_Packages_SMD:TDSON-8-1, symbol BSC030N08NS5ATMA1
- added Q?: IRF4905, TO_SOT_Packages_THT:TO-220_Vertical, symbol IRF4905
- added R? (x2): R, symbol R
Connections:
- new net: Q?.1 (G), Q?.1 (S), R?.2
- new net: D?.1 (K), R?.1
- new net 42V_BATT: D?.2 (A), Q?.2 (D)
- new net 42V_POD: D?.1 (K), Q?.3 (S)
- new net 5V_BBB: Q?.4 (G), R?.1
- new net GND: D?.2 (A), Q?.5 (D), R?.2
Changed lines of the file:
@@
 EESchema Schematic File Version 2
-LIBS:adc081c021
 LIBS:power
 LIBS:device
@@
 LIBS:contrib
 LIBS:valves
-LIBS:LTC4151IMS-1-PBF
-LIBS:Battery_Shield-cache
 EELAYER 25 0
 EELAYER END
 $Descr A4 11693 8268
 encoding utf-8
-Sheet 1 7
+Sheet 1 1
 Title ""
 Date ""
@@
 Comment4 ""
 $EndDescr
+$Comp
+L BSC030N08NS5ATMA1 Q?
+U 1 1 5A7E917C
+P 4300 2650
+F 0 "Q?" H 4100 2950 50  0000 L CNN
+F 1 "BSC030N08NS5ATMA1" H 4100 2400 50  0000 L CNN
+F 2 "TO_SOT_Packages_SMD:TDSON-8-1" H 4300 2850 50  0001 C CIN
+F 3 "" V 4300 2650 50  0001 L CNN
+	1    4300 2650
+	1    0    0    -1
+$EndComp
+$Comp
+L LED D?
+U 1 1 5A7E9290
+P 4000 1550
+F 0 "D?" H 4000 1650 50  0000 C CNN
+F 1 "LED" H 4000 1450 50  0000 C CNN
+F 2 "" H 4000 1550 50  0001 C CNN
+F 3 "" H 4000 1550 50  0001 C CNN
+	1    4000 1550
+	0    -1   -1   0
+$EndComp
+$Comp
+L R R?
+U 1 1 5A7E9392
+P 4000 3050
+F 0 "R?" V 4080 3050 50  0000 C CNN
+F 1 "R" V 4000 3050 50  0000 C CNN
+F 2 "" V 3930 3050 50  0001 C CNN
+F 3 "" H 4000 3050 50  0001 C CNN
+	1    4000 3050
+	1    0    0    -1
+$EndComp
+$Comp
+L R R?
+U 1 1 5A7E9439
+P 4000 2000
+F 0 "R?" V 4080 2000 50  0000 C CNN
+F 1 "R" V 4000 2000 50  0000 C CNN
+F 2 "" V 3930 2000 50  0001 C CNN
+F 3 "" H 4000 2000 50  0001 C CNN
+	1    4000 2000
+	1    0    0    -1
+$EndComp
+$Comp
+L D D?
+U 1 1 5A7E94DC
+P 5150 2500
+F 0 "D?" H 5150 2600 50  0000 C CNN
+F 1 "D" H 5150 2400 50  0000 C CNN
+F 2 "" H 5150 2500 50  0001 C CNN
+F 3 "" H 5150 2500 50  0001 C CNN
+	1    5150 2500
+	0    1    1    0
+$EndComp
+$Comp
+L IRF4905 Q?
+U 1 1 5A7E9597
+P 4800 2150
+F 0 "Q?" H 5050 2225 50  0000 L CNN
+F 1 "IRF4905" H 5050 2150 50  0000 L CNN
+F 2 "TO_SOT_Packages_THT:TO-220_Vertical" H 5050 2075 50  0001 L CIN
+F 3 "" H 4800 2150 50  0001 L CNN
+	1    4800 2150
+	1    0    0    -1
+$EndComp
+$Comp
+L GND #PWR?
+U 1 1 5A7E99F1
+P 4000 3200
+F 0 "#PWR?" H 4000 2950 50  0001 C CNN
+F 1 "GND" H 4000 3050 50  0000 C CNN
+F 2 "" H 4000 3200 50  0001 C CNN
+F 3 "" H 4000 3200 50  0001 C CNN
+	1    4000 3200
+	1    0    0    -1
+$EndComp
+Text HLabel 5150 2350 2    60   Input ~ 0
+42V_POD
+Text HLabel 4000 2750 0    60   Input ~ 0
+5V_BBB
+Text HLabel 4900 1950 1    60   Input ~ 0
+42V_BATT
+Text HLabel 4000 1400 1    60   Input ~ 0
+42V_BATT
+$Comp
+L GND #PWR?
+U 1 1 5A7E993F
+P 5150 2650
+F 0 "#PWR?" H 5150 2400 50  0001 C CNN
+F 1 "GND" H 5150 2500 50  0000 C CNN
+F 2 "" H 5150 2650 50  0001 C CNN
+F 3 "" H 5150 2650 50  0001 C CNN
+	1    5150 2650
+	1    0    0    -1
+$EndComp
+Wire Wire Line
+	4000 2150 4000 2450
+Wire Wire Line
+	4000 1850 4000 1700
+Wire Wire Line
+	4600 2150 4000 2150
+Wire Wire Line
+	4900 2350 5150 2350
+Wire Wire Line
+	4600 2750 4600 3200
+$Comp
+L GND #PWR?
+U 1 1 5A7E9A0E
+P 4600 3200
+F 0 "#PWR?" H 4600 2950 50  0001 C CNN
+F 1 "GND" H 4600 3050 50  0000 C CNN
+F 2 "" H 4600 3200 50  0001 C CNN
+F 3 "" H 4600 3200 50  0001 C CNN
+	1    4600 3200
+	1    0    0    -1
+$EndComp
+Wire Wire Line
+	4000 2750 4000 2900
 $EndSCHEMATC
