File: BatteryShield/protection.sch (KiCad schematic (older format))
At the start: 10 parts

Commit message: Small cosmetic updates
Fixed small cosmetic updates
Changed lines of the file:
@@
 L GND #PWR?
 U 1 1 5B120B55
-P 3250 5850
-F 0 "#PWR?" H 3250 5600 50  0001 C CNN
-F 1 "GND" H 3250 5700 50  0000 C CNN
-F 2 "" H 3250 5850 50  0001 C CNN
-F 3 "" H 3250 5850 50  0001 C CNN
-	1    3250 5850
+P 3200 6600
+F 0 "#PWR?" H 3200 6350 50  0001 C CNN
+F 1 "GND" H 3200 6450 50  0000 C CNN
+F 2 "" H 3200 6600 50  0001 C CNN
+F 3 "" H 3200 6600 50  0001 C CNN
+	1    3200 6600
 	1    0    0    -1
 $EndComp
-Text GLabel 2550 5750 0    60   Input ~ 0
+Text GLabel 3200 5750 1    60   Input ~ 0
 BBB_GND
 Wire Wire Line
-	2550 5750 3250 5750
+	3200 5750 3200 6600
+Text GLabel 3750 6050 2    60   Input ~ 0
+GND_TRACE
 Wire Wire Line
-	3250 5750 3250 5850
+	3750 6050 3200 6050
+Connection ~ 3200 6050
 $EndSCHEMATC

Commit message: Associated a lot of footprints
Now I need to add a lot more :(
Parts:
- removed C? (x2): 10nF, symbol C
- removed D? (x5): DZ2W03600L, symbol D_Zener
- added C? (x2): 10nF, Capacitors_SMD:C_0402, symbol C
- added D? (x5): DZ2W03600L, Diodes_SMD:D_1206, symbol D_Zener
- C?: footprint (none) -> Capacitors_SMD:C_0402
- D?: footprint (none) -> Diodes_SMD:D_1206
Connections:
- net +5V: now also D?.1 (K), D?.1 (K), D?.1 (K)
- net GND: now also C?.2, C?.2, D?.2 (A), D?.2 (A)
- net PACK_A_ON: now also D?.1 (K), D?.2 (A)
- net PACK_B_ON: now also C?.1, D?.1 (K), D?.2 (A)
- net PRECHARGE_N: now also C?.1, D?.2 (A)
Changed lines of the file:
@@
 $Descr A4 11693 8268
 encoding utf-8
-Sheet 11 12
+Sheet 10 12
 Title ""
 Date ""
@@
 Text GLabel 4200 3900 2    60   Input ~ 0
 PRECHARGE_N
-$Comp
-L D_Zener D?
-U 1 1 5B1245DC
-P 3100 4250
-F 0 "D?" H 3100 4350 50  0000 C CNN
-F 1 "DZ2W03600L" H 3100 4150 50  0000 C CNN
-F 2 "" H 3100 4250 50  0001 C CNN
-F 3 "" H 3100 4250 50  0001 C CNN
-	1    3100 4250
-	0    1    1    0
-$EndComp
 Wire Wire Line
 	3250 1200 4600 1200
@@
 Wire Wire Line
 	3100 4650 3100 4400
-$Comp
-L C C?
-U 1 1 5B1248DC
-P 3700 4300
-F 0 "C?" H 3725 4400 50  0000 L CNN
-F 1 "10nF" H 3725 4200 50  0000 L CNN
-F 2 "" H 3738 4150 50  0001 C CNN
-F 3 "" H 3700 4300 50  0001 C CNN
-	1    3700 4300
-	1    0    0    -1
-$EndComp
 Wire Wire Line
 	3700 4150 3700 3900
@@
 Wire Wire Line
 	3700 4650 3700 4450
-$Comp
-L D_Zener D?
-U 1 1 5B124AA1
-P 3100 3600
-F 0 "D?" H 3100 3700 50  0000 C CNN
-F 1 "DZ2W03600L" H 3100 3500 50  0000 C CNN
-F 2 "" H 3100 3600 50  0001 C CNN
-F 3 "" H 3100 3600 50  0001 C CNN
-	1    3100 3600
-	0    1    1    0
-$EndComp
 $Comp
 L +5V #PWR?
@@
 Text GLabel 8150 1850 2    60   Input ~ 0
 PACK_A_ON
-$Comp
-L D_Zener D?
-U 1 1 5B125182
-P 7050 2200
-F 0 "D?" H 7050 2300 50  0000 C CNN
-F 1 "DZ2W03600L" H 7050 2100 50  0000 C CNN
-F 2 "" H 7050 2200 50  0001 C CNN
-F 3 "" H 7050 2200 50  0001 C CNN
-	1    7050 2200
-	0    1    1    0
-$EndComp
 Wire Wire Line
 	6700 1850 8150 1850
@@
 F 0 "C?" H 7675 2350 50  0000 L CNN
 F 1 "10nF" H 7675 2150 50  0000 L CNN
-F 2 "" H 7688 2100 50  0001 C CNN
-F 3 "" H 7650 2250 50  0001 C CNN
+F 2 "Capacitors_SMD:C_0402" H 7688 2100 50  0001 C CNN
+F 3 "https://www.digikey.com/product-detail/en/murata-electronics-north-america/GRM155R71C103KA01D/490-1313-1-ND/587926" H 7650 2250 50  0001 C CNN
 	1    7650 2250
 	1    0    0    -1
@@
 Wire Wire Line
 	7650 2600 7650 2400
-$Comp
-L D_Zener D?
-U 1 1 5B1251A5
-P 7050 1550
-F 0 "D?" H 7050 1650 50  0000 C CNN
-F 1 "DZ2W03600L" H 7050 1450 50  0000 C CNN
-F 2 "" H 7050 1550 50  0001 C CNN
-F 3 "" H 7050 1550 50  0001 C CNN
-	1    7050 1550
-	0    1    1    0
-$EndComp
 $Comp
 L +5V #PWR?
@@
 Text GLabel 8150 3900 2    60   Input ~ 0
 PACK_B_ON
-$Comp
-L D_Zener D?
-U 1 1 5B12529D
-P 7050 4250
-F 0 "D?" H 7050 4350 50  0000 C CNN
-F 1 "DZ2W03600L" H 7050 4150 50  0000 C CNN
-F 2 "" H 7050 4250 50  0001 C CNN
-F 3 "" H 7050 4250 50  0001 C CNN
-	1    7050 4250
-	0    1    1    0
-$EndComp
 Wire Wire Line
 	6700 3900 8150 3900
@@
 Wire Wire Line
 	7050 4650 7050 4400
-$Comp
-L C C?
-U 1 1 5B1252B0
-P 7650 4300
-F 0 "C?" H 7675 4400 50  0000 L CNN
-F 1 "10nF" H 7675 4200 50  0000 L CNN
-F 2 "" H 7688 4150 50  0001 C CNN
-F 3 "" H 7650 4300 50  0001 C CNN
-	1    7650 4300
-	1    0    0    -1
-$EndComp
 Wire Wire Line
 	7650 4150 7650 3900
@@
 Wire Wire Line
 	7650 4650 7650 4450
-$Comp
-L D_Zener D?
-U 1 1 5B1252C0
-P 7050 3600
-F 0 "D?" H 7050 3700 50  0000 C CNN
-F 1 "DZ2W03600L" H 7050 3500 50  0000 C CNN
-F 2 "" H 7050 3600 50  0001 C CNN
-F 3 "" H 7050 3600 50  0001 C CNN
-	1    7050 3600
-	0    1    1    0
-$EndComp
 $Comp
 L +5V #PWR?
@@
 	3750 6050 3200 6050
 Connection ~ 3200 6050
+$Comp
+L D_Zener D?
+U 1 1 5B1245DC
+P 3100 4250
+F 0 "D?" H 3100 4350 50  0000 C CNN
+F 1 "DZ2W03600L" H 3100 4150 50  0000 C CNN
+F 2 "Diodes_SMD:D_1206" H 3100 4250 50  0001 C CNN
+F 3 "https://industrial.panasonic.com/content/data/SC/ds/ds4/DZ2W03600L_E.pdf" H 3100 4250 50  0001 C CNN
+	1    3100 4250
+	0    1    1    0
+$EndComp
+$Comp
+L D_Zener D?
+U 1 1 5B29E487
+P 7050 4250
+F 0 "D?" H 7050 4350 50  0000 C CNN
+F 1 "DZ2W03600L" H 7050 4150 50  0000 C CNN
+F 2 "Diodes_SMD:D_1206" H 7050 4250 50  0001 C CNN
+F 3 "https://industrial.panasonic.com/content/data/SC/ds/ds4/DZ2W03600L_E.pdf" H 7050 4250 50  0001 C CNN
+	1    7050 4250
+	0    1    1    0
+$EndComp
+$Comp
+L D_Zener D?
+U 1 1 5B29E4E1
+P 7050 2200
+F 0 "D?" H 7050 2300 50  0000 C CNN
+F 1 "DZ2W03600L" H 7050 2100 50  0000 C CNN
+F 2 "Diodes_SMD:D_1206" H 7050 2200 50  0001 C CNN
+F 3 "https://industrial.panasonic.com/content/data/SC/ds/ds4/DZ2W03600L_E.pdf" H 7050 2200 50  0001 C CNN
+	1    7050 2200
+	0    1    1    0
+$EndComp
+$Comp
+L D_Zener D?
+U 1 1 5B29E546
+P 3100 3600
+F 0 "D?" H 3100 3700 50  0000 C CNN
+F 1 "DZ2W03600L" H 3100 3500 50  0000 C CNN
+F 2 "Diodes_SMD:D_1206" H 3100 3600 50  0001 C CNN
+F 3 "https://industrial.panasonic.com/content/data/SC/ds/ds4/DZ2W03600L_E.pdf" H 3100 3600 50  0001 C CNN
+	1    3100 3600
+	0    1    1    0
+$EndComp
+$Comp
+L D_Zener D?
+U 1 1 5B29E588
+P 7050 3600
+F 0 "D?" H 7050 3700 50  0000 C CNN
+F 1 "DZ2W03600L" H 7050 3500 50  0000 C CNN
+F 2 "Diodes_SMD:D_1206" H 7050 3600 50  0001 C CNN
+F 3 "https://industrial.panasonic.com/content/data/SC/ds/ds4/DZ2W03600L_E.pdf" H 7050 3600 50  0001 C CNN
+	1    7050 3600
+	0    1    1    0
+$EndComp
+$Comp
+L D_Zener D?
+U 1 1 5B29E5FF
+P 7050 1550
+F 0 "D?" H 7050 1650 50  0000 C CNN
+F 1 "DZ2W03600L" H 7050 1450 50  0000 C CNN
+F 2 "Diodes_SMD:D_1206" H 7050 1550 50  0001 C CNN
+F 3 "https://industrial.panasonic.com/content/data/SC/ds/ds4/DZ2W03600L_E.pdf" H 7050 1550 50  0001 C CNN
+	1    7050 1550
+	0    1    1    0
+$EndComp
+$Comp
+L C C?
+U 1 1 5B29E6BD
+P 7650 4300
+F 0 "C?" H 7675 4400 50  0000 L CNN
+F 1 "10nF" H 7675 4200 50  0000 L CNN
+F 2 "Capacitors_SMD:C_0402" H 7688 4150 50  0001 C CNN
+F 3 "https://www.digikey.com/product-detail/en/murata-electronics-north-america/GRM155R71C103KA01D/490-1313-1-ND/587926" H 7650 4300 50  0001 C CNN
+	1    7650 4300
+	1    0    0    -1
+$EndComp
+$Comp
+L C C?
+U 1 1 5B29E73C
+P 3700 4300
+F 0 "C?" H 3725 4400 50  0000 L CNN
+F 1 "10nF" H 3725 4200 50  0000 L CNN
+F 2 "Capacitors_SMD:C_0402" H 3738 4150 50  0001 C CNN
+F 3 "https://www.digikey.com/product-detail/en/murata-electronics-north-america/GRM155R71C103KA01D/490-1313-1-ND/587926" H 3700 4300 50  0001 C CNN
+	1    3700 4300
+	1    0    0    -1
+$EndComp
 $EndSCHEMATC

Commit message: All footprints added for gen 1 battery board
Woot. Layout soon!!!
Parts:
- D?: footprint (none) -> Diodes_SMD:D_SMA
Changed lines of the file:
@@
 F 0 "D?" H 4300 1650 50  0000 C CNN
 F 1 "SMAJ36CA" H 4300 1450 50  0000 C CNN
-F 2 "" H 4300 1550 50  0001 C CNN
-F 3 "" H 4300 1550 50  0001 C CNN
+F 2 "Diodes_SMD:D_SMA" H 4300 1550 50  0001 C CNN
+F 3 "http://www.littelfuse.com/~/media/electronics/datasheets/tvs_diodes/littelfuse_tvs_diode_smaj_datasheet.pdf.pdf" H 4300 1550 50  0001 C CNN
 	1    4300 1550
 	0    1    1    0
 $EndComp
 $Comp
-L GND #PWR?
+L GND #PWR023
 U 1 1 5B11F8FB
 P 4300 1950
-F 0 "#PWR?" H 4300 1700 50  0001 C CNN
+F 0 "#PWR023" H 4300 1700 50  0001 C CNN
 F 1 "GND" H 4300 1800 50  0000 C CNN
 F 2 "" H 4300 1950 50  0001 C CNN
@@
 Connection ~ 3100 3900
 $Comp
-L GND #PWR?
+L GND #PWR024
 U 1 1 5B12464E
 P 3100 4650
-F 0 "#PWR?" H 3100 4400 50  0001 C CNN
+F 0 "#PWR024" H 3100 4400 50  0001 C CNN
 F 1 "GND" H 3100 4500 50  0000 C CNN
 F 2 "" H 3100 4650 50  0001 C CNN
@@
 Connection ~ 3750 3900
 $Comp
-L GND #PWR?
+L GND #PWR025
 U 1 1 5B124921
 P 3700 4650
-F 0 "#PWR?" H 3700 4400 50  0001 C CNN
+F 0 "#PWR025" H 3700 4400 50  0001 C CNN
 F 1 "GND" H 3700 4500 50  0000 C CNN
 F 2 "" H 3700 4650 50  0001 C CNN
@@
 	3700 4650 3700 4450
 $Comp
-L +5V #PWR?
+L +5V #PWR026
 U 1 1 5B124B04
 P 3100 3350
-F 0 "#PWR?" H 3100 3200 50  0001 C CNN
+F 0 "#PWR026" H 3100 3200 50  0001 C CNN
 F 1 "+5V" H 3100 3490 50  0000 C CNN
 F 2 "" H 3100 3350 50  0001 C CNN
@@
 Connection ~ 7050 1850
 $Comp
-L GND #PWR?
+L GND #PWR027
 U 1 1 5B12518E
 P 7050 2600
-F 0 "#PWR?" H 7050 2350 50  0001 C CNN
+F 0 "#PWR027" H 7050 2350 50  0001 C CNN
 F 1 "GND" H 7050 2450 50  0000 C CNN
 F 2 "" H 7050 2600 50  0001 C CNN
@@
 Connection ~ 7700 1850
 $Comp
-L GND #PWR?
+L GND #PWR028
 U 1 1 5B12519E
 P 7650 2600
-F 0 "#PWR?" H 7650 2350 50  0001 C CNN
+F 0 "#PWR028" H 7650 2350 50  0001 C CNN
 F 1 "GND" H 7650 2450 50  0000 C CNN
 F 2 "" H 7650 2600 50  0001 C CNN
@@
 	7650 2600 7650 2400
 $Comp
-L +5V #PWR?
+L +5V #PWR029
 U 1 1 5B1251AB
 P 7050 1300
-F 0 "#PWR?" H 7050 1150 50  0001 C CNN
+F 0 "#PWR029" H 7050 1150 50  0001 C CNN
 F 1 "+5V" H 7050 1440 50  0000 C CNN
 F 2 "" H 7050 1300 50  0001 C CNN
@@
 Connection ~ 7050 3900
 $Comp
-L GND #PWR?
+L GND #PWR030
 U 1 1 5B1252A9
 P 7050 4650
-F 0 "#PWR?" H 7050 4400 50  0001 C CNN
+F 0 "#PWR030" H 7050 4400 50  0001 C CNN
 F 1 "GND" H 7050 4500 50  0000 C CNN
 F 2 "" H 7050 4650 50  0001 C CNN
@@
 Connection ~ 7700 3900
 $Comp
-L GND #PWR?
+L GND #PWR031
 U 1 1 5B1252B9
 P 7650 4650
-F 0 "#PWR?" H 7650 4400 50  0001 C CNN
+F 0 "#PWR031" H 7650 4400 50  0001 C CNN
 F 1 "GND" H 7650 4500 50  0000 C CNN
 F 2 "" H 7650 4650 50  0001 C CNN
@@
 	7650 4650 7650 4450
 $Comp
-L +5V #PWR?
+L +5V #PWR032
 U 1 1 5B1252C6
 P 7050 3350
-F 0 "#PWR?" H 7050 3200 50  0001 C CNN
+F 0 "#PWR032" H 7050 3200 50  0001 C CNN
 F 1 "+5V" H 7050 3490 50  0000 C CNN
 F 2 "" H 7050 3350 50  0001 C CNN
@@
 	7050 3450 7050 3350
 $Comp
-L GND #PWR?
+L GND #PWR033
 U 1 1 5B120B55
 P 3200 6600
-F 0 "#PWR?" H 3200 6350 50  0001 C CNN
+F 0 "#PWR033" H 3200 6350 50  0001 C CNN
 F 1 "GND" H 3200 6450 50  0000 C CNN
 F 2 "" H 3200 6600 50  0001 C CNN
