File: Node/usb_sub.sch (KiCad schematic (older format))
At the start: 8 parts, among them J1601 Conn_02x03_Odd_Even, J1602 USB_B_Micro, J2201 Conn_02x05_Odd_Even

Commit message: Generated BOM, filled out part numbers for precision resistors and headers.
Parts:
- J1601: MFG. P/N (none) -> GRPB032VWVN-RC; Manufacturer (none) -> Sullins Conn. Solutions; Vendor (none) -> DigiKey; Vendor P/N (none) -> S9015E-03-ND
- J2201: MFG. P/N (none) -> 20021111-00010T4LF; Manufacturer (none) -> Amphenol FCI; Vendor (none) -> DigiKey; Vendor P/N (none) -> 609-3712-ND
Changed lines of the file:
@@
 EESchema Schematic File Version 2
 LIBS:hyper_capstone
+LIBS:Connector
 LIBS:node-cache
 EELAYER 25 0
@@
 ISP_RESET_L
 $Comp
-L +5V #PWR2103
+L +5V #PWR0212
 U 1 1 59F2693E
 P 3250 3700
-F 0 "#PWR2103" H 3250 3550 60  0001 C CNN
+F 0 "#PWR0212" H 3250 3550 60  0001 C CNN
 F 1 "+5V" H 3250 3840 60  0000 C CNN
 F 2 "" H 3250 3700 60  0000 C CNN
@@
 ISP_MOSI
 $Comp
-L GND #PWR2104
+L GND #PWR0213
 U 1 1 59F26978
 P 3250 4150
-F 0 "#PWR2104" H 3250 3900 60  0001 C CNN
+F 0 "#PWR0213" H 3250 3900 60  0001 C CNN
 F 1 "GND" H 3250 4000 60  0000 C CNN
 F 2 "" H 3250 4150 60  0000 C CNN
@@
 5V0_USB
 $Comp
-L GND #PWR2101
+L GND #PWR0214
 U 1 1 59F26F68
 P 3500 2350
-F 0 "#PWR2101" H 3500 2100 60  0001 C CNN
+F 0 "#PWR0214" H 3500 2100 60  0001 C CNN
 F 1 "GND" H 3500 2200 60  0000 C CNN
 F 2 "" H 3500 2350 60  0000 C CNN
@@
 F 2 "Pin_Headers:Pin_Header_Straight_2x03_Pitch2.54mm" H 2750 3950 50  0001 C CNN
 F 3 "" H 2750 3950 50  0001 C CNN
+F 4 "Sullins Conn. Solutions" H 2750 3950 60  0001 C CNN "Manufacturer"
+F 5 "GRPB032VWVN-RC" H 2750 3950 60  0001 C CNN "MFG. P/N"
+F 6 "DigiKey" H 2750 3950 60  0001 C CNN "Vendor"
+F 7 "S9015E-03-ND" H 2750 3950 60  0001 C CNN "Vendor P/N"
 	1    2750 3950
 	1    0    0    -1
@@
 F 2 "Pin_Headers:Pin_Header_Straight_2x05_Pitch1.27mm" H 1700 5250 50  0001 C CNN
 F 3 "" H 1700 5250 50  0001 C CNN
+F 4 "Amphenol FCI" H 1700 5250 60  0001 C CNN "Manufacturer"
+F 5 "20021111-00010T4LF" H 1700 5250 60  0001 C CNN "MFG. P/N"
+F 6 "DigiKey" H 1700 5250 60  0001 C CNN "Vendor"
+F 7 "609-3712-ND" H 1700 5250 60  0001 C CNN "Vendor P/N"
 	1    1700 5250
 	1    0    0    -1
@@
 	1350 5050 1350 4900
 $Comp
-L +3V3 #PWR2105
+L +3V3 #PWR0215
 U 1 1 5A127439
 P 1350 4900
-F 0 "#PWR2105" H 1350 4750 50  0001 C CNN
+F 0 "#PWR0215" H 1350 4750 50  0001 C CNN
 F 1 "+3V3" H 1350 5040 50  0000 C CNN
 F 2 "" H 1350 4900 50  0001 C CNN
@@
 Connection ~ 1350 5250
 $Comp
-L GND #PWR2106
+L GND #PWR0216
 U 1 1 5A1277C9
 P 1350 5550
-F 0 "#PWR2106" H 1350 5300 60  0001 C CNN
+F 0 "#PWR0216" H 1350 5300 60  0001 C CNN
 F 1 "GND" H 1350 5400 60  0000 C CNN
 F 2 "" H 1350 5550 60  0000 C CNN
@@
 Connection ~ 3900 2700
 $Comp
-L GND #PWR2102
+L GND #PWR0217
 U 1 1 5A0DC47F
 P 3900 2750
-F 0 "#PWR2102" H 3900 2500 60  0001 C CNN
+F 0 "#PWR0217" H 3900 2500 60  0001 C CNN
 F 1 "GND" H 3900 2600 60  0000 C CNN
 F 2 "" H 3900 2750 60  0000 C CNN

Commit message: Ghost train
Parts:
- C2201: symbol C -> node-rescue:C
- F1601: symbol Fuse -> node-rescue:Fuse
- J1601: symbol Conn_02x03_Odd_Even -> node-rescue:Conn_02x03_Odd_Even
- J1602: symbol USB_B_Micro -> Connector:USB_B_Micro
- J2201: symbol Conn_02x05_Odd_Even -> node-rescue:Conn_02x05_Odd_Even
- R2201: symbol R -> node-rescue:R
- VR1601, VR1602: symbol Varistor -> node-rescue:Varistor
Changed lines of the file:
@@
-EESchema Schematic File Version 2
-LIBS:hyper_capstone
+EESchema Schematic File Version 4
 LIBS:node-cache
-EELAYER 25 0
+EELAYER 26 0
 EELAYER END
 $Descr A4 11693 8268
@@
 ISP_RESET_L
 $Comp
-L +5V #PWR0212
+L node-rescue:+5V #PWR0212
 U 1 1 59F2693E
 P 3250 3700
@@
 ISP_MOSI
 $Comp
-L GND #PWR0213
+L node-rescue:GND #PWR0213
 U 1 1 59F26978
 P 3250 4150
@@
 5V0_USB
 $Comp
-L GND #PWR0214
+L node-rescue:GND #PWR0214
 U 1 1 59F26F68
 P 3500 2350
@@
 	1300 1500 2350 1500
 $Comp
-L Varistor VR1601
+L node-rescue:Varistor VR1601
 U 1 1 59F27E85
 P 2000 2250
@@
 $EndComp
 $Comp
-L Varistor VR1602
+L node-rescue:Varistor VR1602
 U 1 1 59F28073
 P 2250 2250
@@
 Connection ~ 2250 1900
 $Comp
-L Conn_02x03_Odd_Even J1601
+L node-rescue:Conn_02x03_Odd_Even J1601
 U 1 1 5A0B6EC5
 P 2750 3950
@@
 $EndComp
 $Comp
-L USB_B_Micro J1602
+L Connector:USB_B_Micro J1602
 U 1 1 5A0B6F70
 P 3500 1800
@@
 $EndComp
 $Comp
-L Fuse F1601
+L node-rescue:Fuse F1601
 U 1 1 5A0B6FF5
 P 2500 1500
@@
 SWD_S[0..2]
 $Comp
-L Conn_02x05_Odd_Even J2201
+L node-rescue:Conn_02x05_Odd_Even J2201
 U 1 1 5A127060
 P 1700 5250
@@
 	1350 5050 1350 4900
 $Comp
-L +3V3 #PWR0215
+L node-rescue:+3V3 #PWR0215
 U 1 1 5A127439
 P 1350 4900
@@
 Connection ~ 1350 5250
 $Comp
-L GND #PWR0216
+L node-rescue:GND #PWR0216
 U 1 1 5A1277C9
 P 1350 5550
@@
 	3600 2250 4350 2250
 $Comp
-L C C2201
+L node-rescue:C C2201
 U 1 1 5A0DC278
 P 3900 2450
@@
 $EndComp
 $Comp
-L R R2201
+L node-rescue:R R2201
 U 1 1 5A0DC2A8
 P 4350 2450
@@
 Connection ~ 3900 2700
 $Comp
-L GND #PWR0217
+L node-rescue:GND #PWR0217
 U 1 1 5A0DC47F
 P 3900 2750
