File: Node/Current_Sense.sch (KiCad schematic (older format))
At the start: 34 parts, among them J1001 Conn_01x03, J1002 Conn_01x03, J1003 Conn_01x03, J1004 Conn_01x03, U1001 LM358, U1002 LM358

Commit message: Added ADC
Parts:
- C1001, C1002, C1003, C1004: symbol C -> node-rescue:C
- J1001, J1002, J1003, J1004: symbol Conn_01x03 -> node-rescue:Conn_01x03
- R1001, R1002, R1003, R1004, R1005, R1006, R1007, R1008, R1009, R1010, R1011, R1012, R1013, R1014, R1015, R1016, R1017, R1018, R1019, R1020, R1021, R1022, R1023, R1024: symbol R -> node-rescue:R
- U1001, U1002: symbol LM358 -> node-rescue:LM358
Changed lines of the file:
@@
-EESchema Schematic File Version 2
-LIBS:hyper_capstone
+EESchema Schematic File Version 4
 LIBS:node-cache
-EELAYER 25 0
+EELAYER 26 0
 EELAYER END
 $Descr A4 11693 8268
@@
 out_1
 $Comp
-L R R1005
+L node-rescue:R R1005
 U 1 1 59F12C7E
 P 2200 1800
@@
 $EndComp
 $Comp
-L Conn_01x03 J1001
+L node-rescue:Conn_01x03 J1001
 U 1 1 59F12EE2
 P 1150 1500
@@
 $EndComp
 $Comp
-L LM358 U1001
+L node-rescue:LM358 U1001
 U 1 1 59F15A26
 P 3300 1600
@@
 $EndComp
 $Comp
-L +5V #PWR082
+L node-rescue:+5V #PWR082
 U 1 1 5A0B8F0B
 P 1450 1250
@@
 $EndComp
 $Comp
-L GND #PWR083
+L node-rescue:GND #PWR083
 U 1 1 5A0B9017
 P 1450 1750
@@
 $EndComp
 $Comp
-L GND #PWR084
+L node-rescue:GND #PWR084
 U 1 1 5A0B9199
 P 2200 2000
@@
 $EndComp
 $Comp
-L R R1017
+L node-rescue:R R1017
 U 1 1 5A0BA528
 P 3500 2000
@@
 $EndComp
 $Comp
-L R R1013
+L node-rescue:R R1013
 U 1 1 5A0BA601
 P 2750 2000
@@
 $EndComp
 $Comp
-L GND #PWR085
+L node-rescue:GND #PWR085
 U 1 1 5A0BABD3
 P 3200 2100
@@
 $EndComp
 $Comp
-L +5V #PWR086
+L node-rescue:+5V #PWR086
 U 1 1 5A0BB106
 P 2500 1850
@@
 $EndComp
 $Comp
-L +5V #PWR087
+L node-rescue:+5V #PWR087
 U 1 1 5A0BB212
 P 3200 1200
@@
 $EndComp
 $Comp
-L R R1001
+L node-rescue:R R1001
 U 1 1 5A0BBB86
 P 1850 1500
@@
 $EndComp
 $Comp
-L R R1009
+L node-rescue:R R1009
 U 1 1 5A0BC1EB
 P 2650 850
@@
 Stuff bypass 0Ω and unstuff series 0Ωs\nconverts to normal 0-5V input
 $Comp
-L R R1021
+L node-rescue:R R1021
 U 1 1 5A0BCADB
 P 4050 1600
@@
 	1350 1500 1700 1500
 $Comp
-L C C1001
+L node-rescue:C C1001
 U 1 1 5A0BD6E2
 P 4450 1900
@@
 	4450 2050 4450 2150
 $Comp
-L GND #PWR088
+L node-rescue:GND #PWR088
 U 1 1 5A0BD766
 P 4450 2150
@@
 out_2
 $Comp
-L R R1006
+L node-rescue:R R1006
 U 1 1 5A0BE9DC
 P 2200 3500
@@
 $EndComp
 $Comp
-L LM358 U1001
+L node-rescue:LM358 U1001
 U 2 1 5A0BE9EE
 P 3300 3300
@@
 $EndComp
 $Comp
-L +5V #PWR089
+L node-rescue:+5V #PWR089
 U 1 1 5A0BE9F4
 P 1450 2950
@@
 $EndComp
 $Comp
-L GND #PWR090
+L node-rescue:GND #PWR090
 U 1 1 5A0BE9FA
 P 1450 3450
@@
 $EndComp
 $Comp
-L GND #PWR091
+L node-rescue:GND #PWR091
 U 1 1 5A0BEA00
 P 2200 3700
@@
 $EndComp
 $Comp
-L R R1018
+L node-rescue:R R1018
 U 1 1 5A0BEA06
 P 3500 3700
@@
 $EndComp
 $Comp
-L R R1014
+L node-rescue:R R1014
 U 1 1 5A0BEA0C
 P 2750 3700
@@
 $EndComp
 $Comp
-L GND #PWR092
+L node-rescue:GND #PWR092
 U 1 1 5A0BEA12
 P 3200 3800
@@
 $EndComp
 $Comp
-L +5V #PWR093
+L node-rescue:+5V #PWR093
 U 1 1 5A0BEA18
 P 2500 3550
@@
 $EndComp
 $Comp
-L +5V #PWR094
+L node-rescue:+5V #PWR094
 U 1 1 5A0BEA1E
 P 3200 2900
@@
 $EndComp
 $Comp
-L R R1002
+L node-rescue:R R1002
 U 1 1 5A0BEA24
 P 1850 3200
@@
 $EndComp
 $Comp
-L R R1010
+L node-rescue:R R1010
 U 1 1 5A0BEA2A
 P 2650 2550
@@
 $EndComp
 $Comp
-L R R1022
+L node-rescue:R R1022
 U 1 1 5A0BEA30
 P 4050 3300
@@
 	1350 3200 1700 3200
 $Comp
-L C C1002
+L node-rescue:C C1002
 U 1 1 5A0BEA52
 P 4450 3600
@@
 	4450 3750 4450 3850
 $Comp
-L GND #PWR095
+L node-rescue:GND #PWR095
 U 1 1 5A0BEA5B
 P 4450 3850
@@
 out_3
 $Comp
-L R R1007
+L node-rescue:R R1007
 U 1 1 5A0BEC63
 P 2200 5200
@@
 $EndComp
 $Comp
-L LM358 U1002
+L node-rescue:LM358 U1002
 U 1 1 5A0BEC75
 P 3300 5000
@@
 $EndComp
 $Comp
-L +5V #PWR096
+L node-rescue:+5V #PWR096
 U 1 1 5A0BEC7B
 P 1450 4650
@@
 $EndComp
 $Comp
-L GND #PWR097
+L node-rescue:GND #PWR097
 U 1 1 5A0BEC81
 P 1450 5150
@@
 $EndComp
 $Comp
-L GND #PWR098
+L node-rescue:GND #PWR098
 U 1 1 5A0BEC87
 P 2200 5400
@@
 $EndComp
 $Comp
-L R R1019
+L node-rescue:R R1019
 U 1 1 5A0BEC8D
 P 3500 5400
@@
 $EndComp
 $Comp
-L R R1015
+L node-rescue:R R1015
 U 1 1 5A0BEC93
 P 2750 5400
@@
 $EndComp
 $Comp
-L GND #PWR099
+L node-rescue:GND #PWR099
 U 1 1 5A0BEC99
 P 3200 5500
@@
 $EndComp
 $Comp
-L +5V #PWR0100
+L node-rescue:+5V #PWR0100
 U 1 1 5A0BEC9F
 P 2500 5250
@@
 $EndComp
 $Comp
-L +5V #PWR0101
+L node-rescue:+5V #PWR0101
 U 1 1 5A0BECA5
 P 3200 4600
@@
 $EndComp
 $Comp
-L R R1003
+L node-rescue:R R1003
 U 1 1 5A0BECAB
 P 1850 4900
@@
 $EndComp
 $Comp
-L R R1011
+L node-rescue:R R1011
 U 1 1 5A0BECB1
 P 2650 4250
@@
 $EndComp
 $Comp
-L R R1023
+L node-rescue:R R1023
 U 1 1 5A0BECB7
 P 4050 5000
@@
 	1350 4900 1700 4900
 $Comp
-L C C1003
+L node-rescue:C C1003
 U 1 1 5A0BECD9
 P 4450 5300
@@
 	4450 5450 4450 5550
 $Comp
-L GND #PWR0102
+L node-rescue:GND #PWR0102
 U 1 1 5A0BECE2
 P 4450 5550
@@
 out_4
 $Comp
-L R R1008
+L node-rescue:R R1008
 U 1 1 5A0BF06D
 P 2200 6950
@@
 $EndComp
 $Comp
-L LM358 U1002
+L node-rescue:LM358 U1002
 U 2 1 5A0BF07F
 P 3300 6750
@@
 $EndComp
 $Comp
-L +5V #PWR0103
+L node-rescue:+5V #PWR0103
 U 1 1 5A0BF085
 P 1450 6400
@@
 $EndComp
 $Comp
-L GND #PWR0104
+L node-rescue:GND #PWR0104
 U 1 1 5A0BF08B
 P 1450 6900
@@
 $EndComp
 $Comp
-L GND #PWR0105
+L node-rescue:GND #PWR0105
 U 1 1 5A0BF091
 P 2200 7150
@@
 $EndComp
 $Comp
-L R R1020
+L node-rescue:R R1020
 U 1 1 5A0BF097
 P 3500 7150
@@
 $EndComp
 $Comp
-L R R1016
+L node-rescue:R R1016
 U 1 1 5A0BF09D
 P 2750 7150
@@
 $EndComp
 $Comp
-L GND #PWR0106
+L node-rescue:GND #PWR0106
 U 1 1 5A0BF0A3
 P 3200 7250
@@
 $EndComp
 $Comp
-L +5V #PWR0107
+L node-rescue:+5V #PWR0107
 U 1 1 5A0BF0A9
 P 2500 7000
@@
 $EndComp
 $Comp
-L +5V #PWR0108
+L node-rescue:+5V #PWR0108
 U 1 1 5A0BF0AF
 P 3200 6350
@@
 $EndComp
 $Comp
-L R R1004
+L node-rescue:R R1004
 U 1 1 5A0BF0B5
 P 1850 6650
@@
 $EndComp
 $Comp
-L R R1012
+L node-rescue:R R1012
 U 1 1 5A0BF0BB
 P 2650 6000
@@
 $EndComp
 $Comp
-L R R1024
+L node-rescue:R R1024
 U 1 1 5A0BF0C1
 P 4050 6750
@@
 	1350 6650 1700 6650
 $Comp
-L C C1004
+L node-rescue:C C1004
 U 1 1 5A0BF0E3
 P 4450 7050
@@
 	4450 7200 4450 7300
 $Comp
-L GND #PWR0109
+L node-rescue:GND #PWR0109
 U 1 1 5A0BF0EC
 P 4450 7300
@@
 Operating equation:\nV_out = 1.25 * (I_in*250Ω - 1V)
 $Comp
-L Conn_01x03 J1002
+L node-rescue:Conn_01x03 J1002
 U 1 1 5A0B6D0A
 P 1150 3200
@@
 $EndComp
 $Comp
-L Conn_01x03 J1003
+L node-rescue:Conn_01x03 J1003
 U 1 1 5A0B6DEF
 P 1150 4900
@@
 $EndComp
 $Comp
-L Conn_01x03 J1004
+L node-rescue:Conn_01x03 J1004
 U 1 1 5A0B6E86
 P 1150 6650
