File: Node/Thermocouple_to_analog.sch (KiCad schematic (older format))
At the start: 9 parts, among them U1301 AD849X

Commit message: Added ADC
Parts:
- C1305, C1306, C1307, C1308: symbol C -> node-rescue:C
- R1305, R1306, R1307, R1308: symbol R -> node-rescue:R
- U1301: symbol AD849X -> node-rescue:AD849X
Changed lines of the file:
@@
-EESchema Schematic File Version 2
-LIBS:hyper_capstone
+EESchema Schematic File Version 4
 LIBS:node-cache
-EELAYER 25 0
+EELAYER 26 0
 EELAYER END
 $Descr A4 11693 8268
 encoding utf-8
-Sheet 17 22
+Sheet 13 22
 Title "Node Board"
 Date ""
@@
 $EndDescr
 $Comp
-L C C1306
+L node-rescue:C C1306
 U 1 1 5A0A32E6
 P 4050 3350
@@
 AR Path="/59C995CB/59DBAF6F/5A0A51C2/5A0A32E6" Ref="C1709"  Part="1"
 AR Path="/59C995CB/59DBAF6F/5A0A51C8/5A0A32E6" Ref="C1802"  Part="1"
-F 0 "C1802" H 4075 3450 50  0000 L CNN
+F 0 "C1306" H 4075 3450 50  0000 L CNN
 F 1 "1uF" H 4075 3250 50  0000 L CNN
 F 2 "Capacitors_SMD:C_0805_HandSoldering" H 4088 3200 50  0001 C CNN
@@
 $EndComp
 $Comp
-L C C1305
+L node-rescue:C C1305
 U 1 1 5A0A32EE
 P 4050 3000
@@
 AR Path="/59C995CB/59DBAF6F/5A0A51C2/5A0A32EE" Ref="C1708"  Part="1"
 AR Path="/59C995CB/59DBAF6F/5A0A51C8/5A0A32EE" Ref="C1801"  Part="1"
-F 0 "C1801" H 4075 3100 50  0000 L CNN
+F 0 "C1305" H 4075 3100 50  0000 L CNN
 F 1 "0.1uF" H 4075 2900 50  0000 L CNN
 F 2 "Capacitors_SMD:C_0805_HandSoldering" H 4088 2850 50  0001 C CNN
@@
 $EndComp
 $Comp
-L C C1307
+L node-rescue:C C1307
 U 1 1 5A0A32F6
 P 4050 3750
@@
 AR Path="/59C995CB/59DBAF6F/5A0A51C2/5A0A32F6" Ref="C1710"  Part="1"
 AR Path="/59C995CB/59DBAF6F/5A0A51C8/5A0A32F6" Ref="C1803"  Part="1"
-F 0 "C1803" H 4075 3850 50  0000 L CNN
+F 0 "C1307" H 4075 3850 50  0000 L CNN
 F 1 "0.1uF" H 4075 3650 50  0000 L CNN
 F 2 "Capacitors_SMD:C_0805_HandSoldering" H 4088 3600 50  0001 C CNN
@@
 $EndComp
 $Comp
-L GND #PWR0131
+L node-rescue:GND #PWR0131
 U 1 1 5A0A32FD
 P 4050 3900
@@
 AR Path="/59C995CB/59DBAF6F/5A0A51C2/5A0A32FD" Ref="#PWR0155"  Part="1"
 AR Path="/59C995CB/59DBAF6F/5A0A51C8/5A0A32FD" Ref="#PWR0161"  Part="1"
-F 0 "#PWR0161" H 4050 3650 50  0001 C CNN
+F 0 "#PWR0131" H 4050 3650 50  0001 C CNN
 F 1 "GND" H 4050 3750 50  0000 C CNN
 F 2 "" H 4050 3900 50  0000 C CNN
@@
 $EndComp
 $Comp
-L R R1305
+L node-rescue:R R1305
 U 1 1 5A0A3304
 P 3050 2800
@@
 AR Path="/59C995CB/59DBAF6F/5A0A51C2/5A0A3304" Ref="R1703"  Part="1"
 AR Path="/59C995CB/59DBAF6F/5A0A51C8/5A0A3304" Ref="R1801"  Part="1"
-F 0 "R1801" V 3130 2800 50  0000 C CNN
+F 0 "R1305" V 3130 2800 50  0000 C CNN
 F 1 "1M" V 3050 2800 50  0000 C CNN
 F 2 "Resistors_SMD:R_0805_HandSoldering" V 2980 2800 50  0001 C CNN
@@
 $EndComp
 $Comp
-L R R1307
+L node-rescue:R R1307
 U 1 1 5A0A330C
 P 3650 3600
@@
 AR Path="/59C995CB/59DBAF6F/5A0A51C2/5A0A330C" Ref="R1705"  Part="1"
 AR Path="/59C995CB/59DBAF6F/5A0A51C8/5A0A330C" Ref="R1803"  Part="1"
-F 0 "R1803" V 3730 3600 50  0000 C CNN
+F 0 "R1307" V 3730 3600 50  0000 C CNN
 F 1 "150" V 3650 3600 50  0000 C CNN
 F 2 "Resistors_SMD:R_0805_HandSoldering" V 3580 3600 50  0001 C CNN
@@
 +IN
 $Comp
-L GND #PWR0132
+L node-rescue:GND #PWR0132
 U 1 1 5A0A3314
 P 4400 2900
@@
 AR Path="/59C995CB/59DBAF6F/5A0A51C2/5A0A3314" Ref="#PWR0156"  Part="1"
 AR Path="/59C995CB/59DBAF6F/5A0A51C8/5A0A3314" Ref="#PWR0162"  Part="1"
-F 0 "#PWR0162" H 4400 2650 50  0001 C CNN
+F 0 "#PWR0132" H 4400 2650 50  0001 C CNN
 F 1 "GND" H 4400 2750 50  0000 C CNN
 F 2 "" H 4400 2900 50  0000 C CNN
@@
 $EndComp
 $Comp
-L R R1306
+L node-rescue:R R1306
 U 1 1 5A0A331B
 P 3650 3150
@@
 AR Path="/59C995CB/59DBAF6F/5A0A51C2/5A0A331B" Ref="R1704"  Part="1"
 AR Path="/59C995CB/59DBAF6F/5A0A51C8/5A0A331B" Ref="R1802"  Part="1"
-F 0 "R1802" V 3730 3150 50  0000 C CNN
+F 0 "R1306" V 3730 3150 50  0000 C CNN
 F 1 "150" V 3650 3150 50  0000 C CNN
 F 2 "Resistors_SMD:R_0805_HandSoldering" V 3580 3150 50  0001 C CNN
@@
 $EndComp
 $Comp
-L GND #PWR0133
+L node-rescue:GND #PWR0133
 U 1 1 5A0A3322
 P 2750 2700
@@
 AR Path="/59C995CB/59DBAF6F/5A0A51C2/5A0A3322" Ref="#PWR0157"  Part="1"
 AR Path="/59C995CB/59DBAF6F/5A0A51C8/5A0A3322" Ref="#PWR0163"  Part="1"
-F 0 "#PWR0163" H 2750 2450 50  0001 C CNN
+F 0 "#PWR0133" H 2750 2450 50  0001 C CNN
 F 1 "GND" H 2750 2550 50  0000 C CNN
 F 2 "" H 2750 2700 50  0000 C CNN
@@
 -IN
 $Comp
-L GND #PWR0134
+L node-rescue:GND #PWR0134
 U 1 1 5A0A332A
 P 6250 3000
@@
 AR Path="/59C995CB/59DBAF6F/5A0A51C2/5A0A332A" Ref="#PWR0158"  Part="1"
 AR Path="/59C995CB/59DBAF6F/5A0A51C8/5A0A332A" Ref="#PWR0164"  Part="1"
-F 0 "#PWR0164" H 6250 2750 50  0001 C CNN
+F 0 "#PWR0134" H 6250 2750 50  0001 C CNN
 F 1 "GND" H 6250 2850 50  0000 C CNN
 F 2 "" H 6250 3000 50  0000 C CNN
@@
 $EndComp
 $Comp
-L C C1308
+L node-rescue:C C1308
 U 1 1 5A0A3332
 P 6250 2750
@@
 AR Path="/59C995CB/59DBAF6F/5A0A51C2/5A0A3332" Ref="C1711"  Part="1"
 AR Path="/59C995CB/59DBAF6F/5A0A51C8/5A0A3332" Ref="C1804"  Part="1"
-F 0 "C1804" H 6275 2850 50  0000 L CNN
+F 0 "C1308" H 6275 2850 50  0000 L CNN
 F 1 "0.1uF" H 6275 2650 50  0000 L CNN
 F 2 "Capacitors_SMD:C_0805_HandSoldering" H 6288 2600 50  0001 C CNN
@@
 Connection ~ 4050 3600
 Wire Wire Line
-	2900 3600 3500 3600
+	2900 3600 3050 3600
 Wire Wire Line
 	4050 2750 4400 2750
@@
 Connection ~ 4050 3150
 Wire Wire Line
-	2900 3150 3500 3150
+	2900 3150 3050 3150
 Wire Wire Line
 	4400 2750 4400 2900
@@
 	4850 3850 6200 3850
 Wire Wire Line
-	5650 2450 5650 2900
+	5650 2450 5650 2550
 Wire Wire Line
 	5550 2500 5550 2900
@@
 Filter Freq, Diff: 505.2 Hz\nFilter Freq, CM: 10610.3 Hz
 $Comp
-L AD849X U1301
+L node-rescue:AD849X U1301
 U 1 1 5A0A334F
 P 5550 3350
@@
 AR Path="/59C995CB/59DBAF6F/5A0A51C2/5A0A334F" Ref="U1702"  Part="1"
 AR Path="/59C995CB/59DBAF6F/5A0A51C8/5A0A334F" Ref="U1801"  Part="1"
-F 0 "U1801" H 5900 3650 60  0000 C CNN
+F 0 "U1301" H 5900 3650 60  0000 C CNN
 F 1 "AD849X" H 5800 3050 60  0000 C CNN
 F 2 "Housings_SSOP:MSOP-8_3x3mm_Pitch0.65mm" H 5550 3350 60  0001 C CNN
@@
 	3050 2500 3050 2650
 $Comp
-L GND #PWR0135
+L node-rescue:GND #PWR0135
 U 1 1 5A0A335F
 P 5350 2600
@@
 AR Path="/59C995CB/59DBAF6F/5A0A51C2/5A0A335F" Ref="#PWR0159"  Part="1"
 AR Path="/59C995CB/59DBAF6F/5A0A51C8/5A0A335F" Ref="#PWR0165"  Part="1"
-F 0 "#PWR0165" H 5350 2350 50  0001 C CNN
+F 0 "#PWR0135" H 5350 2350 50  0001 C CNN
 F 1 "GND" H 5350 2450 50  0000 C CNN
 F 2 "" H 5350 2600 50  0000 C CNN
@@
 	6250 2550 5650 2550
 $Comp
-L +5V #PWR0136
+L node-rescue:+5V #PWR0136
 U 1 1 5A0A3604
 P 5650 2450
@@
 AR Path="/59C995CB/59DBAF6F/5A0A51C2/5A0A3604" Ref="#PWR0160"  Part="1"
 AR Path="/59C995CB/59DBAF6F/5A0A51C8/5A0A3604" Ref="#PWR0166"  Part="1"
-F 0 "#PWR0166" H 5650 2300 50  0001 C CNN
+F 0 "#PWR0136" H 5650 2300 50  0001 C CNN
 F 1 "+5V" H 5650 2590 50  0000 C CNN
 F 2 "" H 5650 2450 50  0001 C CNN
@@
 Vref_TC
 Wire Wire Line
-	6100 3350 6950 3350
+	6100 3350 6200 3350
 Wire Wire Line
 	6200 3850 6200 3350
@@
 	4850 3250 4850 3150
 Wire Wire Line
-	4850 3150 3800 3150
+	4850 3150 4050 3150
 Wire Wire Line
 	4950 3450 4750 3450
@@
 	4750 3450 4750 3600
 Wire Wire Line
-	4750 3600 3800 3600
+	4750 3600 4050 3600
 Wire Wire Line
 	3050 3600 3050 4350
@@
 Connection ~ 3050 3600
 $Comp
-L R R1308
+L node-rescue:R R1308
 U 1 1 5A0B1DD9
 P 5300 4350
@@
 AR Path="/59C995CB/59DBAF6F/5A0A51C2/5A0B1DD9" Ref="R1706"  Part="1"
 AR Path="/59C995CB/59DBAF6F/5A0A51C8/5A0B1DD9" Ref="R1804"  Part="1"
-F 0 "R1804" V 5380 4350 50  0000 C CNN
+F 0 "R1308" V 5380 4350 50  0000 C CNN
 F 1 "0" V 5300 4350 50  0000 C CNN
 F 2 "Resistors_SMD:R_0805_HandSoldering" V 5230 4350 50  0001 C CNN
@@
 	6550 4350 6550 3350
 Connection ~ 6550 3350
+Wire Wire Line
+	4050 3600 3800 3600
+Wire Wire Line
+	4050 3150 3800 3150
+Wire Wire Line
+	5650 2550 5650 2900
+Wire Wire Line
+	3050 3150 3500 3150
+Wire Wire Line
+	6200 3350 6550 3350
+Wire Wire Line
+	3050 3600 3500 3600
+Wire Wire Line
+	6550 3350 6950 3350
 $EndSCHEMATC
