File: Node/Volt_step_down.sch (KiCad schematic (older format))
At the start: 12 parts, among them J1101 Conn_01x03, J1102 Conn_01x03

Commit message: Added ADC
Parts:
- C1101, C1102: symbol C -> node-rescue:C
- F1101, F1102: symbol Fuse -> node-rescue:Fuse
- J1101, J1102: symbol Conn_01x03 -> node-rescue:Conn_01x03
- R1101, R1102, R1103, R1104, R1105, R1106: symbol R -> node-rescue:R
Changed lines of the file:
@@
-EESchema Schematic File Version 2
-LIBS:hyper_capstone
+EESchema Schematic File Version 4
 LIBS:node-cache
-EELAYER 25 0
+EELAYER 26 0
 EELAYER END
 $Descr A4 11693 8268
@@
 out_2
 $Comp
-L Conn_01x03 J1101
+L node-rescue:Conn_01x03 J1101
 U 1 1 5A0C421B
 P 1200 2700
@@
 $EndComp
 $Comp
-L +5V #PWR0110
+L node-rescue:+5V #PWR0110
 U 1 1 5A0C4553
 P 1600 2050
@@
 $EndComp
 $Comp
-L GND #PWR0111
+L node-rescue:GND #PWR0111
 U 1 1 5A0C4559
 P 1500 2950
@@
 	1500 2800 1500 2950
 $Comp
-L R R1101
+L node-rescue:R R1101
 U 1 1 5A0C458D
 P 1600 2350
@@
 	2150 3600 2150 3700
 $Comp
-L GND #PWR0112
+L node-rescue:GND #PWR0112
 U 1 1 5A0C511D
 P 2150 3700
@@
 $EndComp
 $Comp
-L C C1101
+L node-rescue:C C1101
 U 1 1 5A0C516E
 P 2500 3450
@@
 $EndComp
 $Comp
-L GND #PWR0113
+L node-rescue:GND #PWR0113
 U 1 1 5A0C521E
 P 2500 3700
@@
 Cap for optional\nLPF
 $Comp
-L R R1104
+L node-rescue:R R1104
 U 1 1 5A0C5E78
 P 2150 3450
@@
 $EndComp
 $Comp
-L R R1103
+L node-rescue:R R1103
 U 1 1 5A0C5E9E
 P 2150 2950
@@
 $EndComp
 $Comp
-L Fuse F1101
+L node-rescue:Fuse F1101
 U 1 1 5A0C5F81
 P 2300 2600
@@
 	2600 2600 2450 2600
 $Comp
-L Conn_01x03 J1102
+L node-rescue:Conn_01x03 J1102
 U 1 1 5A0C65D7
 P 1250 5050
@@
 $EndComp
 $Comp
-L +5V #PWR0114
+L node-rescue:+5V #PWR0114
 U 1 1 5A0C65DD
 P 1650 4400
@@
 $EndComp
 $Comp
-L GND #PWR0115
+L node-rescue:GND #PWR0115
 U 1 1 5A0C65E3
 P 1550 5300
@@
 	1550 5150 1550 5300
 $Comp
-L R R1102
+L node-rescue:R R1102
 U 1 1 5A0C65ED
 P 1650 4700
@@
 	2200 5950 2200 6050
 $Comp
-L GND #PWR0116
+L node-rescue:GND #PWR0116
 U 1 1 5A0C6603
 P 2200 6050
@@
 $EndComp
 $Comp
-L C C1102
+L node-rescue:C C1102
 U 1 1 5A0C6609
 P 2550 5800
@@
 $EndComp
 $Comp
-L GND #PWR0117
+L node-rescue:GND #PWR0117
 U 1 1 5A0C660F
 P 2550 6050
@@
 Connection ~ 2550 5550
 $Comp
-L R R1106
+L node-rescue:R R1106
 U 1 1 5A0C661F
 P 2200 5800
@@
 $EndComp
 $Comp
-L R R1105
+L node-rescue:R R1105
 U 1 1 5A0C6625
 P 2200 5300
@@
 For 0-5V operation, simply remove 20kΩ\nand replaced 82kΩ with a 0Ω
 $Comp
-L Fuse F1102
+L node-rescue:Fuse F1102
 U 1 1 5A0A8A91
 P 2350 4950
@@
 $EndComp
 $Comp
-L +24V #PWR0118
+L node-rescue:+24V #PWR0118
 U 1 1 5A0E14DC
 P 2600 2050
@@
 $EndComp
 $Comp
-L +24V #PWR0119
+L node-rescue:+24V #PWR0119
 U 1 1 5A0E156A
 P 2650 4400
