File: LVDC Distribution Board/Inputs and Fusing.sch (KiCad schematic (older format))
At the start: 18 parts

Commit message: Hi Frank
More schematic work. Figuring out organization mostly.
Parts:
- gave numbers to parts that had none: 1
Connections:
- wire segments 50 -> 53
Other:
- note added: "Lug Terminals"

Commit message: Outputs Finalized
@Frank got all the outputs we talked about added. Also added nmos for cooling pump, inverter control. Current sensors are next and then DCDCs.
Connections:
- wire segments 53 -> 54
Other:
- note added: "Temp Sensor Inputs?"
Changed lines of the file:
@@
 $Descr A4 11693 8268
 encoding utf-8
-Sheet 2 6
+Sheet 2 7
 Title ""
 Date ""
@@
 Wire Wire Line
 	7620 2300 8140 2300
-Connection ~ 5260 4150
 Wire Wire Line
 	5260 2900 5260 4150
@@
 Wire Wire Line
 	5550 3660 5550 4150
-$Comp
-L power:Earth #PWR?
-U 1 1 5C030C09
-P 5260 4290
-F 0 "#PWR?" H 5260 4040 50  0001 C CNN
-F 1 "Earth" H 5260 4140 50  0001 C CNN
-F 2 "" H 5260 4290 50  0001 C CNN
-F 3 "~" H 5260 4290 50  0001 C CNN
-	1    5260 4290
-	1    0    0    -1
-$EndComp
-Wire Wire Line
-	5260 4150 5260 4290
 Text Notes 8520 4320 0    47   Italic 9
 POD_GND
@@
 $EndComp
 Wire Wire Line
-	3380 4370 3380 4140
-Wire Wire Line
-	3380 4140 3180 4140
-Wire Wire Line
-	3380 4140 3580 4140
-Connection ~ 3380 4140
+	3380 4380 3380 4370
+Wire Wire Line
+	3380 4150 3180 4150
+Connection ~ 3380 4150
 Wire Wire Line
 	3180 3560 3180 3480
@@
 $EndComp
 Wire Wire Line
-	3180 4140 2920 4140
+	3180 4150 2920 4150
 Wire Wire Line
 	2920 3610 2750 3610
-Connection ~ 3180 4140
+Connection ~ 3180 4150
 Wire Wire Line
 	2920 3270 2750 3270
@@
 Wire Wire Line
 	3700 2910 3740 2910
-Text Notes 5340 4410 0    47   Italic 9
-BAT_GND
-Wire Wire Line
-	3580 3850 3580 4140
-Wire Wire Line
-	3180 3860 3180 4140
 Wire Wire Line
 	2920 3270 2920 3610
-Connection ~ 2920 3610
-Wire Wire Line
-	2920 3610 2920 4140
+Wire Wire Line
+	2920 3620 2920 4150
 Text Notes 1860 2660 0    50   ~ 0
 Lug Terminals
+Connection ~ 5260 4150
+Connection ~ 3380 4370
+Wire Wire Line
+	3380 4370 3380 4150
+Wire Wire Line
+	3380 4150 3580 4150
+Wire Wire Line
+	3580 3850 3580 4150
+Connection ~ 3580 4150
+Wire Wire Line
+	3580 4150 5260 4150
+Wire Wire Line
+	3180 3860 3180 4150
+Text Notes 2310 4820 0    50   ~ 0
+Temp Sensor Inputs?
 $EndSCHEMATC

Commit message: Huge Chungus
Added all 8  current sensors to the schematic. Looks baller.
Parts:
- added 1k? (x2): R_US, symbol Device:R_US
- added U? (x2): ACS711, symbol LVDC-Library:ACS711
Connections:
- net labels added: +3V3, HPBAT_Voltage, HPBatt_Current, LPBAT_Voltage, LPBatt_Current
- net labels removed: BAT_VOLTAGE1, BAT_VOLTAGE2
- wire segments 54 -> 90
- no-connect marks 0 -> 2
Other:
- note added: "+-31A Capable"

Commit message: Inputs / Outputs Reallyyyy Done
These two schematic sections are very finalized now. Time to do the power conversion section : - )
Parts:
- removed 1k?, 2k: R_US, symbol Device:R_US
- removed BT?: Low Power Battery Pack, symbol Device:Battery
- removed BT?: High Power Battery Pack, symbol Device:Battery
- removed F? (x2): Fuse, symbol Device:Fuse
- added F? (x2): Fuse, symbol Device:Fuse
- added R?: 2k, symbol Device:R_US
- added R?: 1k, symbol Device:R_US
- added R? (x2): 900k, symbol Device:R_US
- added R? (x2): 100k, symbol Device:R_US
- R?: renamed from 2k; value R_US -> 2k
- R?: renamed from 1k?; value R_US -> 1k
Connections:
- net labels added: HPBAT_VSense, LP3V3, LPBAT_VSense
- wire segments 90 -> 95
Other:
- note added: "+-15A Capable"
- note added: "Battery Voltage Sense (30V --> 3V)"
- note removed: "+-31A Capable"

Commit message: Schematic "Done"
-Added Wiznet legacy n0de schematic
-Cleaned up schematic in general
-Other than minor changes, the schematic is finalized.
Parts:
- gave numbers to parts that had none: 24
Changed lines of the file:
@@
 Inputs and Fusing
 $Comp
-L Device:Q_NMOS_GDS Q?
+L Device:Q_NMOS_GDS Q202
 U 1 1 5C01F186
 P 7520 4170
-F 0 "Q?" V 7770 4170 50  0000 C CNN
+F 0 "Q202" V 7770 4170 50  0000 C CNN
 F 1 "Q_NMOS_GDS" V 7861 4170 50  0000 C CNN
 F 2 "" H 7720 4270 50  0001 C CNN
@@
 $EndComp
 $Comp
-L Device:R_US R?
+L Device:R_US R211
 U 1 1 5C02112F
 P 7910 3530
-F 0 "R?" H 7978 3576 50  0000 L CNN
+F 0 "R211" H 7978 3576 50  0000 L CNN
 F 1 "700k" H 7978 3485 50  0000 L CNN
 F 2 "" V 7950 3520 50  0001 C CNN
@@
 	7910 3770 7910 3680
 $Comp
-L Device:Q_NMOS_GDS Q?
+L Device:Q_NMOS_GDS Q201
 U 1 1 5C02823A
 P 6600 4170
-F 0 "Q?" V 6850 4170 50  0000 C CNN
+F 0 "Q201" V 6850 4170 50  0000 C CNN
 F 1 "Q_NMOS_GDS" V 6941 4170 50  0000 C CNN
 F 2 "" H 6800 4270 50  0001 C CNN
@@
 	6800 4270 6970 4270
 $Comp
-L Device:R_US R?
+L Device:R_US R209
 U 1 1 5C029257
 P 6970 3530
-F 0 "R?" H 7038 3576 50  0000 L CNN
+F 0 "R209" H 7038 3576 50  0000 L CNN
 F 1 "700k" H 7038 3485 50  0000 L CNN
 F 2 "" V 7010 3520 50  0001 C CNN
@@
 $EndComp
 $Comp
-L Device:R_US R?
+L Device:R_US R210
 U 1 1 5C0292B3
 P 6970 3980
-F 0 "R?" H 6902 3934 50  0000 R CNN
+F 0 "R210" H 6902 3934 50  0000 R CNN
 F 1 "200k" H 6902 4025 50  0000 R CNN
 F 2 "" V 7010 3970 50  0001 C CNN
@@
 	6970 4130 6970 4270
 $Comp
-L Device:R_US R?
+L Device:R_US R212
 U 1 1 5C0211AB
 P 7910 4010
-F 0 "R?" H 7842 3964 50  0000 R CNN
+F 0 "R212" H 7842 3964 50  0000 R CNN
 F 1 "200k" H 7842 4055 50  0000 R CNN
 F 2 "" V 7950 4000 50  0001 C CNN
@@
 POD_GND
 $Comp
-L Device:LED D?
+L Device:LED D201
 U 1 1 5C033289
 P 5170 3920
-F 0 "D?" V 5208 3803 50  0000 R CNN
+F 0 "D201" V 5208 3803 50  0000 R CNN
 F 1 "BLUE" V 5117 3803 50  0000 R CNN
 F 2 "" H 5170 3920 50  0001 C CNN
@@
 $EndComp
 $Comp
-L Device:LED D?
+L Device:LED D202
 U 1 1 5C033A1A
 P 5540 3920
-F 0 "D?" V 5578 3803 50  0000 R CNN
+F 0 "D202" V 5578 3803 50  0000 R CNN
 F 1 "BLUE" V 5487 3803 50  0000 R CNN
 F 2 "" H 5540 3920 50  0001 C CNN
@@
 $EndComp
 $Comp
-L Device:R_US R?
+L Device:R_US R208
 U 1 1 5C033BD3
 P 5540 3550
-F 0 "R?" H 5470 3520 50  0000 R CNN
+F 0 "R208" H 5470 3520 50  0000 R CNN
 F 1 "2k" H 5472 3595 50  0000 R CNN
 F 2 "" V 5580 3540 50  0001 C CNN
@@
 	5540 3770 5540 3700
 $Comp
-L Connector:Screw_Terminal_01x01 J?
+L Connector:Screw_Terminal_01x01 J204
 U 1 1 5C036982
 P 2060 1940
-F 0 "J?" H 1980 1715 50  0000 C CNN
+F 0 "J204" H 1980 1715 50  0000 C CNN
 F 1 "BAT_LP_IN+" H 1980 1806 50  0000 C CNN
 F 2 "" H 2060 1940 50  0001 C CNN
@@
 $EndComp
 $Comp
-L Connector:Screw_Terminal_01x01 J?
+L Connector:Screw_Terminal_01x01 J202
 U 1 1 5C036A9C
 P 2040 3310
-F 0 "J?" H 1960 3085 50  0000 C CNN
+F 0 "J202" H 1960 3085 50  0000 C CNN
 F 1 "BAT_HP_IN+" H 1960 3176 50  0000 C CNN
 F 2 "" H 2040 3310 50  0001 C CNN
@@
 HPBAT_Voltage
 $Comp
-L Connector:Screw_Terminal_01x01 J?
+L Connector:Screw_Terminal_01x01 J201
 U 1 1 5C03B9DA
 P 2030 4270
-F 0 "J?" H 1950 4045 50  0000 C CNN
+F 0 "J201" H 1950 4045 50  0000 C CNN
 F 1 "BAT_LP_IN-" H 1950 4136 50  0000 C CNN
 F 2 "" H 2030 4270 50  0001 C CNN
@@
 $EndComp
 $Comp
-L Connector:Screw_Terminal_01x01 J?
+L Connector:Screw_Terminal_01x01 J203
 U 1 1 5C03BA42
 P 2040 4810
-F 0 "J?" H 1960 4585 50  0000 C CNN
+F 0 "J203" H 1960 4585 50  0000 C CNN
 F 1 "BAT_LP_IN-" H 1960 4676 50  0000 C CNN
 F 2 "" H 2040 4810 50  0001 C CNN
@@
 Temp Sensor Inputs?
 $Comp
-L LVDC-Library:ACS711 U?
+L LVDC-Library:ACS711 U201
 U 1 1 5C3C05F3
 P 3960 2190
-F 0 "U?" H 3960 2705 50  0000 C CNN
+F 0 "U201" H 3960 2705 50  0000 C CNN
 F 1 "ACS711" H 3960 2614 50  0000 C CNN
 F 2 "" H 3860 2190 50  0001 C CNN
@@
 $EndComp
 $Comp
-L LVDC-Library:ACS711 U?
+L LVDC-Library:ACS711 U202
 U 1 1 5C3C0845
 P 3970 3560
-F 0 "U?" H 3970 4075 50  0000 C CNN
+F 0 "U202" H 3970 4075 50  0000 C CNN
 F 1 "ACS711" H 3970 3984 50  0000 C CNN
 F 2 "" H 3870 3560 50  0001 C CNN
@@
 P 3230 2350
 AR Path="/5BFB302C/5C3EC704" Ref="1k?"  Part="1"
-AR Path="/5BFB3004/5C3EC704" Ref="R?"  Part="1"
-F 0 "R?" H 3380 2290 50  0000 R CNN
+AR Path="/5BFB3004/5C3EC704" Ref="R201"  Part="1"
+F 0 "R201" H 3380 2290 50  0000 R CNN
 F 1 "1k" H 3380 2390 50  0000 R CNN
 F 2 "" V 3270 2340 50  0001 C CNN
@@
 +-15A Capable
 $Comp
-L Device:Fuse F?
+L Device:Fuse F201
 U 1 1 5C439696
 P 2570 1940
-F 0 "F?" V 2373 1940 50  0000 C CNN
+F 0 "F201" V 2373 1940 50  0000 C CNN
 F 1 "Fuse" V 2464 1940 50  0000 C CNN
 F 2 "" V 2500 1940 50  0001 C CNN
@@
 	2420 1940 2260 1940
 $Comp
-L Device:Fuse F?
+L Device:Fuse F202
 U 1 1 5C44409B
 P 2570 3310
-F 0 "F?" V 2373 3310 50  0000 C CNN
+F 0 "F202" V 2373 3310 50  0000 C CNN
 F 1 "Fuse" V 2464 3310 50  0000 C CNN
 F 2 "" V 2500 3310 50  0001 C CNN
@@
 HP_Vin+
 $Comp
-L Device:R_US R?
+L Device:R_US R207
 U 1 1 5C4654A3
 P 5170 3550
-F 0 "R?" H 5100 3520 50  0000 R CNN
+F 0 "R207" H 5100 3520 50  0000 R CNN
 F 1 "2k" H 5102 3595 50  0000 R CNN
 F 2 "" V 5210 3540 50  0001 C CNN
@@
 P 3240 3720
 AR Path="/5BFB302C/5C4657B5" Ref="R?"  Part="1"
-AR Path="/5BFB3004/5C4657B5" Ref="R?"  Part="1"
-F 0 "R?" H 3390 3660 50  0000 R CNN
+AR Path="/5BFB3004/5C4657B5" Ref="R202"  Part="1"
+F 0 "R202" H 3390 3660 50  0000 R CNN
 F 1 "1k" H 3390 3760 50  0000 R CNN
 F 2 "" V 3280 3710 50  0001 C CNN
@@
 $EndComp
 $Comp
-L Device:R_US R?
+L Device:R_US R203
 U 1 1 5C56D49A
 P 3700 5380
-F 0 "R?" H 3768 5426 50  0000 L CNN
+F 0 "R203" H 3768 5426 50  0000 L CNN
 F 1 "900k" H 3768 5335 50  0000 L CNN
 F 2 "" V 3740 5370 50  0001 C CNN
@@
 $EndComp
 $Comp
-L Device:R_US R?
+L Device:R_US R204
 U 1 1 5C56D525
 P 3700 5760
-F 0 "R?" H 3768 5806 50  0000 L CNN
+F 0 "R204" H 3768 5806 50  0000 L CNN
 F 1 "100k" H 3768 5715 50  0000 L CNN
 F 2 "" V 3740 5750 50  0001 C CNN
@@
 LPBAT_VSense
 $Comp
-L Device:R_US R?
+L Device:R_US R205
 U 1 1 5C579D47
 P 5150 5390
-F 0 "R?" H 5218 5436 50  0000 L CNN
+F 0 "R205" H 5218 5436 50  0000 L CNN
 F 1 "900k" H 5218 5345 50  0000 L CNN
 F 2 "" V 5190 5380 50  0001 C CNN
@@
 $EndComp
 $Comp
-L Device:R_US R?
+L Device:R_US R206
 U 1 1 5C579D4D
 P 5150 5770
-F 0 "R?" H 5218 5816 50  0000 L CNN
+F 0 "R206" H 5218 5816 50  0000 L CNN
 F 1 "100k" H 5218 5725 50  0000 L CNN
 F 2 "" V 5190 5760 50  0001 C CNN

Commit message: Rev Protection Fix
- Added LTspice models of reverse protection.
- Fixed reverse protection circuit, verified through spice.
- Added net names to NAP PoE circuit.
Parts:
- J203: value BAT_LP_IN- -> BAT_HP_IN-
- R210, R212: value 200k -> 500k
Connections:
- net labels removed: Earth
- wire segments 95 -> 97
Other:
- note removed: "BAT_GND"
Changed lines of the file:
@@
 U 1 1 5C01F186
 P 7520 4170
-F 0 "Q202" V 7770 4170 50  0000 C CNN
-F 1 "Q_NMOS_GDS" V 7861 4170 50  0000 C CNN
+F 0 "Q202" V 7760 4420 50  0000 C CNN
+F 1 "Q_NMOS_GDS" V 7760 4050 50  0000 C CNN
 F 2 "" H 7720 4270 50  0001 C CNN
 F 3 "DMTH6004SK3-13DICT-ND" H 7520 4170 50  0001 C CNN
@@
 U 1 1 5C02823A
 P 6600 4170
-F 0 "Q201" V 6850 4170 50  0000 C CNN
-F 1 "Q_NMOS_GDS" V 6941 4170 50  0000 C CNN
+F 0 "Q201" V 6820 3930 50  0000 C CNN
+F 1 "Q_NMOS_GDS" V 6830 4480 50  0000 C CNN
 F 2 "" H 6800 4270 50  0001 C CNN
 F 3 "DMTH6004SK3-13DICT-ND" H 6600 4170 50  0001 C CNN
@@
 P 6970 3980
 F 0 "R210" H 6902 3934 50  0000 R CNN
-F 1 "200k" H 6902 4025 50  0000 R CNN
+F 1 "500k" H 6902 4025 50  0000 R CNN
 F 2 "" V 7010 3970 50  0001 C CNN
 F 3 "~" H 6970 3980 50  0001 C CNN
@@
 Wire Wire Line
 	6970 3760 6970 3680
-Connection ~ 6970 4270
-Wire Wire Line
-	6970 4270 7320 4270
 Wire Wire Line
 	7520 3770 7910 3770
@@
 P 7910 4010
 F 0 "R212" H 7842 3964 50  0000 R CNN
-F 1 "200k" H 7842 4055 50  0000 R CNN
+F 1 "500k" H 7842 4055 50  0000 R CNN
 F 2 "" V 7950 4000 50  0001 C CNN
 F 3 "~" H 7910 4010 50  0001 C CNN
@@
 	-1   0    0    1
 $EndComp
-Connection ~ 5360 4270
 Wire Wire Line
 	5170 3770 5170 3700
@@
 	-1   0    0    1
 $EndComp
-Text Notes 5420 4500 0    47   Italic 9
-BAT_GND
 Text GLabel 3640 1500 2    47   Output Italic 0
 LPBAT_Voltage
@@
 P 2040 4810
 F 0 "J203" H 1960 4585 50  0000 C CNN
-F 1 "BAT_LP_IN-" H 1960 4676 50  0000 C CNN
+F 1 "BAT_HP_IN-" H 1960 4676 50  0000 C CNN
 F 2 "" H 2040 4810 50  0001 C CNN
 F 3 "~" H 2040 4810 50  0001 C CNN
@@
 	-1   0    0    1
 $EndComp
-Connection ~ 5170 4270
 Text Notes 1920 1460 0    47   Italic 9
 BATTERY INPUTS
@@
 Lug Terminals
 Wire Wire Line
-	5360 4490 5360 4270
-Wire Wire Line
-	5360 4270 5540 4270
-Wire Wire Line
 	5540 4070 5540 4270
 Wire Wire Line
@@
 	1    0    0    -1
 $EndComp
-Connection ~ 5540 4270
 Wire Wire Line
 	5170 2420 5170 3400
@@
 	3410 3310 3520 3310
 Connection ~ 3410 3310
-Connection ~ 2990 4270
-Wire Wire Line
-	2990 4270 2990 4810
 Wire Wire Line
 	3520 3610 3320 3610
@@
 	3410 2920 3580 2920
 Wire Wire Line
-	5170 4270 5360 4270
-Wire Wire Line
 	5540 4270 6400 4270
-Wire Wire Line
-	2990 4270 5170 4270
-$Comp
-L power:Earth #PWR0106
-U 1 1 5C034112
-P 5360 4490
-F 0 "#PWR0106" H 5360 4240 50  0001 C CNN
-F 1 "Earth" H 5360 4340 50  0001 C CNN
-F 2 "" H 5360 4490 50  0001 C CNN
-F 3 "~" H 5360 4490 50  0001 C CNN
-	1    5360 4490
-	1    0    0    -1
-$EndComp
 Text Notes 4140 3160 0    50   ~ 0
 +-15A Capable
@@
 Wire Wire Line
 	2420 3310 2240 3310
-Wire Wire Line
-	2240 4810 2990 4810
-Wire Wire Line
-	2230 4270 2990 4270
 Text HLabel 8430 2420 2    50   Output ~ 0
 LP_Vin+
@@
 Text Notes 3500 5010 0    50   ~ 0
 Battery Voltage Sense (30V --> 3V)
+Wire Wire Line
+	6970 4270 6970 4500
+Wire Wire Line
+	6970 4500 7910 4500
+Wire Wire Line
+	7910 4500 7910 4280
+Connection ~ 6970 4270
+Wire Wire Line
+	2230 4270 5170 4270
+Wire Wire Line
+	5540 4270 5540 4810
+Wire Wire Line
+	2240 4810 5540 4810
+Connection ~ 5540 4270
+Wire Wire Line
+	7320 4270 7140 4270
+Wire Wire Line
+	7140 4270 7140 4450
+Wire Wire Line
+	7140 4450 5170 4450
+Wire Wire Line
+	5170 4450 5170 4270
+Connection ~ 5170 4270
 $EndSCHEMATC
