File: IndicatorLEDs_PCB/IndicatorLEDs_PCB.kicad_pcb (KiCad board)
At the start: 2 copper layers, 60 x 60 mm, 22 parts, among them J1 M3 LUG, J2 M3 LUG, J3 BMS_I, J4 FRNT_LEDs, J5 M3 LUG, J6 M3 LUG, J7 REAR_LEDs, Q1 Q_PMOS_GSD, Q2 Q_PMOS_GSD, U1 LTV-357

Commit message: Routing done, gerbers gen'd, and bom added, frank order me
Parts:
- added logo1: SN_Block, µ104KiCAD:SN_BLOCK, B.Cu at (75.8, 136.0)
- added logo3: Logo, µ104KiCAD:Paradigm_Logo_Very_Small, B.Cu at (99.8, 135.8)
- added logo4: Logo, Symbol:ESD-Logo_6.6x6mm_SilkScreen, F.Cu at (83.8, 94.0)
- added logo5: Logo, µ104KiCAD:Symbol_HighVoltage_Type2_SilkTop_VerySmall, F.Cu at (59.2, 116.5)
- added logo6: Logo, Symbol:ESD-Logo_6.6x6mm_SilkScreen, B.Cu at (66.2, 141.8)
- added logo7: Logo, Symbol:KiCad-Logo_8mm_SilkScreen, B.Cu at (90.2, 95.0)
- added logo8: Logo, µ104KiCAD:Symbol_HighVoltage_Type2_SilkTop_VerySmall, B.Cu at (58.0, 109.8)
- logo2: moved to B.Cu
- moved logo2 139.0 mm to (79.8, 123.0)
- moved logo1 136.8 mm to (97.0, 136.0)
- moved logo3 136.8 mm to (72.5, 135.5)
- moved J6 16.0 mm to (93.8, 144.0)
- moved J5 13.0 mm to (78.8, 144.0)
- moved R5 6.61 mm to (84.0, 114.2), turned to 0 degrees
- moved Q1 3.34 mm to (84.0, 104.0)
- moved R4 3.29 mm to (84.0, 107.5)
- moved Q2 2.57 mm to (84.0, 117.8), turned to 180 degrees
- moved J3 1.00 mm to (95.7, 129.5)
- moved J4 0.75 mm to (95.7, 102.4)
- moved J7 0.50 mm to (95.7, 115.2)
- moved J1 0.35 mm to (65.8, 96.0)
- moved J2 0.35 mm to (56.0, 124.8)
Routing:
- net GND: track 0.00 -> 226.4 mm, vias 0 -> 36
- net +12V: track 0.00 -> 61.6 mm
- net /HV_Contactor_+: track 0.00 -> 43.2 mm
- net ISO_GND: track 0.00 -> 33.3 mm
- net /GREEN_LED_FRONT: track 0.00 -> 21.5 mm, vias 0 -> 1
- net /RED_LED_FRONT: track 0.00 -> 20.4 mm
- net /HV_Connected: track 0.00 -> 19.7 mm
- net Net-(R1-Pad1): track 0.00 -> 19.1 mm
- net /BMS_Shorted_I: track 0.00 -> 18.1 mm
- added copper zone on B.Cu, net GND
- added copper zone on F.Cu, net GND
Other:
- board text added: "FRONT LEDs"
- board text added: "HV GND"
- board text added: "HV_Contactor"
- board text added: "ORION BMS SHORT"
- board text added: "REAR LEDs"

Commit message: Make Frank Review changes
Other:
- board text added: "ISO FAULT BMS"
- board text removed: "ORION BMS SHORT"
Changed lines of the file:
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@@
   )
   (setup
-    (last_trace_width 0.1524)
+    (last_trace_width 0.25)
     (user_trace_width 0.1524)
     (user_trace_width 0.3048)
@@
     (effects (font (size 1 1) (thickness 0.25)) (justify left))
   )
-  (gr_text "ORION BMS SHORT\n" (at 92.5 125) (layer F.SilkS)
+  (gr_text "ISO FAULT BMS" (at 92.5 125) (layer F.SilkS)
     (effects (font (size 1 1) (thickness 0.25)) (justify left))
   )
