File: Wiring Harnesses/wiringHarnesses/High Voltage.sch (KiCad schematic (older format))
At the start: 0 parts

Commit message: Added node power cables and skeleton for other power cables
Other:
- note added: "Inverter J1\n"
- note added: "Inverter J2\n\n"
Changed lines of the file:
@@
 $Descr A4 11693 8268
 encoding utf-8
-Sheet 1 14
+Sheet 9 20
 Title ""
 Date ""
@@
 Comment4 ""
 $EndDescr
+$Sheet
+S 960  940  2340 1150
+U 5CD39FD0
+F0 "InverterJ1" 79
+F1 "InverterJ1.sch" 79
+$EndSheet
+$Sheet
+S 4690 940  2660 1150
+U 5CD39FD3
+F0 "InverterJ2" 79
+F1 "InverterJ2.sch" 79
+$EndSheet
+Text Notes 1520 1560 0    118  ~ 24
+Inverter J1\n
+Text Notes 5370 1790 0    118  ~ 24
+Inverter J2\n\n
 $EndSCHEMATC

Commit message: Added some bulkheads and internal HV connectors
Changed lines of the file:
@@
 $Descr A4 11693 8268
 encoding utf-8
-Sheet 9 20
+Sheet 8 20
 Title ""
 Date ""
@@
 $EndSheet
 $Sheet
-S 4690 940  2660 1150
+S 4090 890  2660 1150
 U 5CD39FD3
 F0 "InverterJ2" 79
@@
 Text Notes 1520 1560 0    118  ~ 24
 Inverter J1\n
-Text Notes 5370 1790 0    118  ~ 24
+Text Notes 4770 1740 0    118  ~ 24
 Inverter J2\n\n
 $EndSCHEMATC
