File: Wiring Harnesses/wiringHarnesses/InverterJ2.sch (KiCad schematic (older format))
At the start: 0 parts

Commit message: Created J2 inverter connector. Need to wire it up
Parts:
- added J?: Inverter_J2-connectors, symbol wiringHarnesses-rescue:Inverter_J2-connectors
Changed lines of the file:
@@
 EESchema Schematic File Version 4
 LIBS:wiringHarnesses-cache
-EELAYER 26 0
+EELAYER 29 0
 EELAYER END
 $Descr A4 11693 8268
@@
 Comment4 ""
 $EndDescr
+$Comp
+L wiringHarnesses-rescue:Inverter_J2-connectors J?
+U 1 1 5D20C60A
+P 3050 1650
+F 0 "J?" H 2658 1841 79  0000 C CNN
+F 1 "Inverter_J2-connectors" H 2658 1706 79  0000 C CNN
+F 2 "" H 3050 1700 79  0001 C CNN
+F 3 "" H 3050 1700 79  0001 C CNN
+	1    3050 1650
+	1    0    0    -1
+$EndComp
 $EndSCHEMATC

Commit message: updated to include new signal bulkheads. Still unsure of bb bms CAN wiring
Parts:
- removed J?: Inverter_J2-connectors, symbol wiringHarnesses-rescue:Inverter_J2-connectors
Changed lines of the file:
@@
 EESchema Schematic File Version 4
 LIBS:wiringHarnesses-cache
-EELAYER 29 0
+EELAYER 26 0
 EELAYER END
 $Descr A4 11693 8268
 encoding utf-8
-Sheet 10 20
+Sheet 10 21
 Title ""
 Date ""
@@
 Comment4 ""
 $EndDescr
-$Comp
-L wiringHarnesses-rescue:Inverter_J2-connectors J?
-U 1 1 5D20C60A
-P 3050 1650
-F 0 "J?" H 2658 1841 79  0000 C CNN
-F 1 "Inverter_J2-connectors" H 2658 1706 79  0000 C CNN
-F 2 "" H 3050 1700 79  0001 C CNN
-F 3 "" H 3050 1700 79  0001 C CNN
-	1    3050 1650
-	1    0    0    -1
-$EndComp
 $EndSCHEMATC
